Commit message: fix: joint_name

File: sobit_education_description/model/urdf/education_turtolebot_common_library.urdf.xacro (robot description, xacro)
@@ -47,5 +47,5 @@
     <color rgba="1.0 0.4 0.0 1.0"/>
   </material>
-  <joint name="fixed" type="fixed">
+  <joint name="base_arm_fixed_joint" type="fixed">
     <parent link="plate_top_link"/>
     <child link="base_arm_link"/>
@@ -558,5 +558,5 @@
   <!-- rgb_link -->
   <link name="rgb_link"/>
-  <joint name="xtion_joint5" type="fixed">
+  <joint name="rgb_fixed_link" type="fixed">
     <parent link="xtion"/>
     <child link="rgb_link"/>
@@ -567,5 +567,5 @@
   <!-- depth_link -->
   <link name="depth_link"/>
-  <joint name="xtion_joint6" type="fixed">
+  <joint name="depth_fixed_joint" type="fixed">
     <parent link="xtion"/>
     <child link="depth_link"/>
