Commit message: URDFの変更

File: sobit_education_description/robots/test.urdf (robot description, URDF)
Before this commit: robot turtlebot, 55 links, 54 joints
Links:
- removed link base_laser_link
- removed link board_base
- removed link depth_link
- removed link dev_board
- removed link link1
- removed link link10
- removed link link2
- removed link link3
- removed link link4
- removed link link5
- removed link link6
- removed link link7
- removed link link8
- removed link link9
- removed link mic
- removed link mic_link
- removed link mic_stand
- removed link pole_bottom_0_link_add
- removed link pole_bottom_1_link_add
- removed link pole_bottom_2_link_add
- removed link pole_bottom_3_link_add
- removed link rgb_link
- removed link sensor
- removed link xtion
- removed link xtion_link1
- removed link xtion_link2
- removed link xtion_link3
- removed link xtion_link4
- added link arm_base_link, mass 0.08; collision mesh filename=package://sobit_education_description/meshes/Manipulator_X4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; visual mesh filename=package://sobit_education_description/meshes/Manipulator_X4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
- added link arm_flex_dummy_link
- added link arm_flex_link, mass 0.08; collision mesh filename=package://sobit_education_description/meshes/Manipulator_X4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; visual mesh filename=package://sobit_education_description/meshes/Manipulator_X4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
- added link arm_roll_link, mass 0.08; collision mesh filename=package://sobit_education_description/meshes/Manipulator_X4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; visual mesh filename=package://sobit_education_description/meshes/Manipulator_X4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
- added link base_pole_link, mass 1; collision box size=0.02 0.02 0.6; visual box size=0.02 0.02 0.6
- added link elbow_flex_dummy_link
- added link hand_dummy_link, mass 0.08; collision mesh filename=package://sobit_education_description/meshes/Manipulator_X4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; visual mesh filename=package://sobit_education_description/meshes/Manipulator_X4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
- added link hand_l_link, mass 0.08; collision mesh filename=package://sobit_education_description/meshes/ManipulatorX4_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; visual mesh filename=package://sobit_education_description/meshes/ManipulatorX4_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
- added link hand_link
- added link hand_r_link, mass 0.08; collision mesh filename=package://sobit_education_description/meshes/ManipulatorX4_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; visual mesh filename=package://sobit_education_description/meshes/ManipulatorX4_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
- added link wrist_flex_link, mass 0.08; collision mesh filename=package://sobit_education_description/meshes/Manipulator_X4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; visual mesh filename=package://sobit_education_description/meshes/Manipulator_X4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
- added link xtion_pole_link, mass 1; collision box size=0.14 0.02 0.02; visual box size=0.14 0.02 0.02
- added link xtion_stand_link, mass 1; collision box size=0.033 0.033 0.051; visual box size=0.033 0.033 0.051
- added link xtion_tilt_link, mass 1; collision box size=0.02 0.041 0.028; visual box size=0.02 0.041 0.028
Joints:
- removed joint board_base_joint
- removed joint board_joint
- removed joint fixed
- removed joint joint1
- removed joint joint2
- removed joint joint3
- removed joint joint4
- removed joint joint5
- removed joint joint6
- removed joint joint7
- removed joint joint8
- removed joint joint9
- removed joint laser
- removed joint mic_joint1
- removed joint mic_joint2
- removed joint mic_joint3
- removed joint pole_bottom_0_joint_add
- removed joint pole_bottom_1_joint_add
- removed joint pole_bottom_2_joint_add
- removed joint pole_bottom_3_joint_add
- removed joint sensor_joint
- removed joint xtion_fixed
- removed joint xtion_joint1
- removed joint xtion_joint2
- removed joint xtion_joint3
- removed joint xtion_joint4
- removed joint xtion_joint5
- removed joint xtion_joint6
- added joint arm_base_fixed_joint: type fixed, parent plate_top_link, child arm_base_link, origin xyz=0.0 0.0 0.0 rpy=0 0 0, axis 0 0 1, limit lower=-3.14159265359 upper=3.14159265359 effort=30 velocity=1.57079632679
- added joint arm_flex_dummy_joint: type fixed, parent arm_flex_dummy_link, child arm_flex_link, origin xyz=0 0 0.0 rpy=0 0 0, axis 0 0 1, limit lower=-0.1 upper=0.1 effort=30 velocity=1.57079632679
- added joint arm_flex_joint: type revolute, parent arm_roll_link, child arm_flex_dummy_link, origin xyz=0.0 0.0 0.0421 rpy=0 0 0, axis 0 1 0, limit lower=0 upper=1.57079632679 effort=30 velocity=1.57079632679
- added joint arm_roll_joint: type revolute, parent arm_base_link, child arm_roll_link, origin xyz=0.13525 0.0 0.034 rpy=0 0 0, axis 0 0 1, limit lower=-3.14159265359 upper=3.14159265359 effort=30 velocity=1.57079632679
- added joint base_pole_joint: type fixed, parent plate_top_link, child base_pole_link, origin xyz=0 0.0 0.0 rpy=0 0 0, axis 0 0 1, limit lower=-3.14159265359 upper=3.14159265359 effort=30 velocity=1.57079632679
- added joint elbow_flex_dummy_joint: type fixed, parent elbow_flex_dummy_link, child wrist_flex_link, origin xyz=0 0 0.0 rpy=0 0 0, axis 0 0 1, limit lower=-0.1 upper=0.1 effort=30 velocity=1.57079632679
- added joint elbow_flex_joint: type revolute, parent arm_flex_link, child elbow_flex_dummy_link, origin xyz=0.024 0.0 0.148 rpy=0 1.57079632679 0, axis 0 1 0, limit lower=-1.57079632679 upper=1.4155 effort=30 velocity=1.57079632679
- added joint hand_dummy_joint: type revolute, parent wrist_flex_link, child hand_dummy_link, origin xyz=0.0 0.0 0.15 rpy=0 0 0, axis 0 1 0, limit lower=-1.57079632679 upper=1.57079632679 effort=30 velocity=1.57079632679
- added joint hand_joint: type revolute, parent hand_dummy_link, child hand_link, axis 1 0 0, limit lower=0.0 upper=1.57079632679 effort=1 velocity=1
- added joint hand_l_joint: type revolute, parent hand_dummy_link, child hand_l_link, origin xyz=0.0 0.01 0.04225 rpy=0.78 0 0, axis 1 0 0, limit lower=-1.57079632679 upper=0.0 effort=1 velocity=1, mimic joint=hand_joint multiplier=-1.0 offset=0.1
- added joint hand_r_joint: type revolute, parent hand_dummy_link, child hand_r_link, origin xyz=0.0 -0.01 0.04225 rpy=-0.78 0 0, axis 1 0 0, limit lower=0 upper=1.57079632679 effort=1 velocity=1, mimic joint=hand_joint multiplier=1.0 offset=-0.1
- added joint xtion_pole_joint: type fixed, parent base_pole_link, child xtion_pole_link, origin xyz=-0.062 0 0.373 rpy=0 0 0, axis 0 0 1, limit lower=-3.14159265359 upper=3.14159265359 effort=30 velocity=1.57079632679
- added joint xtion_stand_joint: type fixed, parent plate_top_link, child xtion_stand_link, origin xyz=0.14 0 0.0 rpy=0 0 0, axis 0 0 1, limit lower=-3.14159265359 upper=3.14159265359 effort=30 velocity=1.57079632679
- added joint xtion_tilt_joint: type revolute, parent xtion_stand_link, child xtion_tilt_link, origin xyz=0.0265 0 0.03 rpy=0 0 0, axis 0 1 0, limit lower=-1.57079632679 upper=1.57079632679 effort=30 velocity=1.57079632679
- joint plate_bottom_joint: axis 0 0 1 -> (none); limit lower=-3.14 upper=3.14 effort=30 velocity=1.571 -> (none)
- joint plate_middle_joint: axis 0 0 1 -> (none); limit lower=-3.14 upper=3.14 effort=30 velocity=1.571 -> (none); origin xyz=-0.01364 0.0 0.2264 rpy=0 0 0 -> xyz=-0.01364 0.0 0.1874 rpy=0 0 0
- joint plate_top_joint: axis 0 0 1 -> (none); limit lower=-3.14 upper=3.14 effort=30 velocity=1.571 -> (none); origin xyz=-0.01364 0.0  0.4356 rpy=0 0 0 -> xyz=-0.01364 0.0  0.3966 rpy=0 0 0
- joint pole_bottom_0_joint: axis 0 0 1 -> (none); limit lower=-3.14 upper=3.14 effort=30 velocity=1.571 -> (none)
- joint pole_bottom_1_joint: axis 0 0 1 -> (none); limit lower=-3.14 upper=3.14 effort=30 velocity=1.571 -> (none)
- joint pole_bottom_2_joint: axis 0 0 1 -> (none); limit lower=-3.14 upper=3.14 effort=30 velocity=1.571 -> (none)
- joint pole_bottom_3_joint: axis 0 0 1 -> (none); limit lower=-3.14 upper=3.14 effort=30 velocity=1.571 -> (none)
- joint pole_bottom_4_joint: axis 0 0 1 -> (none); limit lower=-3.14 upper=3.14 effort=30 velocity=1.571 -> (none)
- joint pole_bottom_5_joint: axis 0 0 1 -> (none); limit lower=-3.14 upper=3.14 effort=30 velocity=1.571 -> (none)
- joint pole_middle_0_joint: axis 0 0 1 -> (none); limit lower=-3.14 upper=3.14 effort=30 velocity=1.571 -> (none)
- joint pole_middle_1_joint: axis 0 0 1 -> (none); limit lower=-3.14 upper=3.14 effort=30 velocity=1.571 -> (none)
- joint pole_middle_2_joint: axis 0 0 1 -> (none); limit lower=-3.14 upper=3.14 effort=30 velocity=1.571 -> (none)
- joint pole_middle_3_joint: axis 0 0 1 -> (none); limit lower=-3.14 upper=3.14 effort=30 velocity=1.571 -> (none)
- joint pole_top_0_joint: axis 0 0 1 -> (none); limit lower=-3.14 upper=3.14 effort=30 velocity=1.571 -> (none); origin xyz=0.0381 0.1505 0.3312 rpy=0 0 0 -> xyz=0.0381 0.1505 0.292 rpy=0 0 0
- joint pole_top_1_joint: axis 0 0 1 -> (none); limit lower=-3.14 upper=3.14 effort=30 velocity=1.571 -> (none); origin xyz=0.0381 -0.1505 0.3312 rpy=0 0 0 -> xyz=0.0381 -0.1505 0.292 rpy=0 0 0
- joint pole_top_2_joint: axis 0 0 1 -> (none); limit lower=-3.14 upper=3.14 effort=30 velocity=1.571 -> (none); origin xyz=-0.0381 0.1505 0.3312 rpy=0 0 0 -> xyz=-0.0381 0.1505 0.292 rpy=0 0 0
- joint pole_top_3_joint: axis 0 0 1 -> (none); limit lower=-3.14 upper=3.14 effort=30 velocity=1.571 -> (none); origin xyz=-0.0381 -0.1505 0.3312 rpy=0 0 0 -> xyz=-0.0381 -0.1505 0.292 rpy=0 0 0
