Commit message: add/urg_sup_urdf

File: sobit_education_description/robots/sobit_education.urdf.xacro (robot description, xacro)
@@ -15,4 +15,5 @@
   <xacro:include filename="$(find sobit_education_description)/urdf/sensor/matrix.urdf.xacro" />
   <xacro:include filename="$(find sobit_education_description)/urdf/sensor/urg.urdf.xacro" />
+  <xacro:include filename="$(find sobit_education_description)/urdf/urg_sup/urg_sup.urdf.xacro" />
   <xacro:base/>
   <stack_hexagons parent="base_link" />
@@ -20,8 +21,9 @@
   <xacro:hand prefix="hand_motor" parent="wrist_flex_link"/>
   <xacro:pole parent="plate_top_link"/>
+  <xacro:urg_sup parent="plate_bottom_link"/>
   <xacro:xtion_motor prefix="xtion" parent="base_pole_link"/>
   <xacro:sensor_asus_xtion_pro parent="xtion_double_sided_tape_link"/>
   <xacro:mic parent="base_pole_link"/>
   <xacro:matrix parent="base_pole_link"/>
-  <xacro:urg parent="base_link"/>
+  <xacro:urg parent="base_urg_sup_link"/>
 </robot>

File: sobit_education_description/urdf/sensor/urg.urdf (new).xacro (robot description, xacro)
@@ -4,6 +4,5 @@
   <xacro:macro name="urg" params="parent">
     <joint name="base_laser_joint" type="fixed">
-      <!-- <origin xyz="0.18 0.0 0.38" rpy="0 0 0" /> -->
-      <origin xyz="0.0 0.0 0.0" rpy="0 0 0" />
+      <origin xyz="0.18 0.0 0.38" rpy="0 0 0" />
       <parent link="${parent}" />
       <child link="base_laser_link" />

Commit message: fix xacro for noetic

File: sobit_education_description/robots/sobit_education.urdf.xacro (robot description, xacro)
@@ -1,4 +1,4 @@
 <?xml version="1.0" ?>
-<robot name="sobit_education" xmlns:controller="http://playerstage.sourceforge.net/gazebo/xmlschema/#controller" xmlns:interface="http://playerstage.sourceforge.net/gazebo/xmlschema/#interface" xmlns:sensor="http://playerstage.sourceforge.net/gazebo/xmlschema/#sensor" xmlns:xacro="http://www.ros.org/wiki.xacro">
+<robot name="sobit_education" xmlns:controller="http://playerstage.sourceforge.net/gazebo/xmlschema/#controller" xmlns:interface="http://playerstage.sourceforge.net/gazebo/xmlschema/#interface" xmlns:sensor="http://playerstage.sourceforge.net/gazebo/xmlschema/#sensor" xmlns:xacro="http://www.ros.org/wiki/xacro">
   <!-- common xacro -->
   <xacro:include filename="$(find sobit_education_description)/urdf/common.xacro" />
@@ -17,5 +17,5 @@
   <xacro:include filename="$(find sobit_education_description)/urdf/urg_sup/urg_sup.urdf.xacro" />
   <xacro:base/>
-  <stack_hexagons parent="base_link" />
+  <xacro:stack_hexagons parent="base_link" />
   <xacro:arm prefix="arm" parent="plate_top_link"/>
   <xacro:hand prefix="hand_motor" parent="wrist_flex_link"/>

File: sobit_education_description/urdf/common.xacro (robot description, xacro)
@@ -1,6 +1,6 @@
 <?xml version="1.0" ?>
-<robot xmlns:xacro="http://www.ros.org/wiki.xacro">
+<robot xmlns:xacro="http://www.ros.org/wiki/xacro">
   <xacro:property name="M_PI" value="3.14159265359" />
-  <macro name="position_joint_transmission" params="joint reduction">
+  <xacro:macro name="position_joint_transmission" params="joint reduction">
     <transmission name="${joint}_transmission">
       <type>transmission_interface/SimpleTransmission</type>
@@ -13,4 +13,4 @@
       </actuator>
     </transmission>
-  </macro>
+  </xacro:macro>
 </robot>

File: sobit_education_description/urdf/materials.urdf.xacro (robot description, xacro)
@@ -16,3 +16,6 @@
     <color rgba="0.0 0.0 1.0 1.0" />
   </material>
+  <material name="white">
+    <color rgba="1.0 1.0 1.0 1.0"/>
+  </material>
 </robot>

Commit message: update urdf

File: sobit_education_description/robots/sobit_education.urdf.xacro (robot description, xacro)
@@ -4,5 +4,4 @@
   <xacro:include filename="$(find sobit_education_description)/urdf/common.xacro" />
   <xacro:include filename="$(find sobit_education_description)/urdf/materials.urdf.xacro" />
-  <xacro:include filename="$(find urg_node)/urdf/hokuyo_ust10.urdf.xacro" />
   <!-- Add URDF: links, joints -->
   <xacro:include filename="$(find sobit_education_description)/urdf/base/base.urdf.xacro" />
@@ -17,4 +16,5 @@
   <xacro:include filename="$(find sobit_education_description)/urdf/sensor/matrix.urdf.xacro" />
   <xacro:include filename="$(find sobit_education_description)/urdf/sensor/urg.urdf.xacro" />
+  <xacro:include filename="$(find urg_node)/urdf/hokuyo_ust.urdf.xacro" />
   <!-- Connect the previous Links and Joints -->
   <xacro:base/>

File: sobit_education_description/urdf/body/cover.urdf.xacro (robot description, xacro)
@@ -7,5 +7,4 @@
       <child link="${prefix}_link" />
       <axis xyz="0 0 1 "/>
-      <limit effort="30" lower="-3.14" upper="3.14" velocity="1.571 "/>
     </joint>
     <link name="${prefix}_link">
