Commit message: urdf名の変更

File: sobit_education_description/urdf/sensor/urg.urdf.xacro (robot description, xacro)
@@ -3,13 +3,13 @@
   xmlns:xacro="http://ros.org/wiki/xacro">
   <xacro:macro name="urg" params="parent">
-    <joint name="urg_joint" type="fixed">
+    <joint name="base_laser_joint" type="fixed">
       <origin xyz="0.205 0.0 0.01" rpy="0 0 0" />
       <parent link="${parent}" />
-      <child link="urg" />
+      <child link="base_laser_link" />
       <origin rpy="0 0 0" xyz="0.13525 0.0 0.034"/>
       <axis xyz="0 0 1"/>
       <limit effort="30" lower="-3.14" upper="3.14" velocity="1.571"/>
     </joint>
-    <link name="urg">
+    <link name="base_laser_link">
       <visual>
         <geometry>

Commit message: add xtion_tilt_ctrl

File: sobit_education_description/urdf/sensor/urg.urdf.xacro (robot description, xacro)
@@ -4,5 +4,5 @@
   <xacro:macro name="urg" params="parent">
     <joint name="base_laser_joint" type="fixed">
-      <origin xyz="0.205 0.0 0.01" rpy="0 0 0" />
+      <origin xyz="0.11 0.0 0.28" rpy="0 0 0" />
       <parent link="${parent}" />
       <child link="base_laser_link" />

Commit message: urg_urdf

File: sobit_education_description/urdf/sensor/urg.urdf.xacro (robot description, xacro)
@@ -4,5 +4,5 @@
   <xacro:macro name="urg" params="parent">
     <joint name="base_laser_joint" type="fixed">
-      <origin xyz="0.11 0.0 0.28" rpy="0 0 0" />
+      <origin xyz="0.18 0.0 0.38" rpy="0 0 0" />
       <parent link="${parent}" />
       <child link="base_laser_link" />
