Commit message: update/urg_sup_position

File: sobit_education_description/urdf/urg_sup/urg_sup.urdf.xacro (robot description, xacro)
@@ -4,5 +4,5 @@
   <xacro:macro name="urg_sup" params="parent">
     <joint name="base_urg_sup_joint" type="fixed">
-      <origin xyz="0.194084 0.0 0.00475" rpy="0 0 0" />
+      <origin xyz="0.194084 0.0 0.0085" rpy="0 0 0" />
       <parent link="${parent}" />
       <child link="base_urg_sup_link" />
