Commit message: add/new_joint_for_motor

File: sobit_education_description/urdf/arm/arm.transmission (backup).xacro (robot description, xacro)
@@ -3,6 +3,5 @@
   <xacro:macro name="arm_transmission" params="prefix">
     <position_joint_transmission joint="${prefix}_roll_joint" reduction="1" />
-    <position_joint_transmission joint="${prefix}_flex_joint_rgt" reduction="1" />
-    <position_joint_transmission joint="${prefix}_flex_joint_lft" reduction="1" />
+    <position_joint_transmission joint="${prefix}_flex_joint" reduction="1" />
     <position_joint_transmission joint="elbow_flex_joint" reduction="1" />
     <position_joint_transmission joint="wrist_flex_joint" reduction="1" />

File: sobit_education_description/urdf/arm/arm.urdf (backup).xacro (robot description, xacro)
@@ -44,5 +44,5 @@
       </inertial>
     </link>
-    <joint name="${prefix}_flex_joint_rgt" type="revolute">
+    <joint name="${prefix}_flex_joint" type="revolute">
       <parent link="${prefix}_roll_link"/>
       <child link="${prefix}_flex_link"/>
@@ -63,14 +63,4 @@
         <inertia ixx="1.0" ixy="0.0" ixz="0.0" iyy="1.0" iyz="0.0" izz="1.0"/>
       </inertial>
-    </link>
-    <joint name="${prefix}_flex_joint_lft" type="revolute">
-      <parent link="${prefix}_roll_link"/>
-      <child link="${prefix}_flex_link_rgt_lft"/>
-      <origin rpy="0 0 ${M_PI}" xyz="0.0 0.0 0.0"/>
-      <axis xyz="0 -1 0"/>
-      <limit effort="30" lower="${-M_PI/2.0}" upper="${M_PI/2.0}" velocity="${M_PI/2.0}"/>
-    </joint>
-    <link name="${prefix}_flex_link_rgt_lft">
-      <origin rpy="0 0 0" xyz="0 0 0"/>
     </link>
     <joint name="elbow_flex_joint" type="revolute">
