Commit message: add/urdf_new_motors

File: sobit_education_description/urdf/arm/arm.transmission.xacro (robot description, xacro)
@@ -5,5 +5,6 @@
     <position_joint_transmission joint="${prefix}_flex_joint_rgt" reduction="1" />
     <position_joint_transmission joint="${prefix}_flex_joint_lft" reduction="1" />
-    <position_joint_transmission joint="elbow_flex_joint" reduction="1" />
+    <position_joint_transmission joint="elbow_flex_joint_rgt" reduction="1" />
+    <position_joint_transmission joint="elbow_flex_joint_lft" reduction="1" />
     <position_joint_transmission joint="wrist_flex_joint" reduction="1" />
   </xacro:macro>

File: sobit_education_description/urdf/arm/arm.urdf.xacro (robot description, xacro)
@@ -74,5 +74,5 @@
       <origin rpy="0 0 0" xyz="0 0 0"/>
     </link>
-    <joint name="elbow_flex_joint" type="revolute">
+    <joint name="elbow_flex_joint_rgt" type="revolute">
       <parent link="${prefix}_flex_link"/>
       <child link="elbow_flex_link"/>
@@ -82,4 +82,14 @@
     </joint>
     <link name="elbow_flex_link"/>
+    <joint name="elbow_flex_joint_lft" type="revolute">
+      <parent link="${prefix}_flex_link"/>
+      <child link="elbow_flex_link_rgt_lft"/>
+      <origin rpy="0 0 ${M_PI}" xyz="0.0 0.0 0.0"/>
+      <axis xyz="0 -1 0"/>
+      <limit effort="30" lower="${-M_PI/2.0}" upper="1.4155" velocity="${M_PI/2.0}"/>
+    </joint>
+    <link name="elbow_flex_link_rgt_lft">
+      <origin rpy="0 0 0" xyz="0 0 0"/>
+    </link>
     <joint name="wrist_flex_dummy_joint" type="fixed">
       <parent link="elbow_flex_link"/>
