Commit message: hotfix/tf_error

File: sobit_education_description/urdf/arm/arm.urdf.xacro (robot description, xacro)
@@ -28,5 +28,5 @@
       <child link="${prefix}_roll_link"/>
       <origin rpy="0 0 0" xyz="0.13577 0.0 0.04314"/>
-      <axis xyz="0 0 1"/>
+      <axis xyz="0 0 -1"/>
       <limit effort="30" lower="${-M_PI}" upper="${M_PI}" velocity="${M_PI/2.0}"/>
     </joint>
@@ -48,5 +48,5 @@
       <child link="${prefix}_flex_link"/>
       <origin rpy="0 0 0" xyz="0.0 0.0 0.0407"/>
-      <axis xyz="0 1 0"/>
+      <axis xyz="0 -1 0"/>
       <limit effort="30" lower="${-M_PI/2.0}" upper="${M_PI/2.0}" velocity="${M_PI/2.0}"/>
     </joint>
@@ -68,5 +68,5 @@
       <child link="elbow_flex_link"/>
       <origin rpy="0 0 0" xyz="0.0235 0.0 0.148"/>
-      <axis xyz="0 1 0"/>
+      <axis xyz="0 -1 0"/>
       <limit effort="30" lower="${-M_PI/2.0}" upper="1.4155" velocity="${M_PI/2.0}"/>
     </joint>
@@ -96,5 +96,5 @@
       <child link="wrist_flex_link"/>
       <origin rpy="0 0 0" xyz="0.152 0.0 0.0"/>
-      <axis xyz="0 1 0"/>
+      <axis xyz="0 -1 0"/>
       <limit effort="30" lower="${-M_PI/2.0}" upper="${M_PI/2.0}" velocity="${M_PI/2.0}"/>
     </joint>

File: sobit_education_description/urdf/xtion_motor/xtion_motor.urdf.xacro (robot description, xacro)
@@ -8,5 +8,5 @@
       <child link="${prefix}_pan_link"/>
       <origin rpy="${-M_PI/2.0} ${-M_PI/2.0} 0" xyz="0 0.396 0.191"/>
-      <axis xyz="0 0 1"/>
+      <axis xyz="0 0 -1"/>
       <limit effort="30" lower="${-M_PI/2.0}" upper="${M_PI/2.0}" velocity="${M_PI/2.0}"/>
     </joint>
@@ -28,5 +28,5 @@
       <child link="${prefix}_tilt_link"/>
       <origin rpy="${-M_PI/2.0} ${-M_PI/2.0} 0" xyz="0.0 0.0 0.0428"/>
-      <axis xyz="0 0 1"/>
+      <axis xyz="0 0 -1"/>
       <limit effort="30" lower="${-M_PI/2.0}" upper="${M_PI/2.0}" velocity="${M_PI/2.0}"/>
     </joint>
@@ -48,5 +48,5 @@
       <child link="${prefix}_double_sided_tape_link"/>
       <origin rpy="0.05 0 -0.06" xyz="0.02050 0.0 0.0"/>
-      <axis xyz="0 0 1"/>
+      <axis xyz="0 0 -1"/>
       <limit effort="30" lower="${-M_PI/2.0}" upper="${M_PI/2.0}" velocity="${M_PI/2.0}"/>
     </joint>

Commit message: update format

File: sobit_education_description/urdf/arm/arm.urdf.xacro (robot description, xacro)
@@ -4,133 +4,143 @@
   <xacro:include filename="$(find sobit_education_description)/urdf/arm/arm.transmission.xacro" />
   <xacro:macro name="arm" params="prefix parent">
-    <joint name="${prefix}_base_fixed_joint" type="fixed">
-      <parent link="${parent}"/>
-      <child link="${prefix}_base_link"/>
-      <origin rpy="0 0 0" xyz="0.0 0.0 0.0"/>
-      <axis xyz="0 0 1"/>
-      <limit effort="30" lower="${-M_PI}" upper="${M_PI}" velocity="${M_PI/2.0}"/>
+    <joint name="${prefix}_base_joint" type="fixed">
+      <parent link="${parent}" />
+      <child link="${prefix}_base_link" />
+      <origin xyz="0.0 0.0 0.0" rpy="0.0 0.0 0.0" />
+      <axis xyz="0 0 1" />
+      <limit effort="30" lower="${-M_PI}" upper="${M_PI}" velocity="${M_PI/2.0}" />
     </joint>
     <link name="${prefix}_base_link">
       <visual>
-        <origin rpy="0 0 0" xyz="0.0845 0 0"/>
+        <origin xyz="0.0845 0.0 0.0" rpy="0.0 0.0 0.0" />
         <geometry>
-          <mesh filename="package://sobit_education_description/meshes/Manipulator_X4_Joint1_fix.dae"/>
+          <mesh filename="package://sobit_education_description/meshes/Manipulator_X4_Joint1_fix.dae" />
         </geometry>
       </visual>
       <inertial>
-        <origin rpy="0 0 0" xyz="0.0845 0 0"/>
-        <mass value="0.08"/>
-        <inertia ixx="1.0" ixy="0.0" ixz="0.0" iyy="1.0" iyz="0.0" izz="1.0"/>
+        <origin xyz="0.0845 0.0 0.0" rpy="0.0 0.0 0.0" />
+        <mass value="0.08" />
+        <inertia ixx="1.0" ixy="0.0" ixz="0.0"
+                 iyy="1.0" iyz="0.0"
+                 izz="1.0" />
       </inertial>
     </link>
     <joint name="${prefix}_roll_joint" type="revolute">
-      <parent link="${prefix}_base_link"/>
-      <child link="${prefix}_roll_link"/>
-      <origin rpy="0 0 0" xyz="0.13577 0.0 0.04314"/>
-      <axis xyz="0 0 -1"/>
-      <limit effort="30" lower="${-M_PI}" upper="${M_PI}" velocity="${M_PI/2.0}"/>
+      <parent link="${prefix}_base_link" />
+      <child link="${prefix}_roll_link" />
+      <origin xyz="0.13577 0.0 0.04314" rpy="0.0 0.0 0.0" />
+      <axis xyz="0 0 -1" />
+      <limit effort="30" lower="${-M_PI}" upper="${M_PI}" velocity="${M_PI/2.0}" />
     </joint>
     <link name="${prefix}_roll_link">
       <visual>
-        <origin rpy="0 0 0" xyz="-0.001 0 -0.0005"/>
+        <origin xyz="-0.001 0 -0.0005" rpy="0.0 0.0 0.0" />
         <geometry>
-          <mesh filename="package://sobit_education_description/meshes/Manipulator_X4_Joint2_fix.dae"/>
+          <mesh filename="package://sobit_education_description/meshes/Manipulator_X4_Joint2_fix.dae" />
         </geometry>
       </visual>
       <inertial>
-        <origin rpy="0 0 0" xyz="0 0 0.0"/>
-        <mass value="0.08"/>
-        <inertia ixx="1.0" ixy="0.0" ixz="0.0" iyy="1.0" iyz="0.0" izz="1.0"/>
+        <origin xyz="0.0 0.0 0.0" rpy="0.0 0.0 0.0" />
+        <mass value="0.08" />
+        <inertia ixx="1.0" ixy="0.0" ixz="0.0"
+                 iyy="1.0" iyz="0.0"
+                 izz="1.0" />
       </inertial>
     </link>
     <joint name="${prefix}_flex_joint_rgt" type="revolute">
-      <parent link="${prefix}_roll_link"/>
-      <child link="${prefix}_flex_link"/>
-      <origin rpy="0 0 0" xyz="0.0 0.0 0.0407"/>
-      <axis xyz="0 -1 0"/>
-      <limit effort="30" lower="${-M_PI/2.0}" upper="${M_PI/2.0}" velocity="${M_PI/2.0}"/>
+      <parent link="${prefix}_roll_link" />
+      <child link="${prefix}_flex_link" />
+      <origin xyz="0.0 0.0 0.0407" rpy="0.0 0.0 0.0" />
+      <axis xyz="0 -1 0" />
+      <limit effort="30" lower="${-M_PI/2.0}" upper="${M_PI/2.0}" velocity="${M_PI/2.0}" />
     </joint>
     <link name="${prefix}_flex_link">
       <visual>
-        <origin rpy="0 0 0" xyz="0 0.00025 0"/>
+        <origin xyz="0 0.00025 0.0" rpy="0.0 0.0 0.0" />
         <geometry>
-          <mesh filename="package://sobit_education_description/meshes/Manipulator_X4_Joint3_fix.dae"/>
+          <mesh filename="package://sobit_education_description/meshes/Manipulator_X4_Joint3_fix.dae" />
         </geometry>
       </visual>
       <inertial>
-        <origin rpy="0 0 0" xyz="0 0 0"/>
-        <mass value="0.08"/>
-        <inertia ixx="1.0" ixy="0.0" ixz="0.0" iyy="1.0" iyz="0.0" izz="1.0"/>
+        <origin xyz="0.0 0.0 0.0" rpy="0.0 0.0 0.0" />
+        <mass value="0.08" />
+        <inertia ixx="1.0" ixy="0.0" ixz="0.0"
+                 iyy="1.0" iyz="0.0"
+                 izz="1.0" />
       </inertial>
     </link>
     <joint name="${prefix}_flex_joint_lft" type="revolute">
-      <parent link="${prefix}_roll_link"/>
-      <child link="${prefix}_flex_link_rgt_lft"/>
-      <origin rpy="0 0 ${M_PI}" xyz="0.0 0.0 0.0"/>
-      <axis xyz="0 -1 0"/>
-      <limit effort="30" lower="${-M_PI/2.0}" upper="${M_PI/2.0}" velocity="${M_PI/2.0}"/>
+      <parent link="${prefix}_roll_link" />
+      <child link="${prefix}_flex_link_rgt_lft" />
+      <origin xyz="0.0 0.0 0.0" rpy="0 0 ${M_PI}" />
+      <axis xyz="0 -1 0" />
+      <limit effort="30" lower="${-M_PI/2.0}" upper="${M_PI/2.0}" velocity="${M_PI/2.0}" />
     </joint>
     <link name="${prefix}_flex_link_rgt_lft">
-      <origin rpy="0 0 0" xyz="0 0 0"/>
+      <origin xyz="0.0 0.0 0.0" rpy="0.0 0.0 0.0" />
     </link>
     <joint name="elbow_flex_joint_rgt" type="revolute">
-      <parent link="${prefix}_flex_link"/>
-      <child link="elbow_flex_link"/>
-      <origin rpy="0 0 0" xyz="0.0235 0.0 0.148"/>
-      <axis xyz="0 -1 0"/>
-      <limit effort="30" lower="${-M_PI/2.0}" upper="1.4155" velocity="${M_PI/2.0}"/>
+      <parent link="${prefix}_flex_link" />
+      <child link="elbow_flex_link" />
+      <origin xyz="0.0235 0.0 0.148" rpy="0.0 0.0 0.0" />
+      <axis xyz="0 -1 0" />
+      <limit effort="30" lower="${-M_PI/2.0}" upper="1.4155" velocity="${M_PI/2.0}" />
     </joint>
-    <link name="elbow_flex_link"/>
+    <link name="elbow_flex_link" />
     <joint name="elbow_flex_joint_lft" type="revolute">
-      <parent link="${prefix}_flex_link"/>
-      <child link="elbow_flex_link_rgt_lft"/>
-      <origin rpy="0 0 ${M_PI}" xyz="0.0 0.0 0.0"/>
-      <axis xyz="0 -1 0"/>
-      <limit effort="30" lower="${-M_PI/2.0}" upper="1.4155" velocity="${M_PI/2.0}"/>
+      <parent link="${prefix}_flex_link" />
+      <child link="elbow_flex_link_rgt_lft" />
+      <origin xyz="0.0 0.0 0.0" rpy="0 0 ${M_PI}" />
+      <axis xyz="0 -1 0" />
+      <limit effort="30" lower="${-M_PI/2.0}" upper="1.4155" velocity="${M_PI/2.0}" />
     </joint>
     <link name="elbow_flex_link_rgt_lft">
-      <origin rpy="0 0 0" xyz="0 0 0"/>
+      <origin xyz="0.0 0.0 0.0" rpy="0.0 0.0 0.0" />
     </link>
     <joint name="wrist_flex_dummy_joint" type="fixed">
-      <parent link="elbow_flex_link"/>
-      <child link="wrist_flex_dummy_link"/>
-      <origin rpy="0 0 0" xyz="0 0 0.0"/>
-      <axis xyz="0 0 1"/>
-      <limit effort="30" lower="-0.1" upper="0.1" velocity="${M_PI/2.0}"/>
+      <parent link="elbow_flex_link" />
+      <child link="wrist_flex_dummy_link" />
+      <origin xyz="0.0 0.0 0.0" rpy="0.0 0.0 0.0" />
+      <axis xyz="0 0 1" />
+      <limit effort="30" lower="-0.1" upper="0.1" velocity="${M_PI/2.0}" />
     </joint>
     <link name="wrist_flex_dummy_link">
       <visual>
-        <origin rpy="0 ${M_PI/2.0-0.02} 0" xyz="-0.0005 -0.0001 0"/>
+        <origin xyz="-0.0005 -0.0001 0.0" rpy="0.0 ${M_PI/2.0-0.02} 0.0" />
         <geometry>
-          <mesh filename="package://sobit_education_description/meshes/Manipulator_X4_Joint4_fix.dae"/>
+          <mesh filename="package://sobit_education_description/meshes/Manipulator_X4_Joint4_fix.dae" />
         </geometry>
       </visual>
       <inertial>
-        <origin rpy="0 0 0" xyz="0 0 0"/>
-        <mass value="0.08"/>
-        <inertia ixx="1.0" ixy="0.0" ixz="0.0" iyy="1.0" iyz="0.0" izz="1.0"/>
+        <origin xyz="0.0 0.0 0.0" rpy="0.0 0.0 0.0" />
+        <mass value="0.08" />
+        <inertia ixx="1.0" ixy="0.0" ixz="0.0"
+                 iyy="1.0" iyz="0.0"
+                 izz="1.0" />
       </inertial>
     </link>
     <joint name="wrist_flex_joint" type="revolute">
-      <parent link="wrist_flex_dummy_link"/>
-      <child link="wrist_flex_link"/>
-      <origin rpy="0 0 0" xyz="0.152 0.0 0.0"/>
-      <axis xyz="0 -1 0"/>
-      <limit effort="30" lower="${-M_PI/2.0}" upper="${M_PI/2.0}" velocity="${M_PI/2.0}"/>
+      <parent link="wrist_flex_dummy_link" />
+      <child link="wrist_flex_link" />
+      <origin xyz="0.152 0.0 0.0" rpy="0.0 0.0 0.0" />
+      <axis xyz="0 -1 0" />
+      <limit effort="30" lower="${-M_PI/2.0}" upper="${M_PI/2.0}" velocity="${M_PI/2.0}" />
     </joint>
     <link name="wrist_flex_link">
       <visual>
-        <origin rpy="0 ${M_PI/2.0} 0" xyz="-0.0005 -0.0001 0"/>
+        <origin xyz="-0.0005 -0.0001 0.0" rpy="0.0 ${M_PI/2.0} 0.0" />
         <geometry>
-          <mesh filename="package://sobit_education_description/meshes/Manipulator_X4_Gripper_fix.dae"/>
+          <mesh filename="package://sobit_education_description/meshes/Manipulator_X4_Gripper_fix.dae" />
         </geometry>
       </visual>
       <inertial>
-        <origin rpy="0 0 0" xyz="0 0 0"/>
-        <mass value="0.08"/>
-        <inertia ixx="1.0" ixy="0.0" ixz="0.0" iyy="1.0" iyz="0.0" izz="1.0"/>
+        <origin xyz="0.0 0.0 0.0" rpy="0.0 0.0 0.0" />
+        <mass value="0.08" />
+        <inertia ixx="1.0" ixy="0.0" ixz="0.0"
+                 iyy="1.0" iyz="0.0"
+                 izz="1.0" />
       </inertial>
     </link>
-    <xacro:arm_transmission prefix="${prefix}"/>
+    <xacro:arm_transmission prefix="${prefix}" />
   </xacro:macro>
 </robot>
