Commit message: update arm and hand urdf

File: sobit_education_description/urdf/arm/arm.urdf.xacro (robot description, xacro)
@@ -1,41 +1,20 @@
 <?xml version="1.0" encoding="UTF-8" ?>
-<robot name="arm"
-  xmlns:xacro="http://ros.org/wiki/xacro">
+<robot name="arm" xmlns:xacro="http://ros.org/wiki/xacro">
   <xacro:include filename="$(find sobit_education_description)/urdf/arm/arm.transmission.xacro" />
   <xacro:macro name="arm" params="prefix parent">
+    <!-- Include transmission rules -->
+    <xacro:arm_transmission prefix="${prefix}" />
     <joint name="${prefix}_base_joint" type="fixed">
       <parent link="${parent}" />
       <child link="${prefix}_base_link" />
-      <origin xyz="0.0 0.0 0.0" rpy="0.0 0.0 0.0" />
+      <origin xyz="0.127231 0.0 0.0" rpy="0.0 0.0 0.0" />
       <axis xyz="0 0 1" />
-      <limit effort="30" lower="${-M_PI}" upper="${M_PI}" velocity="${M_PI/2.0}" />
+      <!-- <limit effort="30" lower="${-M_PI}" upper="${M_PI}" velocity="${M_PI/2.0}" /> -->
     </joint>
     <link name="${prefix}_base_link">
       <visual>
-        <origin xyz="0.0845 0.0 0.0" rpy="0.0 0.0 0.0" />
+        <origin xyz="0.0 0.0 0.0" rpy="0.0 0.0 ${M_PI/2.0}" />
         <geometry>
-          <mesh filename="package://sobit_education_description/meshes/Manipulator_X4_Joint1_fix.dae" />
-        </geometry>
-      </visual>
-      <inertial>
-        <origin xyz="0.0845 0.0 0.0" rpy="0.0 0.0 0.0" />
-        <mass value="0.08" />
-        <inertia ixx="1.0" ixy="0.0" ixz="0.0"
-                 iyy="1.0" iyz="0.0"
-                 izz="1.0" />
-      </inertial>
-    </link>
-    <joint name="${prefix}_roll_joint" type="revolute">
-      <parent link="${prefix}_base_link" />
-      <child link="${prefix}_roll_link" />
-      <origin xyz="0.13577 0.0 0.04314" rpy="0.0 0.0 0.0" />
-      <axis xyz="0 0 -1" />
-      <limit effort="30" lower="${-M_PI}" upper="${M_PI}" velocity="${M_PI/2.0}" />
-    </joint>
-    <link name="${prefix}_roll_link">
-      <visual>
-        <origin xyz="-0.001 0 -0.0005" rpy="0.0 0.0 0.0" />
-        <geometry>
-          <mesh filename="package://sobit_education_description/meshes/Manipulator_X4_Joint2_fix.dae" />
+          <mesh filename="package://sobit_education_description/meshes/arm/arm_base.stl" scale="0.001 0.001 0.001" />
         </geometry>
       </visual>
@@ -48,16 +27,16 @@
       </inertial>
     </link>
-    <joint name="${prefix}_flex_joint_rgt" type="revolute">
-      <parent link="${prefix}_roll_link" />
-      <child link="${prefix}_flex_link" />
-      <origin xyz="0.0 0.0 0.0407" rpy="0.0 0.0 0.0" />
-      <axis xyz="0 -1 0" />
-      <limit effort="30" lower="${-M_PI/2.0}" upper="${M_PI/2.0}" velocity="${M_PI/2.0}" />
+    <joint name="${prefix}_shoulder_pan_joint" type="revolute">
+      <parent link="${prefix}_base_link" />
+      <child link="${prefix}_shoulder_pan_link" />
+      <origin xyz="0.0 0.00875 0.043" rpy="0.0 0.0 0.0" />
+      <axis xyz="0 0 -1" />
+      <limit effort="30" lower="${-M_PI}" upper="${M_PI}" velocity="${M_PI/2.0}" />
     </joint>
-    <link name="${prefix}_flex_link">
+    <link name="${prefix}_shoulder_pan_link">
       <visual>
-        <origin xyz="0 0.00025 0.0" rpy="0.0 0.0 0.0" />
+        <origin xyz="0.0 0 0.0" rpy="0.0 0.0 ${M_PI/2.0}" />
         <geometry>
-          <mesh filename="package://sobit_education_description/meshes/Manipulator_X4_Joint3_fix.dae" />
+          <mesh filename="package://sobit_education_description/meshes/arm/arm_rotate.stl" scale="0.001 0.001 0.001" />
         </geometry>
       </visual>
@@ -70,33 +49,91 @@
       </inertial>
     </link>
-    <joint name="${prefix}_flex_joint_lft" type="revolute">
-      <parent link="${prefix}_roll_link" />
-      <child link="${prefix}_flex_link_rgt_lft" />
-      <origin xyz="0.0 0.0 0.0" rpy="0 0 ${M_PI}" />
+    <joint name="${prefix}_shoulder_1_tilt_joint" type="revolute">
+      <parent link="${prefix}_shoulder_pan_link" />
+      <child link="${prefix}_shoulder_1_tilt_link" />
+      <origin xyz="0.0 0.0 0.0405" rpy="0 0 ${M_PI}" />
       <axis xyz="0 -1 0" />
       <limit effort="30" lower="${-M_PI/2.0}" upper="${M_PI/2.0}" velocity="${M_PI/2.0}" />
     </joint>
-    <link name="${prefix}_flex_link_rgt_lft">
+    <link name="${prefix}_shoulder_1_tilt_link">
       <origin xyz="0.0 0.0 0.0" rpy="0.0 0.0 0.0" />
     </link>
-    <joint name="elbow_flex_joint_rgt" type="revolute">
-      <parent link="${prefix}_flex_link" />
-      <child link="elbow_flex_link" />
-      <origin xyz="0.0235 0.0 0.148" rpy="0.0 0.0 0.0" />
+    <joint name="${prefix}_shoulder_2_tilt_joint" type="revolute">
+      <parent link="${prefix}_shoulder_pan_link" />
+      <child link="${prefix}_shoulder_2_tilt_link" />
+      <origin xyz="0.0 0.0 0.0405" rpy="0.0 0.0 0.0" />
+      <axis xyz="0 -1 0" />
+      <limit effort="30" lower="${-M_PI/2.0}" upper="${M_PI/2.0}" velocity="${M_PI/2.0}" />
+    </joint>
+    <link name="${prefix}_shoulder_2_tilt_link">
+      <visual>
+        <origin xyz="0 0.0 0.0" rpy="0.0 0.0 ${M_PI/2.0}" />
+        <geometry>
+          <mesh filename="package://sobit_education_description/meshes/arm/arm_upper.stl" scale="0.001 0.001 0.001" />
+        </geometry>
+      </visual>
+      <inertial>
+        <origin xyz="0.0 0.0 0.0" rpy="0.0 0.0 0.0" />
+        <mass value="0.08" />
+        <inertia ixx="1.0" ixy="0.0" ixz="0.0"
+                 iyy="1.0" iyz="0.0"
+                 izz="1.0" />
+      </inertial>
+    </link>
+    <joint name="${prefix}_elbow_1_tilt_joint" type="revolute">
+      <parent link="${prefix}_shoulder_2_tilt_link" />
+      <child link="${prefix}_elbow_1_tilt_link" />
+      <origin xyz="0.02538 0.0 0.148" rpy="0 0 ${M_PI}" />
       <axis xyz="0 -1 0" />
       <limit effort="30" lower="${-M_PI/2.0}" upper="1.4155" velocity="${M_PI/2.0}" />
     </joint>
-    <link name="elbow_flex_link" />
-    <joint name="elbow_flex_joint_lft" type="revolute">
-      <parent link="${prefix}_flex_link" />
-      <child link="elbow_flex_link_rgt_lft" />
-      <origin xyz="0.0 0.0 0.0" rpy="0 0 ${M_PI}" />
+    <link name="${prefix}_elbow_1_tilt_link">
+      <origin xyz="0.0 0.0 0.0" rpy="0.0 0.0 0.0" />
+    </link>
+    <joint name="${prefix}_elbow_2_tilt_joint" type="revolute">
+      <parent link="${prefix}_shoulder_2_tilt_link" />
+      <child link="${prefix}_elbow_2_tilt_link" />
+      <origin xyz="0.02538 0.0 0.148" rpy="0.0 0.0 0.0" />
       <axis xyz="0 -1 0" />
       <limit effort="30" lower="${-M_PI/2.0}" upper="1.4155" velocity="${M_PI/2.0}" />
     </joint>
-    <link name="elbow_flex_link_rgt_lft">
-      <origin xyz="0.0 0.0 0.0" rpy="0.0 0.0 0.0" />
+    <link name="${prefix}_elbow_2_tilt_link">
+      <visual>
+        <origin xyz="0.0 0.0 0.0" rpy="0.0 0.0 ${M_PI/2.0}" />
+        <geometry>
+          <mesh filename="package://sobit_education_description/meshes/arm/arm_lower.stl" scale="0.001 0.001 0.001" />
+        </geometry>
+      </visual>
+      <inertial>
+        <origin xyz="0.0 0.0 0.0" rpy="0.0 0.0 0.0" />
+        <mass value="0.08" />
+        <inertia ixx="1.0" ixy="0.0" ixz="0.0"
+                 iyy="1.0" iyz="0.0"
+                 izz="1.0" />
+      </inertial>
     </link>
-    <joint name="wrist_flex_dummy_joint" type="fixed">
+    <joint name="${prefix}_wrist_tilt_joint" type="revolute">
+      <parent link="${prefix}_elbow_2_tilt_link" />
+      <child link="${prefix}_wrist_tilt_link" />
+      <origin xyz="0.0 0.0 0.150019" rpy="0.0 0.0 0.0" />
+      <axis xyz="0 -1 0" />
+      <limit effort="30" lower="${-M_PI/2.0}" upper="1.4155" velocity="${M_PI/2.0}" />
+    </joint>
+    <link name="${prefix}_wrist_tilt_link">
+      <!-- <visual>
+        <origin xyz="0.0 0.0 0.0" rpy="0.0 0.0 ${M_PI/2.0}" />
+        <geometry>
+          <mesh filename="package://sobit_education_description/meshes/hand/hand_back.stl" scale="0.001 0.001 0.001" />
+        </geometry>
+      </visual>
+      <inertial>
+        <origin xyz="0.0 0.0 0.0" rpy="0.0 0.0 0.0" />
+        <mass value="0.08" />
+        <inertia ixx="1.0" ixy="0.0" ixz="0.0"
+                 iyy="1.0" iyz="0.0"
+                 izz="1.0" />
+      </inertial> -->
+    </link>
+    <!-- <joint name="wrist_flex_dummy_joint" type="fixed">
       <parent link="elbow_flex_link" />
       <child link="wrist_flex_dummy_link" />
@@ -141,6 +178,5 @@
                  izz="1.0" />
       </inertial>
-    </link>
-    <xacro:arm_transmission prefix="${prefix}" />
+    </link> -->
   </xacro:macro>
 </robot>

File: sobit_education_description/urdf/hand/hand.urdf.xacro (robot description, xacro)
@@ -1,35 +1,20 @@
 <?xml version="1.0" encoding="UTF-8" ?>
-<robot name="hand"
-  xmlns:xacro="http://ros.org/wiki/xacro">
-  <xacro:include filename="$(find sobit_education_description)/urdf/hand/hand.transmission.xacro" />
-  <xacro:macro name="hand" params="prefix parent">
-    <joint name="${prefix}_dummy_joint" type="fixed">
+<!-- check! https://answers.ros.org/question/11807/two-joints-for-one-link/ -->
+<robot name="hand" xmlns:xacro="http://ros.org/wiki/xacro">
+  <!-- <xacro:include filename="$(find sobit_education_description)/urdf/hand/hand.transmission.xacro" /> -->
+  <xacro:macro name="hand" params="prefix_hand prefix_finger parent">
+    <!-- <xacro:hand_transmission prefix="${prefix_hand}"/> -->
+    <joint name="${prefix_hand}_base_joint" type="revolute">
       <parent link="${parent}" />
-      <child link="${prefix}_dummy_link" />
+      <child link="${prefix_hand}_base_link" />
       <origin xyz="0.0 0.0 0.0" rpy="0.0 0.0 0.0" />
-      <axis xyz="0 1 0" />
-      <limit effort="30" lower="${-M_PI/2.0}" upper="${M_PI/2.0}" velocity="${M_PI/2.0}" />
+      <axis xyz="0 0 1" />
+      <limit lower="-1.570796327" upper="0" effort="1" velocity="1"/>
     </joint>
-    <link name="${prefix}_dummy_link" />
-    <joint name="${prefix}_joint" type="revolute">
-      <parent link="${prefix}_dummy_link" />
-      <child link="${prefix}_link" />
-      <axis xyz="1 0 0" />
-      <limit lower="0.0" upper="${M_PI/2.0}" effort="1" velocity="1" />
-    </joint>
-    <link name="${prefix}_link" />
-    <joint name="${prefix}_l_joint" type="revolute">
-      <parent link="${prefix}_dummy_link" />
-      <child link="${prefix}_inner_l_joint" />
-      <origin xyz="0.0455 0.0165 0.0" rpy="0.0 0.0 0.0" />
-      <axis xyz="0 0 1" />
-      <limit lower="${-M_PI/2.0}" upper="0.0" effort="1" velocity="1" />
-      <mimic joint="${prefix}_joint" multiplier="1.0" offset="-0.1" />
-    </joint>
-    <link name="${prefix}_inner_l_joint">
+    <link name="${prefix_hand}_base_link">
       <visual>
-        <origin xyz="0.04 -0.017 0.0015" rpy="0.0 0.0 0.0" />
+        <origin xyz="0.0 0.0 0.0" rpy="0.0 0.0 ${M_PI/2.0}" />
         <geometry>
-          <mesh filename="package://sobit_education_description/meshes/sobit_edu_hand.dae" />
+          <mesh filename="package://sobit_education_description/meshes/hand/hand_back.stl" scale="0.001 0.001 0.001" />
         </geometry>
       </visual>
@@ -42,36 +27,101 @@
       </inertial>
     </link>
-    <joint name="${prefix}_inner_r_joint" type="revolute">
-      <parent link="${prefix}_dummy_link" />
-      <child link="${prefix}_inner_r_link" />
-      <origin xyz="0.0455 -0.0165 0.0" rpy="0.0 0.0 0.0" />
-      <axis xyz="0 0 1" />
-      <limit lower="0" upper="${M_PI/2.0}" effort="1" velocity="1" />
-      <mimic joint="${prefix}_joint" multiplier="-1.0" offset="0.1" />
+    <joint name="${prefix_hand}_inner_l_joint" type="revolute">
+      <!-- <parent link="${parent}" /> -->
+      <parent link="${prefix_hand}_base_link" />
+      <child link="${prefix_hand}_inner_l_link" />
+      <origin xyz="-0.028 0.0150335 0.077436" rpy="0.0 0.0 0.0" />
+      <axis xyz="0 0 -1" />
+      <limit lower="-1.570796327" upper="0" effort="1" velocity="1"/>
+      <!-- <mimic joint="${prefix_hand}_joint" multiplier="-1.0" offset="0"/> -->
     </joint>
-    <link name="${prefix}_inner_r_link">
+    <link name="${prefix_hand}_inner_l_link">
       <visual>
-        <origin xyz="0.04 0.017 -0.005" rpy="${M_PI} 0 0" />
+        <origin xyz="0.0 0.0 0.0" rpy="${M_PI/2.0} 0.0 ${M_PI/2.0}" />
         <geometry>
-          <mesh filename="package://sobit_education_description/meshes/sobit_edu_hand.dae" />
+          <mesh filename="package://sobit_education_description/meshes/hand/hand_link_inner_l.stl" scale="0.001 0.001 0.001" />
         </geometry>
       </visual>
-      <inertial>
-        <origin xyz="0.0 0.0 0.0" rpy="0 0 ${M_PI}" />
-        <mass value="0.08" />
-        <inertia ixx="1.0" ixy="0.0" ixz="0.0"
-                 iyy="1.0" iyz="0.0"
-                 izz="1.0" />
-      </inertial>
     </link>
-    <joint name="${prefix}_center_joint" type="fixed">
+    <joint name="${prefix_hand}_inner_r_joint" type="revolute">
       <parent link="${parent}" />
-      <child link="${prefix}_center_link" />
-      <origin xyz="0.15 0.0 0.0" rpy="0.0 0.0 0.0" />
-      <axis xyz="0 1 0" />
-      <limit effort="30" lower="${-M_PI/2.0}" upper="${M_PI/2.0}" velocity="${M_PI/2.0}" />
+      <child link="${prefix_hand}_inner_r_link" />
+      <origin xyz="-0.028 -0.0150335 0.077436" rpy="0.0 0.0 0.0" />
+      <axis xyz="0 0 -1" />
+      <limit lower="-1.570796327" upper="0" effort="1" velocity="1"/>
+      <!-- <mimic joint="${prefix_hand}_joint" multiplier="1.0" offset="0"/> -->
     </joint>
-    <link name="${prefix}_center_link" />
-    <xacro:hand_transmission prefix="${prefix}" />
+    <link name="${prefix_hand}_inner_r_link">
+      <visual>
+        <origin xyz="0.0 0.0 0.0" rpy="${M_PI/2.0} 0.0 ${M_PI/2.0}" />
+        <geometry>
+          <mesh filename="package://sobit_education_description/meshes/hand/hand_link_inner_r.stl" scale="0.001 0.001 0.001" />
+        </geometry>
+      </visual>
+    </link>
+    <joint name="${prefix_hand}_outer_l_joint" type="revolute">
+      <parent link="${parent}" />
+      <child link="${prefix_hand}_outer_l_link" />
+      <origin xyz="-0.028 0.04 0.059065" rpy="0.0 0.0 0.0" />
+      <axis xyz="0 0 1" />
+      <limit lower="-1.570796327" upper="0" effort="1" velocity="1"/>
+      <!-- <mimic joint="${prefix_hand}_joint" multiplier="-1.12" offset="0"/> -->
+    </joint>
+    <link name="${prefix_hand}_outer_l_link">
+      <visual>
+        <origin xyz="0.0 0.0 0.0" rpy="${M_PI/2.0} 0.0 ${M_PI/2.0}" />
+        <geometry>
+          <mesh filename="package://sobit_education_description/meshes/hand/hand_link_outer_l.stl" scale="0.001 0.001 0.001" />
+        </geometry>
+      </visual>
+    </link>
+    <joint name="${prefix_hand}_outer_r_joint" type="revolute">
+      <parent link="${parent}" />
+      <child link="${prefix_hand}_outer_r_link" />
+      <origin xyz="-0.028 -0.04 0.059065" rpy="0.0 0.0 0.0" />
+      <axis xyz="0 0 1" />
+      <limit lower="-1.570796327" upper="0" effort="1" velocity="1"/>
+      <!-- <mimic joint="${prefix_hand}_joint" multiplier="1.12" offset="0"/> -->
+    </joint>
+    <link name="${prefix_hand}_outer_r_link">
+      <visual>
+        <origin xyz="0.0 0.0 0.0" rpy="${M_PI/2.0} 0.0 ${M_PI/2.0}" />
+        <geometry>
+          <mesh filename="package://sobit_education_description/meshes/hand/hand_link_outer_r.stl" scale="0.001 0.001 0.001" />
+        </geometry>
+      </visual>
+    </link>
+    <joint name="${prefix_hand}_${prefix_finger}_l_joint" type="revolute">
+      <parent link="${prefix_hand}_outer_l_link" />
+      <child link="${prefix_hand}_${prefix_finger}_l_link" />
+      <origin xyz="0.019 0.0 0.070114" rpy="0.0 0.0 0.0" />
+      <axis xyz="0 0 1" />
+      <limit lower="-1.570796327" upper="0" effort="1" velocity="1"/>
+      <!-- <mimic joint="${prefix_hand}_joint" multiplier="0.84" offset="0"/> -->
+    </joint>
+    <link name="${prefix_hand}_${prefix_finger}_l_link">
+      <visual>
+        <origin xyz="0.0 0.0 0.0" rpy="${M_PI/2.0} 0.0 ${M_PI/2.0}" />
+        <geometry>
+          <mesh filename="package://sobit_education_description/meshes/hand/hand_finger_l.stl" scale="0.001 0.001 0.001" />
+        </geometry>
+      </visual>
+    </link>
+    <joint name="${prefix_hand}_${prefix_finger}_r_joint" type="revolute">
+      <parent link="${prefix_hand}_outer_r_link" />
+      <child link="${prefix_hand}_${prefix_finger}_r_link" />
+      <origin xyz="0.019 0.0 0.070114" rpy="0.0 0.0 0.0" />
+      <axis xyz="0 0 1" />
+      <limit lower="-1.570796327" upper="0" effort="1" velocity="1"/>
+      <!-- <mimic joint="${prefix_hand}_joint" multiplier="-0.84" offset="0"/> -->
+    </joint>
+    <link name="${prefix_hand}_${prefix_finger}_r_link">
+      <visual>
+        <origin xyz="0.0 0.0 0.0" rpy="${M_PI/2.0} 0.0 ${M_PI/2.0}" />
+        <geometry>
+          <mesh filename="package://sobit_education_description/meshes/hand/hand_finger_r.stl" scale="0.001 0.001 0.001" />
+        </geometry>
+      </visual>
+    </link>
   </xacro:macro>
 </robot>
