Commit message: update urdf and transmission (hand & arm)

File: sobit_education_description/urdf/arm/arm.urdf.xacro (robot description, xacro)
@@ -65,17 +65,9 @@
       <parent link="${prefix}_shoulder_pan_link" />
       <child link="${prefix}_shoulder_1_tilt_link" />
-      <origin xyz="0.0 0.0 0.0405" rpy="0 0 ${M_PI}" />
-      <axis xyz="0 -1 0" />
+      <origin xyz="0.0 0.0 0.0405" rpy="0.0 0.0 0.0" />
+      <axis xyz="0 1 0" />
       <limit effort="30" lower="${-M_PI/2.0}" upper="${M_PI/2.0}" velocity="${M_PI/2.0}" />
     </joint>
-    <link name="${prefix}_shoulder_1_tilt_link" />
-    <joint name="${prefix}_shoulder_2_tilt_joint" type="revolute">
-      <parent link="${prefix}_shoulder_pan_link" />
-      <child link="${prefix}_shoulder_2_tilt_link" />
-      <origin xyz="0.0 0.0 0.0405" rpy="0.0 0.0 0.0" />
-      <axis xyz="0 -1 0" />
-      <limit effort="30" lower="${-M_PI/2.0}" upper="${M_PI/2.0}" velocity="${M_PI/2.0}" />
-    </joint>
-    <link name="${prefix}_shoulder_2_tilt_link">
+    <link name="${prefix}_shoulder_1_tilt_link">
       <visual>
         <origin xyz="0 0.0 0.0" rpy="0.0 0.0 ${M_PI/2.0}" />
@@ -99,20 +91,20 @@
       </inertial>
     </link>
+    <joint name="${prefix}_shoulder_2_tilt_joint" type="revolute">
+      <parent link="${prefix}_shoulder_pan_link" />
+      <child link="${prefix}_shoulder_2_tilt_link" />
+      <origin xyz="0.0 0.0 0.0405" rpy="0.0 0.0 ${M_PI}" />
+      <axis xyz="0 -1 0" />
+      <limit effort="30" lower="${-M_PI/2.0}" upper="${M_PI/2.0}" velocity="${M_PI/2.0}" />
+    </joint>
+    <link name="${prefix}_shoulder_2_tilt_link" />
     <joint name="${prefix}_elbow_1_tilt_joint" type="revolute">
-      <parent link="${prefix}_shoulder_2_tilt_link" />
+      <parent link="${prefix}_shoulder_1_tilt_link" />
       <child link="${prefix}_elbow_1_tilt_link" />
-      <origin xyz="0.02538 0.0 0.148" rpy="0 0 ${M_PI}" />
-      <axis xyz="0 -1 0" />
+      <origin xyz="0.02538 0.0 0.148" rpy="0.0 0.0 0.0" />
+      <axis xyz="0 1 0" />
       <limit effort="30" lower="${-M_PI/2.0}" upper="1.4155" velocity="${M_PI/2.0}" />
     </joint>
-    <link name="${prefix}_elbow_1_tilt_link" />
-    <joint name="${prefix}_elbow_2_tilt_joint" type="revolute">
-      <parent link="${prefix}_shoulder_2_tilt_link" />
-      <child link="${prefix}_elbow_2_tilt_link" />
-      <origin xyz="0.02538 0.0 0.148" rpy="0.0 0.0 0.0" />
-      <axis xyz="0 -1 0" />
-      <limit effort="30" lower="${-M_PI/2.0}" upper="1.4155" velocity="${M_PI/2.0}" />
-    </joint>
-    <link name="${prefix}_elbow_2_tilt_link">
+    <link name="${prefix}_elbow_1_tilt_link">
       <visual>
         <origin xyz="0.0 0.0 0.0" rpy="0.0 0.0 ${M_PI/2.0}" />
@@ -129,5 +121,5 @@
       </collision>
       <inertial>
-        <origin xyz="0.0 0.0 0.0" rpy="0.0 0.0 0.0" />
+        <origin xyz="0.0 0.0 0.0" rpy="0.0 0.0 ${M_PI/2.0}" />
         <mass value="0.08" />
         <inertia ixx="1.0" ixy="0.0" ixz="0.0"
@@ -136,9 +128,17 @@
       </inertial>
     </link>
+    <joint name="${prefix}_elbow_2_tilt_joint" type="revolute">
+      <parent link="${prefix}_shoulder_1_tilt_link" />
+      <child link="${prefix}_elbow_2_tilt_link" />
+      <origin xyz="0.02538 0.0 0.148" rpy="0.0 0.0 ${M_PI}" />
+      <axis xyz="0 -1 0" />
+      <limit effort="30" lower="${-M_PI/2.0}" upper="1.4155" velocity="${M_PI/2.0}" />
+    </joint>
+    <link name="${prefix}_elbow_2_tilt_link" />
     <joint name="${prefix}_wrist_tilt_joint" type="revolute">
-      <parent link="${prefix}_elbow_2_tilt_link" />
+      <parent link="${prefix}_elbow_1_tilt_link" />
       <child link="${prefix}_wrist_tilt_link" />
       <origin xyz="0.0 0.0 0.150019" rpy="0.0 0.0 0.0" />
-      <axis xyz="0 -1 0" />
+      <axis xyz="0 1 0" />
       <limit effort="30" lower="${-M_PI/2.0}" upper="1.4155" velocity="${M_PI/2.0}" />
     </joint>

File: sobit_education_description/urdf/hand/hand.transmission.xacro (robot description, xacro)
@@ -1,6 +1,11 @@
 <?xml version="1.0" ?>
 <robot xmlns:xacro="http://ros.org/wiki/xacro">
-  <xacro:macro name="hand_transmission" params="prefix">
-    <position_joint_transmission joint="${prefix}_base_joint" reduction="1" />
+  <xacro:macro name="hand_transmission" params="prefix_hand prefix_finger">
+    <position_joint_transmission joint="${prefix_hand}_inner_l_joint" reduction="1" />
+    <position_joint_transmission joint="${prefix_hand}_inner_r_joint" reduction="1" />
+    <position_joint_transmission joint="${prefix_hand}_outer_l_joint" reduction="1" />
+    <position_joint_transmission joint="${prefix_hand}_outer_r_joint" reduction="1" />
+    <position_joint_transmission joint="${prefix_hand}_${prefix_finger}_l_joint" reduction="1" />
+    <position_joint_transmission joint="${prefix_hand}_${prefix_finger}_r_joint" reduction="1" />
   </xacro:macro>
 </robot>

File: sobit_education_description/urdf/hand/hand.urdf.xacro (robot description, xacro)
@@ -4,6 +4,6 @@
   <xacro:include filename="$(find sobit_education_description)/urdf/hand/hand.transmission.xacro" />
   <xacro:macro name="hand" params="prefix_hand prefix_finger parent">
-    <xacro:hand_transmission prefix="${prefix_hand}" />
-    <joint name="${prefix_hand}_base_joint" type="revolute">
+    <xacro:hand_transmission prefix_hand="${prefix_hand}" prefix_finger="${prefix_finger}" />
+    <joint name="${prefix_hand}_base_joint" type="fixed">
       <parent link="${parent}" />
       <child link="${prefix_hand}_base_link" />
@@ -38,5 +38,5 @@
       <child link="${prefix_hand}_inner_l_link" />
       <origin xyz="-0.028 0.0150335 0.077436" rpy="0.0 0.0 0.0" />
-      <axis xyz="0 0 -1" />
+      <axis xyz="1 0 0" />
       <limit lower="-1.570796327" upper="0" effort="1" velocity="1" />
       <!-- <mimic joint="${prefix_hand}_joint" multiplier="-1.0" offset="0" /> -->
@@ -68,5 +68,6 @@
       <child link="${prefix_hand}_inner_r_link" />
       <origin xyz="-0.028 -0.0150335 0.077436" rpy="0.0 0.0 0.0" />
-      <axis xyz="0 0 -1" />
+      <axis xyz="-1 0 0" />
+      <mimic joint="${prefix_hand}_inner_l_joint" multiplier="1" offset="0" />
       <limit lower="-1.570796327" upper="0" effort="1" velocity="1" />
       <!-- <mimic joint="${prefix_hand}_joint" multiplier="1.0" offset="0" /> -->
@@ -98,5 +99,6 @@
       <child link="${prefix_hand}_outer_l_link" />
       <origin xyz="-0.028 0.04 0.059065" rpy="0.0 0.0 0.0" />
-      <axis xyz="0 0 1" />
+      <axis xyz="1 0 0" />
+      <mimic joint="${prefix_hand}_inner_l_joint" multiplier="1" offset="0" />
       <limit lower="-1.570796327" upper="0" effort="1" velocity="1" />
       <!-- <mimic joint="${prefix_hand}_joint" multiplier="-1.12" offset="0" /> -->
@@ -128,5 +130,6 @@
       <child link="${prefix_hand}_outer_r_link" />
       <origin xyz="-0.028 -0.04 0.059065" rpy="0.0 0.0 0.0" />
-      <axis xyz="0 0 1" />
+      <axis xyz="-1 0 0" />
+      <mimic joint="${prefix_hand}_inner_l_joint" multiplier="1" offset="0" />
       <limit lower="-1.570796327" upper="0" effort="1" velocity="1" />
       <!-- <mimic joint="${prefix_hand}_joint" multiplier="1.12" offset="0" /> -->
@@ -158,5 +161,6 @@
       <child link="${prefix_hand}_${prefix_finger}_l_link" />
       <origin xyz="0.019 0.0 0.070114" rpy="0.0 0.0 0.0" />
-      <axis xyz="0 0 1" />
+      <axis xyz="1 0 0" />
+      <mimic joint="${prefix_hand}_inner_l_joint" multiplier="-1" offset="0" />
       <limit lower="-1.570796327" upper="0" effort="1" velocity="1" />
       <!-- <mimic joint="${prefix_hand}_joint" multiplier="0.84" offset="0" /> -->
@@ -188,5 +192,6 @@
       <child link="${prefix_hand}_${prefix_finger}_r_link" />
       <origin xyz="0.019 0.0 0.070114" rpy="0.0 0.0 0.0" />
-      <axis xyz="0 0 1" />
+      <axis xyz="-1 0 0" />
+      <mimic joint="${prefix_hand}_inner_l_joint" multiplier="-1" offset="0" />
       <limit lower="-1.570796327" upper="0" effort="1" velocity="1" />
       <!-- <mimic joint="${prefix_hand}_joint" multiplier="-0.84" offset="0" /> -->

Commit message: update joint & transmission

File: sobit_education_description/urdf/arm/arm.urdf.xacro (robot description, xacro)
@@ -8,6 +8,4 @@
       <child link="${prefix}_base_link" />
       <origin xyz="0.123481 0.0 0.00325" rpy="0.0 0.0 0.0" />
-      <axis xyz="0 0 1" />
-      <limit effort="30" lower="${-M_PI}" upper="${M_PI}" velocity="${M_PI/2.0}" />
     </joint>
     <link name="${prefix}_base_link">
@@ -37,5 +35,5 @@
       <child link="${prefix}_shoulder_pan_link" />
       <origin xyz="0.008769 0.0 0.043" rpy="0.0 0.0 0.0" />
-      <axis xyz="0 0 -1" />
+      <axis xyz="0 0 1" />
       <limit effort="30" lower="${-M_PI}" upper="${M_PI}" velocity="${M_PI/2.0}" />
     </joint>
@@ -66,5 +64,5 @@
       <child link="${prefix}_shoulder_1_tilt_link" />
       <origin xyz="0.0 0.0 0.0405" rpy="0.0 0.0 0.0" />
-      <axis xyz="0 1 0" />
+      <axis xyz="0 -1 0" />
       <limit effort="30" lower="${-M_PI/2.0}" upper="${M_PI/2.0}" velocity="${M_PI/2.0}" />
     </joint>
@@ -95,5 +93,6 @@
       <child link="${prefix}_shoulder_2_tilt_link" />
       <origin xyz="0.0 0.0 0.0405" rpy="0.0 0.0 ${M_PI}" />
-      <axis xyz="0 -1 0" />
+      <axis xyz="0 1 0" />
+      <mimic joint="${prefix}_shoulder_1_tilt_joint" multiplier="1" offset="0" />
       <limit effort="30" lower="${-M_PI/2.0}" upper="${M_PI/2.0}" velocity="${M_PI/2.0}" />
     </joint>
@@ -102,7 +101,7 @@
       <parent link="${prefix}_shoulder_1_tilt_link" />
       <child link="${prefix}_elbow_1_tilt_link" />
-      <origin xyz="0.02538 0.0 0.148" rpy="0.0 0.0 0.0" />
-      <axis xyz="0 1 0" />
-      <limit effort="30" lower="${-M_PI/2.0}" upper="1.4155" velocity="${M_PI/2.0}" />
+      <origin xyz="0.02538 0.0 0.148" rpy="0.0 ${M_PI/2.0} 0.0" />
+      <axis xyz="0 -1 0" />
+      <limit effort="30" lower="${-M_PI/2.0}" upper="${M_PI/2.0}" velocity="${M_PI/2.0}" />
     </joint>
     <link name="${prefix}_elbow_1_tilt_link">
@@ -132,6 +131,7 @@
       <child link="${prefix}_elbow_2_tilt_link" />
       <origin xyz="0.02538 0.0 0.148" rpy="0.0 0.0 ${M_PI}" />
-      <axis xyz="0 -1 0" />
-      <limit effort="30" lower="${-M_PI/2.0}" upper="1.4155" velocity="${M_PI/2.0}" />
+      <axis xyz="0 1 0" />
+      <mimic joint="${prefix}_elbow_1_tilt_joint" multiplier="1" offset="0" />
+      <limit effort="30" lower="${-M_PI/2.0}" upper="${M_PI/2.0}" velocity="${M_PI/2.0}" />
     </joint>
     <link name="${prefix}_elbow_2_tilt_link" />

File: sobit_education_description/urdf/back/back.urdf.xacro (robot description, xacro)
@@ -6,6 +6,4 @@
       <child link="${prefix}_base_link"/>
       <origin xyz="-0.070405 0.0 0.00325" rpy="0.0 0.0 0.0" />
-      <axis xyz="0 0 1"/>
-      <limit effort="30" lower="${-M_PI}" upper="${M_PI}" velocity="${M_PI/2.0}"/>
     </joint>
     <link name="${prefix}_base_link">

File: sobit_education_description/urdf/body/cover.urdf.xacro (robot description, xacro)
@@ -6,5 +6,4 @@
       <parent link="${parent}" />
       <child link="${prefix}_link" />
-      <axis xyz="0 0 1 "/>
     </joint>
     <link name="${prefix}_link">

File: sobit_education_description/urdf/hand/hand.transmission.xacro (robot description, xacro)
@@ -2,4 +2,5 @@
 <robot xmlns:xacro="http://ros.org/wiki/xacro">
   <xacro:macro name="hand_transmission" params="prefix_hand prefix_finger">
+    <position_joint_transmission joint="${prefix_hand}_joint" reduction="1" />
     <position_joint_transmission joint="${prefix_hand}_inner_l_joint" reduction="1" />
     <position_joint_transmission joint="${prefix_hand}_inner_r_joint" reduction="1" />

File: sobit_education_description/urdf/hand/hand.urdf.xacro (robot description, xacro)
@@ -9,6 +9,4 @@
       <child link="${prefix_hand}_base_link" />
       <origin xyz="0.0 0.0 0.0" rpy="0.0 0.0 0.0" />
-      <axis xyz="0 0 1" />
-      <limit lower="-1.570796327" upper="0" effort="1" velocity="1" />
     </joint>
     <link name="${prefix_hand}_base_link">
@@ -34,4 +32,12 @@
       </inertial>
     </link>
+    <joint name="${prefix_hand}_joint" type="revolute">
+      <parent link="${prefix_hand}_base_link" />
+      <child link="${prefix_hand}_link" />
+      <origin xyz="-0.028 -0.0150335 0.077436" rpy="0.0 0.0 0.0" />
+      <axis xyz="-1 0 0" />
+      <limit lower="${-M_PI/2.0}" upper="0" effort="1" velocity="1" />
+    </joint>
+    <link name="${prefix_hand}_link" />
     <joint name="${prefix_hand}_inner_l_joint" type="revolute">
       <parent link="${prefix_hand}_base_link" />
@@ -39,6 +45,6 @@
       <origin xyz="-0.028 0.0150335 0.077436" rpy="0.0 0.0 0.0" />
       <axis xyz="1 0 0" />
-      <limit lower="-1.570796327" upper="0" effort="1" velocity="1" />
-      <!-- <mimic joint="${prefix_hand}_joint" multiplier="-1.0" offset="0" /> -->
+      <mimic joint="${prefix_hand}_joint" multiplier="1.0" offset="0" />
+      <limit lower="${-M_PI/2.0}" upper="0" effort="1" velocity="1" />
     </joint>
     <link name="${prefix_hand}_inner_l_link">
@@ -70,6 +76,5 @@
       <axis xyz="-1 0 0" />
       <mimic joint="${prefix_hand}_inner_l_joint" multiplier="1" offset="0" />
-      <limit lower="-1.570796327" upper="0" effort="1" velocity="1" />
-      <!-- <mimic joint="${prefix_hand}_joint" multiplier="1.0" offset="0" /> -->
+      <limit lower="${-M_PI/2.0}" upper="0" effort="1" velocity="1" />
     </joint>
     <link name="${prefix_hand}_inner_r_link">
@@ -101,5 +106,5 @@
       <axis xyz="1 0 0" />
       <mimic joint="${prefix_hand}_inner_l_joint" multiplier="1" offset="0" />
-      <limit lower="-1.570796327" upper="0" effort="1" velocity="1" />
+      <limit lower="${-M_PI/2.0}" upper="0" effort="1" velocity="1" />
       <!-- <mimic joint="${prefix_hand}_joint" multiplier="-1.12" offset="0" /> -->
     </joint>
@@ -132,5 +137,5 @@
       <axis xyz="-1 0 0" />
       <mimic joint="${prefix_hand}_inner_l_joint" multiplier="1" offset="0" />
-      <limit lower="-1.570796327" upper="0" effort="1" velocity="1" />
+      <limit lower="${-M_PI/2.0}" upper="0" effort="1" velocity="1" />
       <!-- <mimic joint="${prefix_hand}_joint" multiplier="1.12" offset="0" /> -->
     </joint>
@@ -161,7 +166,7 @@
       <child link="${prefix_hand}_${prefix_finger}_l_link" />
       <origin xyz="0.019 0.0 0.070114" rpy="0.0 0.0 0.0" />
-      <axis xyz="1 0 0" />
-      <mimic joint="${prefix_hand}_inner_l_joint" multiplier="-1" offset="0" />
-      <limit lower="-1.570796327" upper="0" effort="1" velocity="1" />
+      <axis xyz="-1 0 0" />
+      <mimic joint="${prefix_hand}_inner_l_joint" multiplier="1" offset="0" />
+      <limit lower="${-M_PI/2.0}" upper="0" effort="1" velocity="1" />
       <!-- <mimic joint="${prefix_hand}_joint" multiplier="0.84" offset="0" /> -->
     </joint>
@@ -192,7 +197,7 @@
       <child link="${prefix_hand}_${prefix_finger}_r_link" />
       <origin xyz="0.019 0.0 0.070114" rpy="0.0 0.0 0.0" />
-      <axis xyz="-1 0 0" />
-      <mimic joint="${prefix_hand}_inner_l_joint" multiplier="-1" offset="0" />
-      <limit lower="-1.570796327" upper="0" effort="1" velocity="1" />
+      <axis xyz="1 0 0" />
+      <mimic joint="${prefix_hand}_inner_l_joint" multiplier="1" offset="0" />
+      <limit lower="${-M_PI/2.0}" upper="0" effort="1" velocity="1" />
       <!-- <mimic joint="${prefix_hand}_joint" multiplier="-0.84" offset="0" /> -->
     </joint>

File: sobit_education_description/urdf/head/head.transmission.xacro (robot description, xacro)
@@ -2,6 +2,6 @@
 <robot xmlns:xacro="http://ros.org/wiki/xacro">
   <xacro:macro name="xtion_motor_transmission" params="prefix">
-    <position_joint_transmission joint="${prefix}_pan_joint" reduction="1" />
-    <position_joint_transmission joint="${prefix}_tilt_joint" reduction="1" />
+    <position_joint_transmission joint="${prefix}_camera_pan_joint" reduction="1" />
+    <position_joint_transmission joint="${prefix}_camera_tilt_joint" reduction="1" />
   </xacro:macro>
 </robot>

File: sobit_education_description/urdf/head/head.urdf.xacro (robot description, xacro)
@@ -7,6 +7,4 @@
       <child link="${prefix}_camera_base_link" />
       <origin xyz="0.150 0.0 0.370" rpy="0.0 0.0 0.0" />
-      <axis xyz="0 0 -1" />
-      <limit effort="30" lower="${-M_PI/2.0}" upper="${M_PI/2.0}" velocity="${M_PI/2.0}" />
     </joint>
     <link name="${prefix}_camera_base_link">
@@ -94,6 +92,4 @@
       <child link="${prefix}_double_sided_tape_link" />
       <origin xyz="0.0 0.0 0.029" rpy="0.0 0.0 0.0" />
-      <axis xyz="0 0 -1" />
-      <limit effort="30" lower="${-M_PI/2.0}" upper="${M_PI/2.0}" velocity="${M_PI/2.0}" />
     </joint>
     <link name="${prefix}_double_sided_tape_link" />

File: sobit_education_description/urdf/sensor/matrix.urdf.xacro (robot description, xacro)
@@ -9,5 +9,4 @@
       <child link="${prefix}_base_link" />
       <origin xyz="0.0 0.0 0.620" rpy="0.0 0.0 0.0" />
-      <axis xyz="0 1 0" />
     </joint>
     <link name="${prefix}_base_link">
@@ -38,5 +37,4 @@
       <child link="${prefix}_board_link" />
       <origin xyz="0.0 0.0 0.0295" rpy="0.0 0.0 0.0" />
-      <axis xyz="0 1 0" />
     </joint>
     <link name="${prefix}_board_link">

File: sobit_education_description/urdf/sensor/mic.urdf.xacro (robot description, xacro)
@@ -7,5 +7,4 @@
       <child link="${prefix}_base_link" />
       <origin xyz="0.190 0.0 0.610" rpy="0.0 0.0 0.0" />
-      <axis xyz="0 1 0" />
     </joint>
     <link name="${prefix}_base_link">
@@ -36,5 +35,4 @@
       <child link="mic" />
       <origin xyz="-0.017007 0.0 0.020" rpy="0.0 0.0 0.0" />
-      <axis xyz="0 1 0" />
     </joint>
     <link name="mic">

File: sobit_education_description/urdf/sensor/urg.urdf.xacro (robot description, xacro)
@@ -6,6 +6,4 @@
       <parent link="${parent}" />
       <child link="${prefix}_base_link" />
-      <axis xyz="0 0 1" />
-      <limit effort="30" lower="-3.14" upper="3.14" velocity="1.571" />
     </joint>
     <link name="${prefix}_base_link">

Commit message: update urdf

File: sobit_education_description/urdf/arm/arm.urdf.xacro (robot description, xacro)
@@ -140,5 +140,5 @@
       <child link="${prefix}_wrist_tilt_link" />
       <origin xyz="0.0 0.0 0.150019" rpy="0.0 0.0 0.0" />
-      <axis xyz="0 1 0" />
+      <axis xyz="0 -1 0" />
       <limit effort="30" lower="${-M_PI/2.0}" upper="1.4155" velocity="${M_PI/2.0}" />
     </joint>

File: sobit_education_description/urdf/hand/hand.urdf.xacro (robot description, xacro)
@@ -1,4 +1,3 @@
 <?xml version="1.0" encoding="UTF-8" ?>
-<!-- check! https://answers.ros.org/question/11807/two-joints-for-one-link/ -->
 <robot name="hand" xmlns:xacro="http://ros.org/wiki/xacro">
   <xacro:include filename="$(find sobit_education_description)/urdf/hand/hand.transmission.xacro" />
@@ -71,9 +70,9 @@
     </link>
     <joint name="${prefix_hand}_inner_r_joint" type="revolute">
-      <parent link="${parent}" />
+      <parent link="${prefix_hand}_base_link" />
       <child link="${prefix_hand}_inner_r_link" />
       <origin xyz="-0.028 -0.0150335 0.077436" rpy="0.0 0.0 0.0" />
       <axis xyz="-1 0 0" />
-      <mimic joint="${prefix_hand}_inner_l_joint" multiplier="1" offset="0" />
+      <mimic joint="${prefix_hand}_joint" multiplier="1.0" offset="0" />
       <limit lower="${-M_PI/2.0}" upper="0" effort="1" velocity="1" />
     </joint>
@@ -101,11 +100,10 @@
     </link>
     <joint name="${prefix_hand}_outer_l_joint" type="revolute">
-      <parent link="${parent}" />
+      <parent link="${prefix_hand}_base_link" />
       <child link="${prefix_hand}_outer_l_link" />
       <origin xyz="-0.028 0.04 0.059065" rpy="0.0 0.0 0.0" />
       <axis xyz="1 0 0" />
-      <mimic joint="${prefix_hand}_inner_l_joint" multiplier="1" offset="0" />
-      <limit lower="${-M_PI/2.0}" upper="0" effort="1" velocity="1" />
-      <!-- <mimic joint="${prefix_hand}_joint" multiplier="-1.12" offset="0" /> -->
+      <mimic joint="${prefix_hand}_joint" multiplier="1.0" offset="0" />
+      <limit lower="${-M_PI/2.0}" upper="0" effort="1" velocity="1" />
     </joint>
     <link name="${prefix_hand}_outer_l_link">
@@ -132,11 +130,10 @@
     </link>
     <joint name="${prefix_hand}_outer_r_joint" type="revolute">
-      <parent link="${parent}" />
+      <parent link="${prefix_hand}_base_link" />
       <child link="${prefix_hand}_outer_r_link" />
       <origin xyz="-0.028 -0.04 0.059065" rpy="0.0 0.0 0.0" />
       <axis xyz="-1 0 0" />
-      <mimic joint="${prefix_hand}_inner_l_joint" multiplier="1" offset="0" />
-      <limit lower="${-M_PI/2.0}" upper="0" effort="1" velocity="1" />
-      <!-- <mimic joint="${prefix_hand}_joint" multiplier="1.12" offset="0" /> -->
+      <mimic joint="${prefix_hand}_joint" multiplier="1.0" offset="0" />
+      <limit lower="${-M_PI/2.0}" upper="0" effort="1" velocity="1" />
     </joint>
     <link name="${prefix_hand}_outer_r_link">
@@ -167,7 +164,6 @@
       <origin xyz="0.019 0.0 0.070114" rpy="0.0 0.0 0.0" />
       <axis xyz="-1 0 0" />
-      <mimic joint="${prefix_hand}_inner_l_joint" multiplier="1" offset="0" />
-      <limit lower="${-M_PI/2.0}" upper="0" effort="1" velocity="1" />
-      <!-- <mimic joint="${prefix_hand}_joint" multiplier="0.84" offset="0" /> -->
+      <mimic joint="${prefix_hand}_joint" multiplier="1.0" offset="0" />
+      <limit lower="${-M_PI/2.0}" upper="0" effort="1" velocity="1" />
     </joint>
     <link name="${prefix_hand}_${prefix_finger}_l_link">
@@ -198,7 +194,6 @@
       <origin xyz="0.019 0.0 0.070114" rpy="0.0 0.0 0.0" />
       <axis xyz="1 0 0" />
-      <mimic joint="${prefix_hand}_inner_l_joint" multiplier="1" offset="0" />
-      <limit lower="${-M_PI/2.0}" upper="0" effort="1" velocity="1" />
-      <!-- <mimic joint="${prefix_hand}_joint" multiplier="-0.84" offset="0" /> -->
+      <mimic joint="${prefix_hand}_joint" multiplier="1.0" offset="0" />
+      <limit lower="${-M_PI/2.0}" upper="0" effort="1" velocity="1" />
     </joint>
     <link name="${prefix_hand}_${prefix_finger}_r_link">

File: sobit_education_description/urdf/head/head.urdf.xacro (robot description, xacro)
@@ -34,5 +34,5 @@
       <child link="${prefix}_camera_pan_link" />
       <origin xyz="0.04125 0.0 0.0255" rpy="0.0 0.0 0.0" />
-      <axis xyz="0 0 -1" />
+      <axis xyz="0 0 1" />
       <limit effort="30" lower="${-M_PI/2.0}" upper="${M_PI/2.0}" velocity="${M_PI/2.0}" />
     </joint>
@@ -63,5 +63,5 @@
       <child link="${prefix}_camera_tilt_link" />
       <origin xyz="0.0 0.0 0.0435" rpy="0.0 0.0 0.0" />
-      <axis xyz="0 0 -1" />
+      <axis xyz="0 1 0" />
       <limit effort="30" lower="${-M_PI/2.0}" upper="${M_PI/2.0}" velocity="${M_PI/2.0}" />
     </joint>
