Commit message: update base urdf

File: sobit_education_description/urdf/base/base.urdf.xacro (robot description, xacro)
@@ -6,6 +6,5 @@
       kobuki_description/launch/view_model.launch
  -->
-<robot name="base"
-  xmlns:xacro="http://ros.org/wiki/xacro">
+<robot name="base" xmlns:xacro="http://ros.org/wiki/xacro">
   <xacro:include filename="$(find kobuki_description)/urdf/common_properties.urdf.xacro" />
   <xacro:include filename="$(find kobuki_description)/urdf/kobuki_gazebo.urdf.xacro" />
@@ -44,6 +43,5 @@
         <!-- COM experimentally determined -->
         <origin xyz="0.01 0 0" />
-        <mass value="2.4" />
-        <!-- 2.4/2.6 kg for small/big battery pack -->
+        <mass value="2.4" /> <!-- 2.4/2.6 kg for small/big battery pack -->
         <!-- Kobuki's inertia tensor is approximated by a cylinder with homogeneous mass distribution
              More details: http://en.wikipedia.org/wiki/List_of_moment_of_inertia_tensors
@@ -53,14 +51,16 @@
              izz = 1/2 * m * r^2
           -->
-        <inertia ixx="0.019995" ixy="0.0" ixz="0.0" iyy="0.019995" iyz="0.0" izz="0.03675" />
-      </inertial>
-    </link>
-    <joint name="wheel_left_joint" type="continuous">
-      <parent link="base_link" />
-      <child link="wheel_left_link" />
+        <inertia ixx="0.019995" ixy="0.0" ixz="0.0"
+                 iyy="0.019995" iyz="0.0"
+                 izz="0.03675" />
+      </inertial>
+    </link>
+    <joint name="wheel_l_joint" type="continuous">
+      <parent link="base_link" />
+      <child link="wheel_l_link" />
       <origin xyz="0.00 ${0.23/2} 0.0250" rpy="${-M_PI/2} 0 0" />
       <axis xyz="0 0 1" />
     </joint>
-    <link name="wheel_left_link">
+    <link name="wheel_l_link">
       <visual>
         <geometry>
@@ -71,21 +71,23 @@
       <collision>
         <geometry>
-          <cylinder length="0.0206" radius="0.0352" />
-        </geometry>
-        <origin rpy="0 0 0" xyz="0 0 0" />
-      </collision>
-      <inertial>
-        <mass value="0.01" />
-        <origin xyz="0 0 0" />
-        <inertia ixx="0.001" ixy="0.0" ixz="0.0" iyy="0.001" iyz="0.0" izz="0.001" />
-      </inertial>
-    </link>
-    <joint name="wheel_right_joint" type="continuous">
-      <parent link="base_link" />
-      <child link="wheel_right_link" />
+          <cylinder length="0.0206" radius="0.035" />
+        </geometry>
+        <origin rpy="0 0 0" xyz="0 0 0" />
+      </collision>
+      <inertial>
+        <mass value="0.01" />
+        <origin xyz="0 0 0" />
+        <inertia ixx="0.001" ixy="0.0" ixz="0.0"
+                 iyy="0.001" iyz="0.0"
+                 izz="0.001" />
+      </inertial>
+    </link>
+    <joint name="wheel_r_joint" type="continuous">
+      <parent link="base_link" />
+      <child link="wheel_r_link" />
       <origin xyz="0.00 -${0.23/2} 0.0250" rpy="${-M_PI/2} 0 0" />
       <axis xyz="0 0 1" />
     </joint>
-    <link name="wheel_right_link">
+    <link name="wheel_r_link">
       <visual>
         <geometry>
@@ -96,20 +98,22 @@
       <collision>
         <geometry>
-          <cylinder length="0.0206" radius="0.0350" />
-        </geometry>
-        <origin rpy="0 0 0" xyz="0 0 0" />
-      </collision>
-      <inertial>
-        <mass value="0.01" />
-        <origin xyz="0 0 0" />
-        <inertia ixx="0.001" ixy="0.0" ixz="0.0" iyy="0.001" iyz="0.0" izz="0.001" />
-      </inertial>
-    </link>
-    <joint name="caster_front_joint" type="fixed">
-      <parent link="base_link" />
-      <child link="caster_front_link" />
+          <cylinder length="0.0206" radius="0.035" />
+        </geometry>
+        <origin rpy="0 0 0" xyz="0 0 0" />
+      </collision>
+      <inertial>
+        <mass value="0.01" />
+        <origin xyz="0 0 0" />
+        <inertia ixx="0.001" ixy="0.0" ixz="0.0"
+                 iyy="0.001" iyz="0.0"
+                 izz="0.001" />
+      </inertial>
+    </link>
+    <joint name="caster_f_joint" type="fixed">
+      <parent link="base_link" />
+      <child link="caster_f_link" />
       <origin xyz="0.115 0.0 0.007" rpy="${-M_PI/2} 0 0" />
     </joint>
-    <link name="caster_front_link">
+    <link name="caster_f_link">
       <collision>
         <geometry>
@@ -121,13 +125,15 @@
         <mass value="0.01" />
         <origin xyz="0 0 0" />
-        <inertia ixx="0.001" ixy="0.0" ixz="0.0" iyy="0.001" iyz="0.0" izz="0.001" />
-      </inertial>
-    </link>
-    <joint name="caster_back_joint" type="fixed">
-      <parent link="base_link" />
-      <child link="caster_back_link" />
+        <inertia ixx="0.001" ixy="0.0" ixz="0.0"
+                 iyy="0.001" iyz="0.0"
+                 izz="0.001" />
+      </inertial>
+    </link>
+    <joint name="caster_b_joint" type="fixed">
+      <parent link="base_link" />
+      <child link="caster_b_link" />
       <origin xyz="-0.135 0.0 0.009" rpy="${-M_PI/2} 0 0" />
     </joint>
-    <link name="caster_back_link">
+    <link name="caster_b_link">
       <collision>
         <geometry>
@@ -139,5 +145,7 @@
         <mass value="0.01" />
         <origin xyz="0 0 0" />
-        <inertia ixx="0.001" ixy="0.0" ixz="0.0" iyy="0.001" iyz="0.0" izz="0.001" />
+        <inertia ixx="0.001" ixy="0.0" ixz="0.0"
+                 iyy="0.001" iyz="0.0"
+                 izz="0.001" />
       </inertial>
     </link>
@@ -153,43 +161,53 @@
         <mass value="0.001" />
         <origin xyz="0 0 0" rpy="0 0 0" />
-        <inertia ixx="0.0001" ixy="0" ixz="0" iyy="0.000001" iyz="0" izz="0.0001" />
-      </inertial>
-    </link>
-    <joint name="cliff_sensor_left_joint" type="fixed">
+        <inertia ixx="0.0001" ixy="0" ixz="0"
+                 iyy="0.000001" iyz="0"
+                 izz="0.0001" />
+      </inertial>
+    </link>
+    <joint name="cliff_sensor_l_joint" type="fixed">
       <origin xyz="0.08734 0.13601 0.0214" rpy="0 ${M_PI/2} 0" />
       <parent link="base_link" />
-      <child link="cliff_sensor_left_link" />
-    </joint>
-    <link name="cliff_sensor_left_link">
+      <child link="cliff_sensor_l_link" />
+    </joint>
+    <link name="cliff_sensor_l_link">
       <inertial>
         <mass value="0.0001" />
         <origin xyz="0 0 0" />
-        <inertia ixx="0.0001" ixy="0.0" ixz="0.0" iyy="0.0001" iyz="0.0" izz="0.0001" />
-      </inertial>
-    </link>
-    <joint name="cliff_sensor_right_joint" type="fixed">
+        <inertia ixx="0.0001" ixy="0.0" ixz="0.0"
+                 iyy="0.0001" iyz="0.0"
+                 izz="0.0001" />
+      </inertial>
+    </link>
+    <joint name="cliff_sensor_r_joint" type="fixed">
       <origin xyz="0.085 -0.13601 0.0214" rpy="0 ${M_PI/2} 0" />
       <parent link="base_link" />
-      <child link="cliff_sensor_right_link" />
-    </joint>
-    <link name="cliff_sensor_right_link">
+      <child link="cliff_sensor_r_link" />
+    </joint>
+    <link name="cliff_sensor_r_link">
       <inertial>
         <mass value="0.0001" />
         <origin xyz="0 0 0" />
-        <inertia ixx="0.0001" ixy="0.0" ixz="0.0" iyy="0.0001" iyz="0.0" izz="0.0001" />
-      </inertial>
-    </link>
-    <joint name="cliff_sensor_front_joint" type="fixed">
+        <inertia ixx="0.0001" ixy="0.0" ixz="0.0"
+                 iyy="0.0001" iyz="0.0"
+                 izz="0.0001" />
+      </inertial>
+    </link>
+    <joint name="cliff_sensor_f_joint" type="fixed">
       <origin xyz="0.156 0.00 0.0214" rpy="0 ${M_PI/2} 0" />
       <parent link="base_link" />
-      <child link="cliff_sensor_front_link" />
-    </joint>
-    <link name="cliff_sensor_front_link">
+      <child link="cliff_sensor_f_link" />
+    </joint>
+    <link name="cliff_sensor_f_link">
       <inertial>
         <mass value="0.0001" />
         <origin xyz="0 0 0" />
-        <inertia ixx="0.0001" ixy="0.0" ixz="0.0" iyy="0.0001" iyz="0.0" izz="0.0001" />
-      </inertial>
-    </link>
+        <inertia ixx="0.0001" ixy="0.0" ixz="0.0"
+                 iyy="0.0001" iyz="0.0"
+                 izz="0.0001" />
+      </inertial>
+    </link>
+    <!-- Kobuki Gazebo simulation details -->
+    <!-- <xacro:kobuki_sim/> -->
   </xacro:macro>
 </robot>
