Commit message: update link/joint name

File: sobit_education_description/urdf/hand/hand.urdf.xacro (robot description, xacro)
@@ -5,69 +5,73 @@
   <xacro:macro name="hand" params="prefix parent">
     <joint name="${prefix}_dummy_joint" type="fixed">
-      <parent link="${parent}"/>
-      <child link="${prefix}_dummy_link"/>
-      <origin rpy="0 0 0" xyz="0.0 0.0 0.0"/>
-      <axis xyz="0 1 0"/>
-      <limit effort="30" lower="${-M_PI/2.0}" upper="${M_PI/2.0}" velocity="${M_PI/2.0}"/>
+      <parent link="${parent}" />
+      <child link="${prefix}_dummy_link" />
+      <origin xyz="0.0 0.0 0.0" rpy="0.0 0.0 0.0" />
+      <axis xyz="0 1 0" />
+      <limit effort="30" lower="${-M_PI/2.0}" upper="${M_PI/2.0}" velocity="${M_PI/2.0}" />
     </joint>
-    <link name="${prefix}_dummy_link"/>
+    <link name="${prefix}_dummy_link" />
     <joint name="${prefix}_joint" type="revolute">
-      <parent link="${prefix}_dummy_link"/>
-      <child link="${prefix}_link"/>
+      <parent link="${prefix}_dummy_link" />
+      <child link="${prefix}_link" />
       <axis xyz="1 0 0" />
       <limit lower="0.0" upper="${M_PI/2.0}" effort="1" velocity="1" />
     </joint>
-    <link name="${prefix}_link"/>
+    <link name="${prefix}_link" />
     <joint name="${prefix}_l_joint" type="revolute">
-      <parent link="${prefix}_dummy_link"/>
-      <child link="${prefix}_l_link"/>
-      <origin rpy="0 0 0" xyz="0.0455 0.0165 0.0"/>
+      <parent link="${prefix}_dummy_link" />
+      <child link="${prefix}_inner_l_joint" />
+      <origin xyz="0.0455 0.0165 0.0" rpy="0.0 0.0 0.0" />
       <axis xyz="0 0 1" />
       <limit lower="${-M_PI/2.0}" upper="0.0" effort="1" velocity="1" />
-      <mimic joint="${prefix}_joint" multiplier="1.0" offset="-0.1"/>
+      <mimic joint="${prefix}_joint" multiplier="1.0" offset="-0.1" />
     </joint>
-    <link name="${prefix}_l_link">
+    <link name="${prefix}_inner_l_joint">
       <visual>
-        <origin rpy="0 0 0" xyz="0.04 -0.017 0.0015"/>
+        <origin xyz="0.04 -0.017 0.0015" rpy="0.0 0.0 0.0" />
         <geometry>
-          <mesh filename="package://sobit_education_description/meshes/sobit_edu_hand.dae"/>
+          <mesh filename="package://sobit_education_description/meshes/sobit_edu_hand.dae" />
         </geometry>
       </visual>
       <inertial>
-        <origin rpy="0 0 0" xyz="0 0 0"/>
-        <mass value="0.08"/>
-        <inertia ixx="1.0" ixy="0.0" ixz="0.0" iyy="1.0" iyz="0.0" izz="1.0"/>
+        <origin xyz="0.0 0.0 0.0" rpy="0.0 0.0 0.0" />
+        <mass value="0.08" />
+        <inertia ixx="1.0" ixy="0.0" ixz="0.0"
+                 iyy="1.0" iyz="0.0"
+                 izz="1.0" />
       </inertial>
     </link>
-    <joint name="${prefix}_r_joint" type="revolute">
-      <parent link="${prefix}_dummy_link"/>
-      <child link="${prefix}_r_link"/>
-      <origin rpy="0 0 0" xyz="0.0455 -0.0165 0.0"/>
+    <joint name="${prefix}_inner_r_joint" type="revolute">
+      <parent link="${prefix}_dummy_link" />
+      <child link="${prefix}_inner_r_link" />
+      <origin xyz="0.0455 -0.0165 0.0" rpy="0.0 0.0 0.0" />
       <axis xyz="0 0 1" />
       <limit lower="0" upper="${M_PI/2.0}" effort="1" velocity="1" />
-      <mimic joint="${prefix}_joint" multiplier="-1.0" offset="0.1"/>
+      <mimic joint="${prefix}_joint" multiplier="-1.0" offset="0.1" />
     </joint>
-    <link name="${prefix}_r_link">
+    <link name="${prefix}_inner_r_link">
       <visual>
-        <origin rpy="${M_PI} 0 0" xyz="0.04 0.017 -0.005"/>
+        <origin xyz="0.04 0.017 -0.005" rpy="${M_PI} 0 0" />
         <geometry>
-          <mesh filename="package://sobit_education_description/meshes/sobit_edu_hand.dae"/>
+          <mesh filename="package://sobit_education_description/meshes/sobit_edu_hand.dae" />
         </geometry>
       </visual>
       <inertial>
-        <origin rpy="0 0 ${M_PI}" xyz="0 0 0"/>
-        <mass value="0.08"/>
-        <inertia ixx="1.0" ixy="0.0" ixz="0.0" iyy="1.0" iyz="0.0" izz="1.0"/>
+        <origin xyz="0.0 0.0 0.0" rpy="0 0 ${M_PI}" />
+        <mass value="0.08" />
+        <inertia ixx="1.0" ixy="0.0" ixz="0.0"
+                 iyy="1.0" iyz="0.0"
+                 izz="1.0" />
       </inertial>
     </link>
     <joint name="${prefix}_center_joint" type="fixed">
-      <parent link="${parent}"/>
-      <child link="${prefix}_center_link"/>
-      <origin rpy="0 0 0" xyz="0.15 0.0 0.0"/>
-      <axis xyz="0 1 0"/>
-      <limit effort="30" lower="${-M_PI/2.0}" upper="${M_PI/2.0}" velocity="${M_PI/2.0}"/>
+      <parent link="${parent}" />
+      <child link="${prefix}_center_link" />
+      <origin xyz="0.15 0.0 0.0" rpy="0.0 0.0 0.0" />
+      <axis xyz="0 1 0" />
+      <limit effort="30" lower="${-M_PI/2.0}" upper="${M_PI/2.0}" velocity="${M_PI/2.0}" />
     </joint>
-    <link name="${prefix}_center_link"/>
-    <xacro:hand_transmission prefix="${prefix}"/>
+    <link name="${prefix}_center_link" />
+    <xacro:hand_transmission prefix="${prefix}" />
   </xacro:macro>
 </robot>
