Commit message: update colors

File: sobit_education_description/urdf/materials.urdf.xacro (robot description, xacro)
@@ -17,5 +17,11 @@
   </material>
   <material name="white">
-    <color rgba="1.0 1.0 1.0 1.0"/>
+    <color rgba="1.0 1.0 1.0 1.0" />
+  </material>
+  <material name="grey">
+    <color rgba="0.3 0.3 0.3 1.0" />
+  </material>
+  <material name="dark_grey">
+    <color rgba="0.175 0.175 0.175 1.0" />
   </material>
 </robot>
