Commit message: update collision

File: sobit_education_description/urdf/body/cover.urdf.xacro (robot description, xacro)
@@ -17,5 +17,5 @@
       </visual>
       <collision>
-        <origin xyz="0.0 0.0 0.0" rpy="0.0 0.0 0.0" />
+        <origin xyz="0.0 0.0 0.0" rpy="0.0 ${M_PI/2.0} ${-M_PI/2.0}" />
         <geometry>
           <mesh filename="package://sobit_education_description/meshes/body/cover.stl" scale="0.001 0.001 0.001" />
