Commit message: remove arm hand head gazebo and fix base gazebo

File: sobit_edu_description/urdf/base/base.urdf.xacro (robot description, xacro)
@@ -54,5 +54,5 @@
       </inertial>
     </link>
-    <joint name="wheel_l_joint" type="fixed">
+    <joint name="wheel_l_joint" type="continuous">
       <parent link="base_link" />
       <child link="wheel_l_link" />
@@ -81,5 +81,5 @@
       </inertial>
     </link>
-    <joint name="wheel_r_joint" type="fixed">
+    <joint name="wheel_r_joint" type="continuous">
       <parent link="base_link" />
       <child link="wheel_r_link" />
@@ -198,49 +198,4 @@
       </inertial>
     </link>
-    <gazebo reference="base_link">
-	  <selfCollide>true</selfCollide>
-      <mu1>1.0</mu1>
-      <mu2>1.0</mu2>
-    </gazebo>
-    <gazebo reference="caster_front_link">
-	  <selfCollide>true</selfCollide>
-      <mu1>0.0</mu1>
-      <mu2>0.0</mu2>
-    </gazebo>
-    <gazebo reference="caster_back_link">
-	  <selfCollide>true</selfCollide>
-      <mu1>0.0</mu1>
-      <mu2>0.0</mu2>
-    </gazebo>
-    <gazebo reference="wheel_l_link">
-	  <selfCollide>true</selfCollide>
-      <mu1>1.0</mu1>
-      <mu2>1.0</mu2>
-    </gazebo>
-    <gazebo reference="wheel_r_link">
-	  <selfCollide>true</selfCollide>
-      <mu1>1.0</mu1>
-      <mu2>1.0</mu2>
-    </gazebo>
-    <gazebo>
-      <plugin name="differential_drive_controller" filename="libgazebo_ros_diff_drive.so">
-        <leftJoint>wheel_l_joint</leftJoint>
-        <rightJoint>wheel_r_joint</rightJoint>
-        <wheelSeparation>0.23</wheelSeparation>
-        <wheelDiameter>0.070</wheelDiameter>
-        <wheelAcceleration>1.0</wheelAcceleration>
-        <wheelTorque>20</wheelTorque>
-        <commandTopic>/mobile_base/commands/velocity</commandTopic>
-        <odometryTopic>odom</odometryTopic>
-        <odometryFrame>odom</odometryFrame>
-        <robotBaseFrame>base_footprint</robotBaseFrame>
-        <odometrySource>1</odometrySource>
-        <publishWheelTF>true</publishWheelTF>
-        <publishOdom>true</publishOdom>
-        <publishWheelJointState>true</publishWheelJointState>
-        <legacyMode>false</legacyMode>
-        <updateRate>50.0</updateRate>
-      </plugin>
-    </gazebo>
   </xacro:macro>
 </robot>
