Commit message: ADD meshes of xtion

File: sobit_edu_description/urdf/sensor/xtion.urdf.xacro (robot description, xacro)
@@ -40,5 +40,5 @@
         <!-- <origin xyz="0.0025 0.0265 0.004" rpy="0 0 0"/> -->
         <geometry>
-          <mesh filename="file://$(find sobit_pro_description)/meshes/sensor/xtion/xtion_pro_camera.dae"/>
+          <mesh filename="file://$(find sobit_edu_description)/meshes/sensor/xtion/xtion_pro_camera.dae"/>
         </geometry>
       </visual>
