Commit message: FIX lidar_frame

File: sobit_edu_description/urdf/gazebo.urdf.xacro (robot description, xacro)
@@ -5,9 +5,9 @@
     <!-- Sensor: LiDAR -->
     <xacro:if value="${enable_gz_lidar}">
-      <gazebo reference="sim_laser_frame">
+      <gazebo reference="lidar_laser">
         <sensor name="lidar" type="gpu_lidar">
           <pose>0 0 0 0 0 0</pose>
-          <ignition_frame_id>${robot_name}/sim_laser_frame</ignition_frame_id>
-          <!-- <gz_frame_id>${robot_name}/sim_laser_frame</gz_frame_id> -->
+          <ignition_frame_id>${robot_name}/lidar_laser</ignition_frame_id>
+          <!-- <gz_frame_id>${robot_name}/lidar_laser</gz_frame_id> -->
           <topic>${robot_name}/scan</topic>
           <always_on>1</always_on>

File: sobit_edu_description/urdf/sensor/lidar.urdf.xacro (robot description, xacro)
@@ -31,5 +31,5 @@
       </inertial>
     </link>
-    <joint name="${prefix}_sim_joint" type="fixed">
+    <!-- <joint name="${prefix}_sim_joint" type="fixed">
       <parent link="${prefix}_base_link" />
       <child link="sim_laser_frame" />
@@ -44,5 +44,5 @@
                  izz="0.001" />
       </inertial>
-    </link>
+    </link> -->
     <xacro:hokuyo_ust_mount prefix="${prefix}" parent="${prefix}_base_link" topic="scan" >
       <origin xyz="0.1105 0.0 0.0" rpy="0.0 0.0 0.0" />
