Commit message: Update setup of install.sh and tiny changes

File: sobit_edu_description/urdf/arm/arm.urdf.xacro (robot description, xacro)
@@ -147,5 +147,5 @@
       <child link="${prefix}_wrist_tilt_link" />
       <origin xyz="0.149873  0.0 0.0" rpy="${M_PI/2.0} 0.0 ${M_PI/2.0}" />
-      <axis xyz="0 -1 0" />
+      <axis xyz="0 1 0" />
       <limit effort="30" lower="${-M_PI/2.0}" upper="1.4155" velocity="${M_PI/2.0}" />
     </joint>

Commit message: CHANGE urdf of arm

File: sobit_edu_description/urdf/arm/arm.urdf.xacro (robot description, xacro)
@@ -1,156 +1,314 @@
 <?xml version="1.0" encoding="UTF-8" ?>
+<!-- OpenManipulator X1000 (Arm) -->
 <robot name="arm" xmlns:xacro="http://ros.org/wiki/xacro">
   <xacro:include filename="$(find sobit_edu_description)/urdf/arm/arm.transmission.xacro" />
-  <xacro:include filename="$(find sobit_edu_description)/urdf/arm/arm.gazebo.xacro" />
   <xacro:macro name="arm" params="prefix parent">
+    <!-- Joint: Platform -->
+    <joint name="${prefix}_platform_joint" type="fixed">
+      <parent link="${parent}"/>
+      <child link="${prefix}_platform_link"/>
+      <origin xyz="0.122 0.0 0.0115" rpy="0 0 0"/>
+    </joint>
+    <!-- Link: Platform -->
+    <link name="${prefix}_platform_link">
+      <visual>
+        <origin xyz="0 0 0" rpy="0 0 ${M_PI/2}"/>
+        <geometry>
+          <mesh filename="file://$(find sobit_edu_description)/meshes/arm/omx1_link_base.stl" scale="0.001 0.001 0.001"/>
+        </geometry>
+        <material name="black"/>
+      </visual>
+      <collision>
+        <origin xyz="${0.005-0.1/2} 0.0 ${-0.0156+0.0686/2}" rpy="0 0 0"/>
+        <geometry>
+          <box size="0.1000 0.1200 0.0686"/>
+        </geometry>
+      </collision>
+      <inertial>
+        <origin xyz="${0.005-0.1/2} 0.0 ${-0.0156+0.0686/2}" rpy="0 0 0"/>
+        <mass value="0.336" />
+        <inertia  ixx="${1/12*0.336*(0.1000**2+0.0686**2)}" ixy="0.0" ixz="0.0"
+                  iyy="${1/12*0.336*(0.1200**2+0.0686**2)}" iyz="0.0"
+                  izz="${1/12*0.336*(0.1000**2+0.1200**2)}" />
+      </inertial>
+    </link>
+    <!-- Joint: Base -->
     <joint name="${prefix}_base_joint" type="fixed">
-      <parent link="${parent}" />
-      <child link="${prefix}_base_link" />
-      <origin xyz="0.123481 0.0 0.00325" rpy="0.0 0.0 0.0" />
-      <!-- <origin xyz="0.0 0.0 0.0" rpy="0.0 0.0 0.0" /> -->
-    </joint>
+      <parent link="${prefix}_platform_link"/>
+      <child link="${prefix}_base_link"/>
+      <origin xyz="-0.02925 0.0 0.022" rpy="0 ${-M_PI/2} ${M_PI}"/>
+      <!-- <origin xyz="${-0.0112-0.016/2} 0.0 0.008" rpy="0 0 0"/> -->
+    </joint>
+    <!-- Link: Base -->
     <link name="${prefix}_base_link">
       <visual>
-        <origin xyz="0.0 0.0 0.0" rpy="0.0 0.0 ${M_PI/2.0}" />
-        <geometry>
-          <mesh filename="file://$(find sobit_edu_description)/meshes/arm/arm_base.stl" scale="0.001 0.001 0.001" />
-        </geometry>
-        <material name="black" />
-      </visual>
-      <collision>
-        <!-- <origin xyz="0.0 0.01 0.0237" rpy="0.0 0.0 ${M_PI/2.0}" /> -->
-        <origin xyz="0.0 0.0 0.0" rpy="0.0 0.0 ${M_PI/2.0}" />
-        <geometry>
-          <!-- <box size="0.06 0.06 0.0474"/> -->
-          <mesh filename="file://$(find sobit_edu_description)/meshes/arm/arm_base.stl" scale="0.001 0.001 0.001" />
-        </geometry>
-      </collision>
-      <inertial>
-        <origin xyz="0.0 0.01 0.0237" rpy="0.0 0.0 0.0" />
-        <mass value="0.011" />
-        <inertia ixx="${1/12*0.011*(0.0474**2+0.06**2)}"  ixy="0.0" ixz="0.0"
-                 iyy="${1/12*0.011*(0.06**2+0.0474**2)}"  iyz="0.0"
-                 izz="${1/12*0.011*(0.06**2+0.06**2)}" />
-      </inertial>
-    </link>
-    <joint name="${prefix}_shoulder_pan_joint" type="revolute">
-      <parent link="${prefix}_base_link" />
-      <child link="${prefix}_shoulder_pan_link" />
-      <origin xyz="0.008769 0.0 0.043" rpy="0.0 0.0 0.0" />
-      <axis xyz="0 0 1" />
-      <limit effort="30" lower="${-M_PI}" upper="${M_PI}" velocity="${M_PI/2.0}" />
-    </joint>
-    <link name="${prefix}_shoulder_pan_link">
-      <visual>
-        <origin xyz="0.0 0.0 0.0" rpy="0.0 0.0 ${M_PI/2.0}" />
-        <geometry>
-          <mesh filename="file://$(find sobit_edu_description)/meshes/arm/arm_lower.stl" scale="0.001 0.001 0.001" />
-        </geometry>
-        <material name="black" />
-      </visual>
-      <collision>
-        <!-- <origin xyz="0.0 0.0 0.025875" rpy="0.0 0.0 ${M_PI/2.0}" /> -->
-        <origin xyz="0.0 0.0 0.0" rpy="0.0 0.0 ${M_PI/2.0}" />
-        <geometry>
-          <!-- <box size="0.117 0.0285 0.05175"/> -->
-          <mesh filename="file://$(find sobit_edu_description)/meshes/arm/arm_lower.stl" scale="0.001 0.001 0.001" />
-        </geometry>
-      </collision>
-      <inertial>
-        <origin xyz="0.0 0.0 0.0" rpy="0.0 0.0 0.025875" />
-        <mass value="0.023" />
-        <inertia ixx="${1/12*0.023*(0.05175**2+0.0285**2)}"  ixy="0.0" ixz="0.0"
-                 iyy="${1/12*0.023*(0.117**2+0.05175**2)}"  iyz="0.0"
-                 izz="${1/12*0.023*(0.117**2+0.0285**2)}" />
-      </inertial>
-    </link>
-    <joint name="${prefix}_shoulder_1_tilt_joint" type="revolute">
-      <parent link="${prefix}_shoulder_pan_link" />
-      <child link="${prefix}_shoulder_1_tilt_link" />
-      <origin xyz="0.0 0.0 0.0405" rpy="0.0 ${M_PI/2.0} 0.0" />
-      <axis xyz="0 -1 0" />
-      <limit effort="30" lower="${-M_PI/2.0}" upper="${M_PI/2.0}" velocity="${M_PI/2.0}" />
-    </joint>
-    <link name="${prefix}_shoulder_1_tilt_link">
-      <visual>
-        <origin xyz="0 0.0 0.0" rpy="0.0 0.0 ${M_PI/2.0}" />
-        <geometry>
-          <mesh filename="file://$(find sobit_edu_description)/meshes/arm/arm_rotate.stl" scale="0.001 0.001 0.001" />
-        </geometry>
-        <material name="black" />
-      </visual>
-      <collision>
-        <origin xyz="0.0 0.0 0.0" rpy="0.0 0.0 ${M_PI/2.0}" />
-        <geometry>
-          <!-- <box size="0.117 0.1696 0.0475"/> -->
-          <mesh filename="file://$(find sobit_edu_description)/meshes/arm/arm_rotate.stl" scale="0.001 0.001 0.001" />
-        </geometry>
-      </collision>
-      <inertial>
-        <origin xyz="0.0 0.0 0.0" rpy="0.0 0.0 0.0" />
-        <mass value="0.0179" />
-        <inertia ixx="${1/12*0.0179*(0.0475**2+0.1696**2)}"  ixy="0.0" ixz="0.0"
-                 iyy="${1/12*0.0179*(0.117**2+0.0475**2)}"  iyz="0.0"
-                 izz="${1/12*0.0179*(0.117**2+0.1696**2)}" />
-      </inertial>
-    </link>
-    <joint name="${prefix}_shoulder_2_tilt_joint" type="revolute">
-      <parent link="${prefix}_shoulder_pan_link" />
-      <child link="${prefix}_shoulder_2_tilt_link" />
-      <origin xyz="0.0 0.0 0.0405" rpy="0.0 0.0 ${M_PI}" />
-      <axis xyz="0 -1 0" />
-      <mimic joint="${prefix}_shoulder_1_tilt_joint" multiplier="1" offset="0" />
-      <limit effort="30" lower="${-M_PI/2.0}" upper="${M_PI/2.0}" velocity="${M_PI/2.0}" />
-    </joint>
-    <link name="${prefix}_shoulder_2_tilt_link" />
-    <joint name="${prefix}_elbow_1_tilt_joint" type="revolute">
-      <parent link="${prefix}_shoulder_1_tilt_link" />
-      <child link="${prefix}_elbow_1_tilt_link" />
-      <origin xyz="-0.148139 0.0 0.021810" rpy="${M_PI/2.0} ${-M_PI/2.0} 0.0" />
-      <axis xyz="0 0 1" />
-      <limit effort="30" lower="${-M_PI/2.0}" upper="${M_PI/2.0}" velocity="${M_PI/2.0}" />
-    </joint>
-    <link name="${prefix}_elbow_1_tilt_link">
-      <visual>
-        <origin xyz="0.0 0.0 0.0" rpy="0.0 0.0 ${M_PI/2.0}" />
-        <geometry>
-          <mesh filename="file://$(find sobit_edu_description)/meshes/arm/arm_upper.stl" scale="0.001 0.001 0.001" />
-        </geometry>
-        <material name="black" />
-      </visual>
-      <collision>
-        <origin xyz="0.0 0.0 0.0" rpy="0.0 0.0 ${M_PI/2.0}" />
-        <geometry>
-          <!-- <box size="0.0285 0.16375 0.0439"/> -->
-          <mesh filename="file://$(find sobit_edu_description)/meshes/arm/arm_upper.stl" scale="0.001 0.001 0.001" />
-        </geometry>
-      </collision>
-      <inertial>
-        <origin xyz="0.0 0.0 0.0" rpy="0.0 0.0 ${M_PI/2.0}" />
-        <mass value="0.046" />
-        <inertia ixx="${1/12*0.046*(0.0475**2+0.1696**2)}"  ixy="0.0" ixz="0.0"
-                 iyy="${1/12*0.046*(0.117**2+0.0475**2)}"  iyz="0.0"
-                 izz="${1/12*0.046*(0.117**2+0.1696**2)}" />
-      </inertial>
-    </link>
-    <joint name="${prefix}_elbow_2_tilt_joint" type="revolute">
-      <parent link="${prefix}_shoulder_1_tilt_link" />
-      <child link="${prefix}_elbow_2_tilt_link" />
-      <origin xyz="0.02538 0.0 0.148" rpy="0.0 0.0 ${M_PI}" />
-      <axis xyz="0 1 0" />
-      <mimic joint="${prefix}_elbow_1_tilt_joint" multiplier="1" offset="0" />
-      <limit effort="30" lower="${-M_PI/2.0}" upper="${M_PI/2.0}" velocity="${M_PI/2.0}" />
-    </joint>
-    <link name="${prefix}_elbow_2_tilt_link" />
-    <joint name="${prefix}_wrist_tilt_joint" type="revolute">
-      <parent link="${prefix}_elbow_1_tilt_link" />
-      <child link="${prefix}_wrist_tilt_link" />
-      <origin xyz="0.149873  0.0 0.0" rpy="${M_PI/2.0} 0.0 ${M_PI/2.0}" />
-      <axis xyz="0 1 0" />
-      <limit effort="30" lower="${-M_PI/2.0}" upper="1.4155" velocity="${M_PI/2.0}" />
-    </joint>
-    <link name="${prefix}_wrist_tilt_link" />
+        <origin xyz="0 0 0" rpy="0 0 ${M_PI/2}"/>
+        <geometry>
+          <mesh filename="file://$(find sobit_edu_description)/meshes/arm/omx1_link1.stl" scale="0.001 0.001 0.001"/>
+        </geometry>
+        <material name="black"/>
+      </visual>
+      <collision>
+        <origin xyz="0.0 0.0 ${0.0585/2}" rpy="0 0 0"/>
+        <geometry>
+          <box size="0.0440 0.0335 0.0585"/>
+        </geometry>
+      </collision>
+      <inertial>
+        <origin xyz="0.0 0.0 ${0.0585/2}" rpy="0 0 0"/>
+        <mass value="0.205" />
+        <inertia  ixx="${1/12*0.205*(0.0440**2+0.0585**2)}" ixy="0.0" ixz="0.0"
+                  iyy="${1/12*0.205*(0.0335**2+0.0585**2)}" iyz="0.0"
+                  izz="${1/12*0.205*(0.0440**2+0.0335**2)}" />
+      </inertial>
+    </link>
+    <!-- Act 1: Shoulder Roll -->
+    <joint name="${prefix}_shoulder_roll_joint" type="revolute">
+      <parent link="${prefix}_base_link"/>
+      <child link="${prefix}_shoulder_roll_link"/>
+      <origin xyz="0.0268 0.0 0.0465" rpy="${M_PI} ${-M_PI/2} 0"/>
+      <axis xyz="0 0 1"/>
+      <limit velocity="4.8" effort="25" lower="${-M_PI}" upper="${M_PI}" />
+    </joint>
+    <!--  Act 1: Shoulder Roll -->
+    <link name="${prefix}_shoulder_roll_link">
+      <visual>
+        <origin xyz="0.0 0.0 0.0" rpy="0 0 ${M_PI/2}"/>
+        <geometry>
+          <mesh filename="file://$(find sobit_edu_description)/meshes/arm/omx1_link2.stl" scale="0.001 0.001 0.001"/>
+        </geometry>
+        <material name="black"/>
+      </visual>
+      <collision>
+        <origin xyz="0.0 0.0 ${0.0647/2}" rpy="0 0 0"/>
+        <geometry>
+          <box size="0.0335 0.1130 0.0647"/>
+        </geometry>
+      </collision>
+      <inertial>
+        <origin xyz="0.0 0.0 ${0.0647/2}" rpy="0 0 0"/>
+        <mass value="0.392" />
+        <inertia  ixx="${1/12*0.392*(0.0335**2+0.0647**2)}" ixy="0.0" ixz="0.0"
+                  iyy="${1/12*0.392*(0.1130**2+0.0647**2)}" iyz="0.0"
+                  izz="${1/12*0.392*(0.0335**2+0.1130**2)}" />
+      </inertial>
+    </link>
+    <!--  Act 2: Shoulder Pitch (right) -->
+    <joint name="${prefix}_shoulder_pitch_joint" type="revolute">
+      <parent link="${prefix}_shoulder_roll_link"/>
+      <child link="${prefix}_shoulder_pitch_link"/>
+      <origin xyz="0.0 0.0 0.05095" rpy="0 0 0"/>
+      <axis xyz="0 1 0"/>
+      <limit velocity="4.8" effort="25" lower="${-M_PI/2}" upper="${M_PI/2}" />
+    </joint>
+    <!--  Act 2: Shoulder Pitch (right) -->
+    <link name="${prefix}_shoulder_pitch_link">
+      <visual>
+        <origin xyz="0 0 0" rpy="0 0 ${M_PI/2}"/>
+        <geometry>
+          <mesh filename="file://$(find sobit_edu_description)/meshes/arm/omx1_link3.stl" scale="0.001 0.001 0.001"/>
+        </geometry>
+        <material name="black"/>
+      </visual>
+      <collision>
+        <origin xyz="${0.03575-0.0585/2} 0.0 ${-0.016+(0.14475+0.016)/2}" rpy="0 0 0"/>
+        <geometry>
+          <box size="0.0585 0.0440 ${0.14475+0.016}"/>
+        </geometry>
+      </collision>
+      <inertial>
+        <origin xyz="${0.03575-0.0585/2} 0.0 ${-0.016+(0.14475+0.016)/2}" rpy="0 0 0"/>
+        <mass value="0.261" />
+        <inertia  ixx="${1/12*0.261*(0.0585**2+(0.14475+0.016)**2)}" ixy="0.0" ixz="0.0"
+                  iyy="${1/12*0.261*(0.0440**2+(0.14475+0.016)**2)}" iyz="0.0"
+                  izz="${1/12*0.261*(0.0585**2+0.0440**2)}" />
+      </inertial>
+    </link>
+    <!--  Act 3: Shoulder Pitch (left) -->
+    <joint name="${prefix}_shoulder_pitch_sub_joint" type="revolute">
+      <parent link="${prefix}_shoulder_roll_link"/>
+      <child link="${prefix}_shoulder_pitch_sub_link"/>
+      <origin xyz="0.0 0.0 0.05095" rpy="0 0 0"/>
+      <axis xyz="0 1 0"/>
+      <limit velocity="4.8" effort="25" lower="${-M_PI/2}" upper="${M_PI/2}" />
+      <!-- <mimic joint="${prefix}_shoulder_pitch_joint" multiplier="-1" offset="0"/> -->
+    </joint>
+    <!--  Act 3: Shoulder Pitch (left) -->
+    <link name="${prefix}_shoulder_pitch_sub_link">
+      <!-- <visual>
+        <origin xyz="0 0 0" rpy="0 0 ${M_PI/2}"/>
+        <geometry>
+          <mesh filename="file://$(find sobit_light_description)/meshes/arm/omx1_link3.stl" scale="0.001 0.001 0.001"/>
+        </geometry>
+        <material name="black"/>
+      </visual> -->
+      <!-- <collision>
+        <origin xyz="${0.03575-0.0585/2} 0.0 ${-0.016+(0.14475+0.016)/2}" rpy="0 0 0"/>
+        <geometry>
+          <box size="0.0585 0.0440 ${0.14475+0.016}"/>
+        </geometry>
+      </collision> -->
+      <inertial>
+        <origin xyz="${0.03575-0.0585/2} 0.0 ${-0.016+(0.14475+0.016)/2}" rpy="0 0 0"/>
+        <mass value="0.261" />
+        <inertia  ixx="${1/12*0.261*(0.0585**2+(0.14475+0.016)**2)}" ixy="0.0" ixz="0.0"
+                  iyy="${1/12*0.261*(0.0440**2+(0.14475+0.016)**2)}" iyz="0.0"
+                  izz="${1/12*0.261*(0.0585**2+0.0440**2)}" />
+      </inertial>
+    </link>
+    <!--  Act 4: Elbow Pitch -->
+    <joint name="${prefix}_elbow_pitch_joint" type="revolute">
+      <parent link="${prefix}_shoulder_pitch_link"/>
+      <child link="${prefix}_elbow_pitch_link"/>
+      <origin xyz="0.022 -0.0 0.128" rpy="0 0 0"/>
+      <axis xyz="0 1 0"/>
+      <limit velocity="4.8" effort="25" lower="${-M_PI/2}" upper="${M_PI/2}" />
+    </joint>
+    <!--  Act 4: Elbow Pitch -->
+    <link name="${prefix}_elbow_pitch_link">
+      <visual>
+        <origin xyz="0 0 0" rpy="0 0 ${M_PI/2}"/>
+        <geometry>
+          <mesh filename="file://$(find sobit_edu_description)/meshes/arm/omx1_link4.stl" scale="0.001 0.001 0.001"/>
+        </geometry>
+        <material name="black"/>
+      </visual>
+      <collision>
+        <origin xyz="${0.0835-0.0860/2} 0.0 ${0.03525-0.04875/2}" rpy="0 0 0"/>
+        <geometry>
+          <box size="0.0860 0.0530 0.04875"/>
+        </geometry>
+      </collision>
+      <inertial>
+        <origin xyz="${0.0835-0.0860/2} 0.0 ${0.03525-0.04875/2}" rpy="0 0 0"/>
+        <mass value="0.157" />
+        <inertia  ixx="${1/12*0.157*(0.0860**2+0.04875**2)}" ixy="0.0" ixz="0.0"
+                  iyy="${1/12*0.157*(0.0530**2+0.04875**2)}" iyz="0.0"
+                  izz="${1/12*0.157*(0.0860**2+0.0530**2)}" />
+      </inertial>
+    </link>
+    <!--  Act 5: Forearm Roll -->
+    <joint name="${prefix}_forearm_roll_joint" type="revolute">
+      <parent link="${prefix}_elbow_pitch_link"/>
+      <child link="${prefix}_forearm_roll_link"/>
+      <origin xyz="0.0835 0.0 0.0" rpy="0 0 0"/>
+      <axis xyz="1 0 0"/>
+      <limit velocity="4.8" effort="25" lower="${-M_PI}" upper="${M_PI}" />
+    </joint>
+    <!--  Act 5: Forearm Roll -->
+    <link name="${prefix}_forearm_roll_link">
+      <visual>
+        <origin xyz="0 0 0" rpy="0 0 ${M_PI/2}"/>
+        <geometry>
+          <mesh filename="file://$(find sobit_edu_description)/meshes/arm/omx1_link5.stl" scale="0.001 0.001 0.001"/>
+        </geometry>
+        <material name="black"/>
+      </visual>
+      <collision>
+        <origin xyz="${0.05175/2} 0.0 0.0" rpy="0 0 0"/>
+        <geometry>
+          <box size="0.05175 0.03700 0.0285"/>
+        </geometry>
+      </collision>
+      <inertial>
+        <origin xyz="${0.05175/2} 0.0 0.0" rpy="0 0 0"/>
+        <mass value="0.093" />
+        <inertia  ixx="${1/12*0.093*(0.05175**2+0.0285**2)}" ixy="0.0" ixz="0.0"
+                  iyy="${1/12*0.093*(0.03700**2+0.0285**2)}" iyz="0.0"
+                  izz="${1/12*0.093*(0.05175**2+0.0370**2)}" />
+      </inertial>
+    </link>
+    <!--  Act 6: Wrist Pitch -->
+    <joint name="${prefix}_wrist_pitch_joint" type="revolute">
+      <parent link="${prefix}_forearm_roll_link"/>
+      <child link="${prefix}_wrist_pitch_link"/>
+      <origin xyz="0.0405 0.0 0.0" rpy="0 0 0"/>
+      <axis xyz="0 1 0"/>
+      <limit velocity="4.8" effort="25" lower="${-M_PI/2}" upper="${M_PI/2}" />
+    </joint>
+    <!--  Act 6: Wrist Pitch -->
+    <link name="${prefix}_wrist_pitch_link">
+      <visual>
+        <origin xyz="0 0 0" rpy="0 0 ${M_PI/2}"/>
+        <geometry>
+          <mesh filename="file://$(find sobit_edu_description)/meshes/arm/omx1_link6.stl" scale="0.001 0.001 0.001"/>
+        </geometry>
+        <material name="black"/>
+      </visual>
+      <collision>
+        <origin xyz="${0.064-0.0665/2} 0.0 ${0.03525-0.0465/2}" rpy="0 0 0"/>
+        <geometry>
+          <box size="0.0665 0.0410 0.0465"/>
+        </geometry>
+      </collision>
+      <inertial>
+        <origin xyz="${0.064-0.0665/2} 0.0 ${0.03525-0.0465/2}" rpy="0 0 0"/>
+        <mass value="0.106" />
+        <inertia  ixx="${1/12*0.106*(0.0665**2+0.0465**2)}" ixy="0.0" ixz="0.0"
+                  iyy="${1/12*0.106*(0.0410**2+0.0465**2)}" iyz="0.0"
+                  izz="${1/12*0.106*(0.0665**2+0.0410**2)}" />
+      </inertial>
+    </link>
+    <!--  Act 7: Wrist Roll -->
+    <joint name="${prefix}_wrist_roll_joint" type="revolute">
+      <parent link="${prefix}_wrist_pitch_link"/>
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