Commit message: CHANGE urdf of arm

File: sobit_edu_description/urdf/controllers.urdf.xacro (robot description, xacro)
@@ -18,19 +18,23 @@
       </hardware>
       <!-- Position Drive: Arm -->
-      <joint name="arm_shoulder_pan_joint">
-        <param name="id">10</param>
-        <command_interface name="position">
-          <param name="min">-3.141592654</param>
-          <param name="max">3.141592654</param>
-        </command_interface>
-        <command_interface name="velocity"/>
-        <state_interface name="position">
-          <param name="initial_value">0.0</param>
-        </state_interface>
-        <state_interface name="velocity"/>
-        <state_interface name="effort"/>
-      </joint>
-      <joint name="arm_shoulder_1_tilt_joint">
-        <param name="id">11</param>
+      <joint name="arm_shoulder_roll_joint">
+        <xacro:unless value="${$(arg enable_gz)}">
+          <param name="id">10</param>
+        </xacro:unless>
+        <command_interface name="position">
+          <param name="min">-3.141592654</param>
+          <param name="max">3.141592654</param>
+        </command_interface>
+        <command_interface name="velocity"/>
+        <state_interface name="position">
+          <param name="initial_value">0.0</param>
+        </state_interface>
+        <state_interface name="velocity"/>
+        <state_interface name="effort"/>
+      </joint>
+      <joint name="arm_shoulder_pitch_sub_joint">
+        <xacro:unless value="${$(arg enable_gz)}">
+          <param name="id">12</param>
+        </xacro:unless>
         <!-- <param name="mimic">arm_shoulder_pitch_joint</param>
         <param name="multiplier">-1</param> -->
@@ -48,6 +52,8 @@
         <state_interface name="effort"/>
       </joint>
-      <joint name="arm_shoulder_2_tilt_joint">
-        <param name="id">12</param>
+      <joint name="arm_shoulder_pitch_joint">
+        <xacro:unless value="${$(arg enable_gz)}">
+          <param name="id">11</param>
+        </xacro:unless>
         <command_interface name="position">
           <param name="min">-1.570796327</param>
@@ -61,39 +67,60 @@
         <state_interface name="effort"/>
       </joint>
-      <joint name="arm_elbow_1_tilt_joint">
-        <param name="id">13</param>
-        <command_interface name="position">
-          <param name="min">-1.570796327</param>
-          <param name="max">1.570796327</param>
-        </command_interface>
-        <command_interface name="velocity"/>
-        <state_interface name="position">
-          <param name="initial_value">-1.40</param>
-        </state_interface>
-        <state_interface name="velocity"/>
-        <state_interface name="effort"/>
-      </joint>
-      <joint name="arm_elbow_2_tilt_joint">
+      <joint name="arm_elbow_pitch_joint">
+        <xacro:unless value="${$(arg enable_gz)}">
+          <param name="id">13</param>
+        </xacro:unless>
+        <command_interface name="position">
+          <param name="min">-1.570796327</param>
+          <param name="max">1.570796327</param>
+        </command_interface>
+        <command_interface name="velocity"/>
+        <state_interface name="position">
+          <param name="initial_value">0.0</param>
+        </state_interface>
+        <state_interface name="velocity"/>
+        <state_interface name="effort"/>
+      </joint>
+      <joint name="arm_forearm_roll_joint">
+        <xacro:unless value="${$(arg enable_gz)}">
           <param name="id">14</param>
-        <command_interface name="position">
-          <param name="min">-3.141592654</param>
-          <param name="max">3.141592654</param>
-        </command_interface>
-        <command_interface name="velocity"/>
-        <state_interface name="position">
-          <param name="initial_value">1.4</param>
-        </state_interface>
-        <state_interface name="velocity"/>
-        <state_interface name="effort"/>
-      </joint>
-      <joint name="arm_wrist_tilt_joint">
-        <param name="id">15</param>
-        <command_interface name="position">
-          <param name="min">-1.570796327</param>
-          <param name="max">1.570796327</param>
-        </command_interface>
-        <command_interface name="velocity"/>
-        <state_interface name="position">
-          <param name="initial_value">-0.17</param>
+        </xacro:unless>
+        <command_interface name="position">
+          <param name="min">-3.141592654</param>
+          <param name="max">3.141592654</param>
+        </command_interface>
+        <command_interface name="velocity"/>
+        <state_interface name="position">
+          <param name="initial_value">0.0</param>
+        </state_interface>
+        <state_interface name="velocity"/>
+        <state_interface name="effort"/>
+      </joint>
+      <joint name="arm_wrist_pitch_joint">
+        <xacro:unless value="${$(arg enable_gz)}">
+          <param name="id">15</param>
+        </xacro:unless>
+        <command_interface name="position">
+          <param name="min">-1.570796327</param>
+          <param name="max">1.570796327</param>
+        </command_interface>
+        <command_interface name="velocity"/>
+        <state_interface name="position">
+          <param name="initial_value">0.0</param>
+        </state_interface>
+        <state_interface name="velocity"/>
+        <state_interface name="effort"/>
+      </joint>
+      <joint name="arm_wrist_roll_joint">
+        <xacro:unless value="${$(arg enable_gz)}">
+          <param name="id">16</param>
+        </xacro:unless>
+        <command_interface name="position">
+          <param name="min">-3.141592654</param>
+          <param name="max">3.141592654</param>
+        </command_interface>
+        <command_interface name="velocity"/>
+        <state_interface name="position">
+          <param name="initial_value">0.0</param>
         </state_interface>
         <state_interface name="velocity"/>
@@ -102,5 +129,7 @@
       <!-- Position Drive: Hand -->
       <joint name="hand_joint">
-        <param name="id">16</param>
+        <xacro:unless value="${$(arg enable_gz)}">
+          <param name="id">17</param>
+        </xacro:unless>
         <command_interface name="position"/>
         <command_interface name="velocity"/>
@@ -111,4 +140,15 @@
         <state_interface name="effort"/>
       </joint>
+      <xacro:if value="${$(arg enable_gz)}">
+        <joint name="hand_sub_joint">
+          <param name="mimic">hand_joint</param>
+          <param name="multiplier">-1</param>
+          <command_interface name="position"/>
+          <command_interface name="velocity"/>
+          <state_interface name="position"/>
+          <state_interface name="velocity"/>
+          <state_interface name="effort"/>
+        </joint>
+      </xacro:if>
       <!-- Position Drive: Head -->
       <joint name="head_camera_pan_joint">

Commit message: develop library

File: sobit_edu_description/urdf/arm/arm.urdf.xacro (robot description, xacro)
@@ -100,5 +100,5 @@
       <origin xyz="0.0 0.0 0.05095" rpy="0 0 0"/>
       <axis xyz="0 1 0"/>
-      <limit velocity="4.8" effort="25" lower="${-M_PI/2}" upper="${M_PI/2}" />
+      <limit velocity="4.8" effort="25" lower="${-M_PI/2}" upper="${3*M_PI/4}" />
     </joint>
     <!--  Act 2: Shoulder Pitch (right) -->
@@ -131,5 +131,5 @@
       <origin xyz="0.0 0.0 0.05095" rpy="0 0 0"/>
       <axis xyz="0 1 0"/>
-      <limit velocity="4.8" effort="25" lower="${-M_PI/2}" upper="${M_PI/2}" />
+      <limit velocity="4.8" effort="25" lower="${-3*M_PI/4}" upper="${M_PI/2}" />
       <!-- <mimic joint="${prefix}_shoulder_pitch_joint" multiplier="-1" offset="0"/> -->
     </joint>

File: sobit_edu_description/urdf/controllers.urdf.xacro (robot description, xacro)
@@ -41,5 +41,5 @@
         <!-- <command_interface name="position"/> -->
         <command_interface name="position">
-          <param name="min">-1.570796327</param>
+          <param name="min">-2.356194490192345</param>
           <param name="max">1.570796327</param>
         </command_interface>
@@ -58,5 +58,5 @@
         <command_interface name="position">
           <param name="min">-1.570796327</param>
-          <param name="max">1.570796327</param>
+          <param name="max">2.356194490192345</param>
         </command_interface>
         <command_interface name="velocity"/>

Commit message: FIX urdf and mesh of hand

File: sobit_edu_description/urdf/arm/arm.urdf.xacro (robot description, xacro)
@@ -270,5 +270,5 @@
         <origin xyz="${0.0505/2} 0.0 ${0.03775-0.0495/2}" rpy="0 0 0"/>
         <geometry>
-          <box size="0.0505 0.0335 0.0495"/>
+          <box size="0.0505 0.1886 0.0495"/>
         </geometry>
       </collision>

File: sobit_edu_description/urdf/hand/hand.urdf.xacro (robot description, xacro)
@@ -67,5 +67,5 @@
       <origin xyz="0.0 0.04 0.0" rpy="0 0 0"/>
       <axis xyz="0 1 0"/>
-      <limit velocity="4.8" effort="1" lower="0.0" upper="${0.02675-0.055}" />
+      <limit velocity="4.8" effort="1" lower="-0.01791787" upper="0.02901195" />
     </joint>
     <!--  Act 8: Hand Finger (left) -->

Commit message: FIX name of mesh files

File: sobit_edu_description/urdf/arm/arm.urdf.xacro (robot description, xacro)
@@ -139,5 +139,5 @@
         <origin xyz="0 0 0" rpy="0 0 ${M_PI/2}"/>
         <geometry>
-          <mesh filename="file://$(find sobit_light_description)/meshes/arm/omx1_link3.stl" scale="0.001 0.001 0.001"/>
+          <mesh filename="file://$(find sobit_edu_description)/meshes/arm/omx1_link3.stl" scale="0.001 0.001 0.001"/>
         </geometry>
         <material name="black"/>

File: sobit_edu_description/urdf/hand/hand.urdf.xacro (robot description, xacro)
@@ -14,5 +14,5 @@
         <origin xyz="0 0 0" rpy="0 0 ${M_PI/2}"/>
         <geometry>
-          <mesh filename="file://$(find sobit_edu_description)/meshes/hand/omx1_link9-10_hand.stl" scale="0.001 0.001 0.001"/>
+          <mesh filename="file://$(find sobit_edu_description)/meshes/hand/omx1_link9_10_hand.stl" scale="0.001 0.001 0.001"/>
         </geometry>
         <material name="black"/>
@@ -43,5 +43,5 @@
         <origin xyz="0 0 0" rpy="0 ${M_PI} ${M_PI/2}"/>
         <geometry>
-          <mesh filename="file://$(find sobit_edu_description)/meshes/hand/omx1_link9-10_hand.stl" scale="0.001 0.001 0.001"/>
+          <mesh filename="file://$(find sobit_edu_description)/meshes/hand/omx1_link9_10_hand.stl" scale="0.001 0.001 0.001"/>
         </geometry>
         <material name="black"/>
@@ -74,5 +74,5 @@
         <origin xyz="0.0 0.0 0" rpy="0 0 ${M_PI/2}"/>
         <geometry>
-          <mesh filename="file://$(find sobit_edu_description)/meshes/hand/omx1_link11-12_finger.stl" scale="0.001 0.001 0.001"/>
+          <mesh filename="file://$(find sobit_edu_description)/meshes/hand/omx1_link11_12_finger.stl" scale="0.001 0.001 0.001"/>
         </geometry>
         <material name="black"/>
@@ -106,5 +106,5 @@
         <origin xyz="0.0 -0.0 0" rpy="0 ${M_PI} ${M_PI/2}"/>
         <geometry>
-          <mesh filename="file://$(find sobit_edu_description)/meshes/hand/omx1_link11-12_finger.stl" scale="0.001 0.001 0.001"/>
+          <mesh filename="file://$(find sobit_edu_description)/meshes/hand/omx1_link11_12_finger.stl" scale="0.001 0.001 0.001"/>
         </geometry>
         <material name="black"/>
@@ -135,5 +135,5 @@
         <origin xyz="0.0 -0.0 0" rpy="0 0 ${M_PI/2}"/>
         <geometry>
-          <mesh filename="file://$(find sobit_edu_description)/meshes/hand/omx1_link13-14_finger.stl" scale="0.001 0.001 0.001"/>
+          <mesh filename="file://$(find sobit_edu_description)/meshes/hand/omx1_link13_14_finger.stl" scale="0.001 0.001 0.001"/>
         </geometry>
         <material name="black"/>
@@ -164,5 +164,5 @@
         <origin xyz="0.0 -0.0 0" rpy="0 ${M_PI} ${M_PI/2}"/>
         <geometry>
-          <mesh filename="file://$(find sobit_edu_description)/meshes/hand/omx1_link13-14_finger.stl" scale="0.001 0.001 0.001"/>
+          <mesh filename="file://$(find sobit_edu_description)/meshes/hand/omx1_link13_14_finger.stl" scale="0.001 0.001 0.001"/>
         </geometry>
         <material name="black"/>
