Commit message: FIX mimic param in sobit_edu_description

File: sobit_edu_description/urdf/arm/arm.transmission.xacro (robot description, xacro)
@@ -5,5 +5,4 @@
     <position_joint_transmission joint="${prefix}_shoulder_roll_joint"    reduction="1" />
     <position_joint_transmission joint="${prefix}_shoulder_pitch_joint" reduction="1" />
-    <position_joint_transmission joint="${prefix}_shoulder_pitch_sub_joint" reduction="1" />
     <position_joint_transmission joint="${prefix}_elbow_pitch_joint"    reduction="1" />
     <position_joint_transmission joint="${prefix}_forearm_roll_joint" reduction="1" />

File: sobit_edu_description/urdf/arm/arm.urdf.xacro (robot description, xacro)
@@ -130,7 +130,7 @@
       <child link="${prefix}_shoulder_pitch_sub_link"/>
       <origin xyz="0.0 0.0 0.05095" rpy="0 0 0"/>
-      <axis xyz="0 1 0"/>
-      <limit velocity="4.8" effort="25" lower="${-3*M_PI/4}" upper="${M_PI/2}" />
-      <!-- <mimic joint="${prefix}_shoulder_pitch_joint" multiplier="-1" offset="0"/> -->
+      <axis xyz="0 -1 0"/>
+      <limit velocity="4.8" effort="25" lower="${M_PI/2}" upper="${-3*M_PI/4}" />
+      <mimic joint="${prefix}_shoulder_pitch_joint" multiplier="-1" offset="0"/>
     </joint>
     <!--  Act 3: Shoulder Pitch (left) -->

File: sobit_edu_description/urdf/controllers.urdf.xacro (robot description, xacro)
@@ -133,18 +133,6 @@
         <param name="Return_Delay_Time">0</param>
       </xacro:unless>
-      <!-- <param name="mimic">arm_shoulder_pitch_joint</param>
-      <param name="multiplier">-1</param> -->
-      <!-- <command_interface name="position"/> -->
-      <command_interface name="position">
-        <param name="min">-2.356194490192345</param>
-        <param name="max">1.570796327</param>
-      </command_interface>
-      <!-- <command_interface name="velocity"/> -->
-      <state_interface name="position">
-        <param name="initial_value">0.0</param>
-      </state_interface>
-      <!-- <state_interface name="position"/> -->
-      <state_interface name="velocity"/>
-      <state_interface name="effort"/>
+      <param name="mimic">arm_shoulder_pitch_joint</param>
+      <param name="multiplier">-1</param>
     </joint>
     <joint name="arm_shoulder_pitch_joint">
@@ -262,9 +250,4 @@
         <param name="mimic">hand_joint</param>
         <param name="multiplier">-1</param>
-        <!-- <command_interface name="position"/> -->
-        <!-- <command_interface name="velocity"/> -->
-        <state_interface name="position"/>
-        <state_interface name="velocity"/>
-        <state_interface name="effort"/>
       </joint>
     </xacro:if>
