Commit message: add support for azure kinect

File: sobit_edu_description/robots/sobit_edu.urdf.xacro (robot description, xacro)
@@ -12,9 +12,10 @@
   <xacro:include filename="$(find sobit_edu_description)/urdf/back/back.urdf.xacro" />
   <xacro:include filename="$(find sobit_edu_description)/urdf/head/head.urdf.xacro" />
+  <xacro:include filename="$(find sobit_edu_description)/urdf/sensor/matrix.urdf.xacro" />
+  <xacro:include filename="$(find sobit_edu_description)/urdf/sensor/mic.urdf.xacro" />
+  <xacro:include filename="$(find sobit_edu_description)/urdf/sensor/lidar.urdf.xacro" />
   <xacro:include filename="$(find sobit_edu_description)/urdf/sensor/head_camera.urdf.xacro" />
-  <xacro:include filename="$(find sobit_edu_description)/urdf/sensor/mic.urdf.xacro" />
-  <xacro:include filename="$(find sobit_edu_description)/urdf/sensor/matrix.urdf.xacro" />
-  <xacro:include filename="$(find sobit_edu_description)/urdf/sensor/lidar.urdf.xacro" />
   <xacro:include filename="$(find urg_node)/urdf/hokuyo_ust.urdf.xacro" />
+  <xacro:include filename="$(find azure_kinect_ros_driver)/urdf/azure_kinect.urdf.xacro" />
   <!-- Connect the previous Links and Joints -->
   <xacro:base/>
@@ -25,5 +26,5 @@
   <xacro:back prefix="back" parent="plate_top_link" />
   <xacro:head prefix="head" parent="back_base_link" />
-  <xacro:head_camera prefix="head_camera" parent="head_double_sided_tape_link" />
+  <xacro:head_camera prefix="head_camera" parent="head_camera_tilt_link" />
   <xacro:mic prefix="mic" parent="back_base_link" />
   <xacro:matrix prefix="matrix" parent="back_base_link" />

File: sobit_edu_description/urdf/head/head.urdf.xacro (robot description, xacro)
@@ -23,5 +23,5 @@
       </collision>
       <inertial>
-        <origin rpy="0.0 0.0 0.0" xyz="0.0 0.0 0.0" />
+        <origin xyz="0.0 0.0 0.0" rpy="${M_PI/2.0} 0.0 ${M_PI/2.0}" />
         <mass value="0.08" />
         <inertia ixx="1.0" ixy="0.0" ixz="0.0"
@@ -52,5 +52,5 @@
       </collision>
       <inertial>
-        <origin rpy="0.0 0.0 0.0" xyz="0.0 0.0 0.0" />
+        <origin xyz="0.0 0.0 0.0" rpy="0.0 0.0 ${-M_PI/2.0}" />
         <mass value="0.08" />
         <inertia ixx="1.0" ixy="0.0" ixz="0.0"
@@ -63,10 +63,10 @@
       <child link="${prefix}_camera_tilt_link" />
       <origin xyz="0.0 0.0 0.0435" rpy="0.0 0.0 0.0" />
-      <axis xyz="0 1 0" />
+      <axis xyz="0 -1 0" />
       <limit effort="30" lower="${-M_PI/2.0}" upper="${M_PI/2.0}" velocity="${M_PI/2.0}" />
     </joint>
     <link name="${prefix}_camera_tilt_link">
       <visual>
-        <origin xyz="0.0 0.0 0.0" rpy="${M_PI/2.0} 0.0 0.0" />
+        <origin xyz="0.0 0.0 0.0" rpy="0.0 0.0 ${M_PI/2.0}" />
         <geometry>
           <mesh filename="package://sobit_edu_description/meshes/head/head_camera_tilt.stl" scale="0.001 0.001 0.001" />
@@ -75,5 +75,5 @@
       </visual>
       <collision>
-        <origin xyz="0.0 0.0 0.0" rpy="${M_PI/2.0} 0.0 0.0" />
+        <origin xyz="0.0 0.0 0.0" rpy="0.0 0.0 ${M_PI/2.0}" />
         <geometry>
           <mesh filename="package://sobit_edu_description/meshes/head/head_camera_tilt.stl" scale="0.001 0.001 0.001" />
@@ -81,5 +81,5 @@
       </collision>
       <inertial>
-        <origin rpy="0.0 0.0 0.0" xyz="0.0 0.0 0.0" />
+        <origin xyz="0.0 0.0 0.0" rpy="0.0 0.0 ${M_PI/2.0}" />
         <mass value="0.08" />
         <inertia ixx="1.0" ixy="0.0" ixz="0.0"
@@ -88,10 +88,4 @@
       </inertial>
     </link>
-    <joint name="${prefix}_double_sided_tape_joint" type="fixed">
-      <parent link="${prefix}_camera_tilt_link" />
-      <child link="${prefix}_double_sided_tape_link" />
-      <origin xyz="0.0 0.0 0.029" rpy="0.0 0.0 0.0" />
-    </joint>
-    <link name="${prefix}_double_sided_tape_link" />
     <xacro:head_transmission prefix="${prefix}" />
   </xacro:macro>

File: sobit_edu_description/urdf/sensor/head_camera.urdf.xacro (robot description, xacro)
@@ -2,127 +2,14 @@
 <!-- Reference: https://github.com/M_PIrobot/M_PI-kobuki-git/blob/master/M_PIko_description/urdf/xtion.urdf.xacro -->
 <robot name="head_camera" xmlns:xacro="http://ros.org/wiki/xacro">
-  <xacro:include filename="$(find turtlebot_description)/urdf/turtlebot_gazebo.urdf.xacro" />
-  <xacro:include filename="$(find turtlebot_description)/urdf/turtlebot_properties.urdf.xacro" />
-  <!-- Xacro properties -->
-  <xacro:property name="xtion_pro_depth_rel_rgb_py" value="0.0270" />
-  <xacro:property name="xtion_pro_cam_rel_rgb_py"   value="-0.0220" />
-  <!-- Parameterised in part by the values in turtlebot_properties.urdf.xacro -->
-  <!-- xtion_pro_cam_py allows for a camera displaced so the depth optical frame aligns with robot center -->
   <xacro:macro name="head_camera" params="prefix parent">
-    <joint name="${prefix}_rgb_joint" type="fixed">
-      <origin xyz="0.01088 0.02 0.0125" rpy="0 0 0" />
+    <joint name="${prefix}_joint" type="fixed">
       <parent link="${parent}" />
-      <child link="${prefix}_rgb_frame" />
+      <child link="${prefix}_link" />
+      <origin xyz="-0.0065 0.0 0.0395" rpy="0.0 0.0 0.0" />
     </joint>
-    <link name="${prefix}_rgb_frame" />
-    <joint name="${prefix}_rgb_optical_joint" type="fixed">
-      <origin xyz="0 0 0" rpy="${-M_PI/2} 0 ${-M_PI/2}" />
-      <parent link="${prefix}_rgb_frame" />
-      <child link="${prefix}_rgb_optical_frame" />
-    </joint>
-    <link name="${prefix}_rgb_optical_frame" />
-    <joint name="${prefix}_joint" type="fixed">
-      <origin xyz="0 ${xtion_pro_cam_rel_rgb_py} 0" rpy="0 0 0" />
-      <parent link="${prefix}_rgb_frame" />
-      <child link="${prefix}_link" />
-    </joint>
-    <link name="${prefix}_link">
-      <visual>
-        <origin xyz="-0.015 0.0035 0.004" rpy="0 0 0" />
-        <geometry>
-          <mesh filename="package://turtlebot_description/meshes/sensors/xtion_pro_camera.dae" />
-        </geometry>
-      </visual>
-      <collision>
-        <origin xyz="0.0 0.0 0.0" rpy="0 0 0" />
-        <geometry>
-        <box size="0.0730 0.2760 0.0720" />
-      </geometry>
-      </collision>
-      <inertial>
-        <mass value="0.170" />
-        <origin xyz="0 0 0" />
-        <inertia ixx="0.001152600" ixy="0.0" ixz="0.0"
-                 iyy="0.000148934" iyz="0.0"
-                 izz="0.001154654" />
-      </inertial>
-    </link>
-    <joint name="${prefix}_depth_joint" type="fixed">
-      <origin xyz="0 ${xtion_pro_depth_rel_rgb_py} 0" rpy="0 0 0" />
-      <parent link="${prefix}_rgb_frame" />
-      <child link="${prefix}_depth_frame" />
-    </joint>
-    <link name="${prefix}_depth_frame" />
-    <joint name="${prefix}_depth_optical_joint" type="fixed">
-      <origin xyz="0 0 0" rpy="${-M_PI/2} 0 ${-M_PI/2}" />
-      <parent link="${prefix}_depth_frame" />
-      <child link="${prefix}_depth_optical_frame" />
-    </joint>
-    <link name="${prefix}_depth_optical_frame" />
-    <!-- RGBD sensor for simulation, same as Kinect -->
-    <xacro:turtlebot_sim_3dsensor/>
-    <!-- Asus mount -->
-    <!-- <joint name="mount_xtion_pro_joint" type="fixed">
-      <origin xyz="-0.1024 0.0 0.272" rpy="0 0 0" />
-      <parent link="${parent}" />
-      <child link="mount_xtion_pro_link" />
-    </joint>
-    <link name="mount_xtion_pro_link">
-      <visual>
-        <origin xyz="0 0 0" rpy="${-M_PI/2} 0 0" />
-        <geometry>
-          <mesh filename="package://turtlebot_description/meshes/sensors/xtion_pro_stack.dae" />
-        </geometry>
-      </visual>
-      <collision>
-        <origin xyz="0.0 0.0 0.0" rpy="0 0 0" />
-        <geometry>
-        <box size="0.0330 0.2760 0.0120" />
-      </geometry>
-      </collision>
-      <inertial>
-        <mass value="0.170" />
-        <origin xyz="0 0 0" />
-        <inertia ixx="0.001152600" ixy="0.0" ixz="0.0"
-                 iyy="0.000148934" iyz="0.0"
-                 izz="0.001154654" />
-      </inertial>
-    </link> -->
-    <!-- <gazebo reference="${prefix}_link">
-      <sensor type="depth" name="camera">
-        <always_on>true</always_on>
-        <update_rate>20.0</update_rate>
-        <camera>
-          <horizontal_fov>${60.0*M_M_PI/180.0}</horizontal_fov>
-          <image>
-            <format>B8G8R8</format>
-            <width>640</width>
-            <height>480</height>
-          </image>
-          <clip>
-            <near>0.05</near>
-            <far>8.0</far>
-          </clip>
-        </camera>
-        <plugin name="kinect_camera_controller" filename="libgazebo_ros_openni_kinect.so">
-          <cameraName>camera</cameraName>
-          <alwaysOn>true</alwaysOn>
-          <updateRate>10</updateRate>
-          <imageToM_PIcName>rgb/image_raw</imageToM_PIcName>
-          <depthImageToM_PIcName>depth/image_raw</depthImageToM_PIcName>
-          <pointCloudToM_PIcName>depth/points</pointCloudToM_PIcName>
-          <cameraInfoToM_PIcName>rgb/camera_info</cameraInfoToM_PIcName>
-          <depthImageCameraInfoToM_PIcName>depth/camera_info</depthImageCameraInfoToM_PIcName>
-          <frameName>camera_depth_optical_frame</frameName>
-          <baseline>0.1</baseline>
-          <distortion_k1>0.0</distortion_k1>
-          <distortion_k2>0.0</distortion_k2>
-          <distortion_k3>0.0</distortion_k3>
-          <distortion_t1>0.0</distortion_t1>
-          <distortion_t2>0.0</distortion_t2>
-          <pointCloudCutoff>0.4</pointCloudCutoff>
-        </plugin>
-      </sensor>
-    </gazebo> -->
+    <link name="${prefix}_link"/>
+    <xacro:azure_kinect parent="${prefix}_link" tf_prefix="${prefix}_" add_cover="false">
+      <origin xyz="0.0 0 0.0" rpy="0 0 0"/>
+    </xacro:azure_kinect>
   </xacro:macro>
 </robot>
