Commit message: [UPD]required dependencies

File: sobit_edu_description/robots/sobit_edu.urdf.xacro (robot description, xacro)
@@ -4,4 +4,6 @@
   <xacro:include filename="$(find sobit_edu_description)/urdf/common.xacro" />
   <xacro:include filename="$(find sobit_edu_description)/urdf/materials.urdf.xacro" />
+  <xacro:include filename="$(find sobit_edu_description)/urdf/transmission.urdf.xacro" />
+  <xacro:include filename="$(find sobit_edu_description)/urdf/controllers.urdf.xacro" />
   <!-- Add URDF: links, joints -->
   <xacro:include filename="$(find sobit_edu_description)/urdf/base/base.urdf.xacro" />
@@ -9,7 +11,10 @@
   <xacro:include filename="$(find sobit_edu_description)/urdf/body/cover.urdf.xacro" />
   <xacro:include filename="$(find sobit_edu_description)/urdf/arm/arm.urdf.xacro" />
+  <xacro:include filename="$(find sobit_edu_description)/urdf/arm/arm.transmission.xacro" />
   <xacro:include filename="$(find sobit_edu_description)/urdf/hand/hand.urdf.xacro" />
+   <xacro:include filename="$(find sobit_edu_description)/urdf/hand/hand.transmission.xacro" />
   <xacro:include filename="$(find sobit_edu_description)/urdf/back/back.urdf.xacro" />
   <xacro:include filename="$(find sobit_edu_description)/urdf/head/head.urdf.xacro" />
+  <xacro:include filename="$(find sobit_edu_description)/urdf/head/head.transmission.xacro" />
   <xacro:include filename="$(find sobit_edu_description)/urdf/sensor/matrix.urdf.xacro" />
   <xacro:include filename="$(find sobit_edu_description)/urdf/sensor/mic.urdf.xacro" />
@@ -17,5 +22,5 @@
   <xacro:include filename="$(find sobit_edu_description)/urdf/sensor/head_camera.urdf.xacro" />
   <xacro:include filename="$(find urg_node)/urdf/hokuyo_ust.urdf.xacro" />
-  <xacro:include filename="$(find azure_kinect_ros_driver)/urdf/azure_kinect.urdf.xacro" />
+  <!-- <xacro:include filename="$(find azure_kinect_ros_driver)/urdf/azure_kinect.urdf.xacro" /> -->
   <!-- Connect the previous Links and Joints -->
   <xacro:base/>

File: sobit_edu_description/urdf/arm/arm.urdf.xacro (robot description, xacro)
@@ -12,5 +12,5 @@
         <origin xyz="0.0 0.0 0.0" rpy="0.0 0.0 ${M_PI/2.0}" />
         <geometry>
-          <mesh filename="package://sobit_edu_description/meshes/arm/arm_base.stl" scale="0.001 0.001 0.001" />
+          <mesh filename="file://$(find sobit_edu_description)/meshes/arm/arm_base.stl" scale="0.001 0.001 0.001" />
         </geometry>
         <material name="black" />
@@ -19,5 +19,5 @@
         <origin xyz="0.0 0.0 0.0" rpy="0.0 0.0 ${M_PI/2.0}" />
         <geometry>
-          <mesh filename="package://sobit_edu_description/meshes/arm/arm_base.stl" scale="0.001 0.001 0.001" />
+          <mesh filename="file://$(find sobit_edu_description)/meshes/arm/arm_base.stl" scale="0.001 0.001 0.001" />
         </geometry>
       </collision>
@@ -41,5 +41,5 @@
         <origin xyz="0.0 0 0.0" rpy="0.0 0.0 ${M_PI/2.0}" />
         <geometry>
-          <mesh filename="package://sobit_edu_description/meshes/arm/arm_rotate.stl" scale="0.001 0.001 0.001" />
+          <mesh filename="file://$(find sobit_edu_description)/meshes/arm/arm_rotate.stl" scale="0.001 0.001 0.001" />
         </geometry>
         <material name="black" />
@@ -48,5 +48,5 @@
         <origin xyz="0.0 0 0.0" rpy="0.0 0.0 ${M_PI/2.0}" />
         <geometry>
-          <mesh filename="package://sobit_edu_description/meshes/arm/arm_rotate.stl" scale="0.001 0.001 0.001" />
+          <mesh filename="file://$(find sobit_edu_description)/meshes/arm/arm_rotate.stl" scale="0.001 0.001 0.001" />
         </geometry>
       </collision>
@@ -70,5 +70,5 @@
         <origin xyz="0 0.0 0.0" rpy="0.0 0.0 ${M_PI/2.0}" />
         <geometry>
-          <mesh filename="package://sobit_edu_description/meshes/arm/arm_upper.stl" scale="0.001 0.001 0.001" />
+          <mesh filename="file://$(find sobit_edu_description)/meshes/arm/arm_upper.stl" scale="0.001 0.001 0.001" />
         </geometry>
         <material name="black" />
@@ -77,5 +77,5 @@
         <origin xyz="0 0.0 0.0" rpy="0.0 0.0 ${M_PI/2.0}" />
         <geometry>
-          <mesh filename="package://sobit_edu_description/meshes/arm/arm_upper.stl" scale="0.001 0.001 0.001" />
+          <mesh filename="file://$(find sobit_edu_description)/meshes/arm/arm_upper.stl" scale="0.001 0.001 0.001" />
         </geometry>
       </collision>
@@ -108,5 +108,5 @@
         <origin xyz="0.0 0.0 0.0" rpy="0.0 0.0 ${M_PI/2.0}" />
         <geometry>
-          <mesh filename="package://sobit_edu_description/meshes/arm/arm_lower.stl" scale="0.001 0.001 0.001" />
+          <mesh filename="file://$(find sobit_edu_description)/meshes/arm/arm_lower.stl" scale="0.001 0.001 0.001" />
         </geometry>
         <material name="black" />
@@ -115,5 +115,5 @@
         <origin xyz="0.0 0.0 0.0" rpy="0.0 0.0 ${M_PI/2.0}" />
         <geometry>
-          <mesh filename="package://sobit_edu_description/meshes/arm/arm_lower.stl" scale="0.001 0.001 0.001" />
+          <mesh filename="file://$(find sobit_edu_description)/meshes/arm/arm_lower.stl" scale="0.001 0.001 0.001" />
         </geometry>
       </collision>

File: sobit_edu_description/urdf/back/back.urdf.xacro (robot description, xacro)
@@ -11,5 +11,5 @@
         <origin xyz="0.0 0.0 0.0" rpy="0.0 0.0 ${M_PI/2}" />
         <geometry>
-          <mesh filename="package://sobit_edu_description/meshes/back/back_base.stl" scale="0.001 0.001 0.001" />
+          <mesh filename="file://$(find sobit_edu_description)/meshes/back/back_base.stl" scale="0.001 0.001 0.001" />
         </geometry>
         <material name="grey" />
@@ -18,5 +18,5 @@
         <origin xyz="0.0 0.0 0.0" rpy="0.0 0.0 ${M_PI/2}" />
         <geometry>
-          <mesh filename="package://sobit_edu_description/meshes/back/back_base.stl" scale="0.001 0.001 0.001" />
+          <mesh filename="file://$(find sobit_edu_description)/meshes/back/back_base.stl" scale="0.001 0.001 0.001" />
         </geometry>
       </collision>

File: sobit_edu_description/urdf/base/base.urdf.xacro (robot description, xacro)
@@ -9,4 +9,6 @@
   <xacro:include filename="$(find kobuki_description)/urdf/common_properties.urdf.xacro" />
   <xacro:include filename="$(find kobuki_description)/urdf/kobuki_gazebo.urdf.xacro" />
+  <!-- <xacro:include filename="file://$(find kobuki_description)/urdf/common_properties.urdf.xacro" />
+  <xacro:include filename="file://$(find kobuki_description)/urdf/kobuki_gazebo.urdf.xacro" /> -->
   <!-- Kobuki -->
   <xacro:macro name="base">
@@ -30,5 +32,5 @@
         <geometry>
           <!-- new mesh -->
-          <mesh filename="package://kobuki_description/meshes/main_body.dae" />
+          <mesh filename="file://$(find kobuki_description)/meshes/main_body.dae" />
         </geometry>
         <origin xyz="0.001 0 0.05199" rpy="0 0 0" />
@@ -65,5 +67,5 @@
       <visual>
         <geometry>
-          <mesh filename="package://kobuki_description/meshes/wheel.dae" />
+          <mesh filename="file://$(find kobuki_description)/meshes/wheel.dae" />
         </geometry>
         <origin xyz="0 0 0" rpy="0 0 0" />
@@ -92,5 +94,5 @@
       <visual>
         <geometry>
-          <mesh filename="package://kobuki_description/meshes/wheel.dae" />
+          <mesh filename="file://$(find kobuki_description)/meshes/wheel.dae" />
         </geometry>
         <origin xyz="0 0 0" rpy="0 0 0" />

File: sobit_edu_description/urdf/body/cover.urdf.xacro (robot description, xacro)
@@ -11,5 +11,5 @@
         <origin xyz="0.0 0.0 0.0" rpy="0.0 ${M_PI/2.0} ${-M_PI/2.0}" />
         <geometry>
-          <mesh filename="package://sobit_edu_description/meshes/body/cover.stl" scale="0.001 0.001 0.001" />
+          <mesh filename="file://$(find sobit_edu_description)/meshes/body/cover.stl" scale="0.001 0.001 0.001" />
         </geometry>
         <material name="blue" />
@@ -18,5 +18,5 @@
         <origin xyz="0.0 0.0 0.0" rpy="0.0 ${M_PI/2.0} ${-M_PI/2.0}" />
         <geometry>
-          <mesh filename="package://sobit_edu_description/meshes/body/cover.stl" scale="0.001 0.001 0.001" />
+          <mesh filename="file://$(find sobit_edu_description)/meshes/body/cover.stl" scale="0.001 0.001 0.001" />
         </geometry>
       </collision>

File: sobit_edu_description/urdf/body/stacks.urdf.xacro (robot description, xacro)
@@ -4,5 +4,5 @@
  -->
 <robot name="stack_hexagons" xmlns:xacro="http://ros.org/wiki/xacro">
-  <xacro:include filename="$(find turtlebot_description)/urdf/common_properties.urdf.xacro" />
+  <xacro:include filename="$(find turtlebot2_description)/urdf/common_properties.urdf.xacro" />
   <!-- Xacro properties -->
   <xacro:property name="M_SCALE" value="0.001" />
@@ -20,5 +20,5 @@
         <geometry>
           <!-- <mesh filename="package://turtlebot_description/meshes/stacks/hexagons/pole_bottom.dae" /> -->
-          <mesh filename="package://sobit_edu_description/meshes/body/pole_bottom_39mm.stl" scale="${M_SCALE} ${M_SCALE} ${M_SCALE}" />
+          <mesh filename="file://$(find sobit_edu_description)/meshes/body/pole_bottom_39mm.stl" scale="${M_SCALE} ${M_SCALE} ${M_SCALE}" />
         </geometry>
         <material name="grey" />
@@ -50,5 +50,5 @@
         <geometry>
           <!-- <mesh filename="package://turtlebot_description/meshes/stacks/hexagons/pole_middle.dae" /> -->
-          <mesh filename="package://sobit_edu_description/meshes/body/pole_middle_90mm.stl" scale="${M_SCALE} ${M_SCALE} ${M_SCALE}" />
+          <mesh filename="file://$(find sobit_edu_description)/meshes/body/pole_middle_90mm.stl" scale="${M_SCALE} ${M_SCALE} ${M_SCALE}" />
         </geometry>
         <material name="grey" />
@@ -80,5 +80,5 @@
         <geometry>
           <!-- <mesh filename="package://turtlebot_description/meshes/stacks/hexagons/pole_top.dae" /> -->
-          <mesh filename="package://sobit_edu_description/meshes/body/pole_top_200mm.stl" scale="${M_SCALE} ${M_SCALE} ${M_SCALE}" />
+          <mesh filename="file://$(find sobit_edu_description)/meshes/body/pole_top_200mm.stl" scale="${M_SCALE} ${M_SCALE} ${M_SCALE}" />
         </geometry>
         <material name="grey" />
@@ -109,5 +109,5 @@
         <origin xyz="0.0 0.0 0.0" rpy="0.0 0.0 0.0" />
         <geometry>
-          <mesh filename="package://turtlebot_description/meshes/stacks/hexagons/pole_kinect.dae" />
+          <mesh filename="file://$(find turtlebot2_description)/meshes/stacks/hexagons/pole_kinect.dae" />
         </geometry>
       </visual>
@@ -148,5 +148,5 @@
         <origin xyz="0.0 0.0 0.0" rpy="0.0 0.0 0.0" />
         <geometry>
-          <mesh filename="package://turtlebot_description/meshes/stacks/hexagons/plate_bottom.dae" />
+          <mesh filename="file://$(find turtlebot2_description)/meshes/stacks/hexagons/plate_bottom.dae" />
         </geometry>
       </visual>
@@ -182,5 +182,5 @@
         <origin xyz="0.0 0.0 0.0" rpy="0.0 0.0 0.0" />
         <geometry>
-          <mesh filename="package://turtlebot_description/meshes/stacks/hexagons/plate_middle.dae" />
+          <mesh filename="file://$(find turtlebot2_description)/meshes/stacks/hexagons/plate_middle.dae" />
         </geometry>
       </visual>
@@ -188,5 +188,5 @@
         <origin xyz="0.01364 0.0 0.0" rpy="0.0 0.0 0.0" />
         <geometry>
-          <mesh filename="package://turtlebot_description/meshes/stacks/hexagons/plate_simple.stl" scale="${M_SCALE} ${M_SCALE} ${M_SCALE}" />
+          <mesh filename="file://$(find turtlebot2_description)/meshes/stacks/hexagons/plate_simple.stl" scale="${M_SCALE} ${M_SCALE} ${M_SCALE}" />
         </geometry>
       </collision>
@@ -215,5 +215,5 @@
         <origin xyz="0.0 0.0 -0.0" rpy="0.0 0.0 0.0" />
         <geometry>
-          <mesh filename="package://turtlebot_description/meshes/stacks/hexagons/plate_top.dae" />
+          <mesh filename="file://$(find turtlebot2_description)/meshes/stacks/hexagons/plate_top.dae" />
         </geometry>
       </visual>
@@ -221,5 +221,5 @@
         <origin xyz="0.01364 0.0 0.0" rpy="0.0 0.0 0.0" />
         <geometry>
-          <mesh filename="package://turtlebot_description/meshes/stacks/hexagons/plate_simple.stl" scale="${M_SCALE} ${M_SCALE} ${M_SCALE}" />
+          <mesh filename="file://$(find turtlebot2_description)/meshes/stacks/hexagons/plate_simple.stl" scale="${M_SCALE} ${M_SCALE} ${M_SCALE}" />
         </geometry>
       </collision>

File: sobit_edu_description/urdf/hand/hand.urdf.xacro (robot description, xacro)
@@ -12,5 +12,5 @@
         <origin xyz="0.0 0.0 0.0" rpy="0.0 0.0 ${M_PI/2.0}" />
         <geometry>
-          <mesh filename="package://sobit_edu_description/meshes/hand/hand_back.stl" scale="0.001 0.001 0.001" />
+          <mesh filename="file://$(find sobit_edu_description)/meshes/hand/hand_back.stl" scale="0.001 0.001 0.001" />
         </geometry>
         <material name="black" />
@@ -19,5 +19,5 @@
         <origin xyz="0.0 0.0 0.0" rpy="0.0 0.0 ${M_PI/2.0}" />
         <geometry>
-          <mesh filename="package://sobit_edu_description/meshes/hand/hand_back.stl" scale="0.001 0.001 0.001" />
+          <mesh filename="file://$(find sobit_edu_description)/meshes/hand/hand_back.stl" scale="0.001 0.001 0.001" />
         </geometry>
       </collision>
@@ -50,12 +50,12 @@
         <origin xyz="0.0 0.0 0.0" rpy="${M_PI/2.0} 0.0 ${M_PI/2.0}" />
         <geometry>
-          <mesh filename="package://sobit_edu_description/meshes/hand/hand_inner_l.stl" scale="0.001 0.001 0.001" />
-        </geometry>
-        <material name="black" />
-      </visual>
-      <collision>
-        <origin xyz="0.0 0.0 0.0" rpy="${M_PI/2.0} 0.0 ${M_PI/2.0}" />
-        <geometry>
-          <mesh filename="package://sobit_edu_description/meshes/hand/hand_inner_l.stl" scale="0.001 0.001 0.001" />
+          <mesh filename="file://$(find sobit_edu_description)/meshes/hand/hand_inner_l.stl" scale="0.001 0.001 0.001" />
+        </geometry>
+        <material name="black" />
+      </visual>
+      <collision>
+        <origin xyz="0.0 0.0 0.0" rpy="${M_PI/2.0} 0.0 ${M_PI/2.0}" />
+        <geometry>
+          <mesh filename="file://$(find sobit_edu_description)/meshes/hand/hand_inner_l.stl" scale="0.001 0.001 0.001" />
         </geometry>
       </collision>
@@ -80,12 +80,12 @@
         <origin xyz="0.0 0.0 0.0" rpy="${M_PI/2.0} 0.0 ${M_PI/2.0}" />
         <geometry>
-          <mesh filename="package://sobit_edu_description/meshes/hand/hand_inner_r.stl" scale="0.001 0.001 0.001" />
-        </geometry>
-        <material name="black" />
-      </visual>
-      <collision>
-        <origin xyz="0.0 0.0 0.0" rpy="${M_PI/2.0} 0.0 ${M_PI/2.0}" />
-        <geometry>
-          <mesh filename="package://sobit_edu_description/meshes/hand/hand_inner_r.stl" scale="0.001 0.001 0.001" />
+          <mesh filename="file://$(find sobit_edu_description)/meshes/hand/hand_inner_r.stl" scale="0.001 0.001 0.001" />
+        </geometry>
+        <material name="black" />
+      </visual>
+      <collision>
+        <origin xyz="0.0 0.0 0.0" rpy="${M_PI/2.0} 0.0 ${M_PI/2.0}" />
+        <geometry>
+          <mesh filename="file://$(find sobit_edu_description)/meshes/hand/hand_inner_r.stl" scale="0.001 0.001 0.001" />
         </geometry>
       </collision>
@@ -110,12 +110,12 @@
         <origin xyz="0.0 0.0 0.0" rpy="${M_PI/2.0} 0.0 ${M_PI/2.0}" />
         <geometry>
-          <mesh filename="package://sobit_edu_description/meshes/hand/hand_outer_l.stl" scale="0.001 0.001 0.001" />
-        </geometry>
-        <material name="black" />
-      </visual>
-      <collision>
-        <origin xyz="0.0 0.0 0.0" rpy="${M_PI/2.0} 0.0 ${M_PI/2.0}" />
-        <geometry>
-          <mesh filename="package://sobit_edu_description/meshes/hand/hand_outer_l.stl" scale="0.001 0.001 0.001" />
+          <mesh filename="file://$(find sobit_edu_description)/meshes/hand/hand_outer_l.stl" scale="0.001 0.001 0.001" />
+        </geometry>
+        <material name="black" />
+      </visual>
+      <collision>
+        <origin xyz="0.0 0.0 0.0" rpy="${M_PI/2.0} 0.0 ${M_PI/2.0}" />
+        <geometry>
+          <mesh filename="file://$(find sobit_edu_description)/meshes/hand/hand_outer_l.stl" scale="0.001 0.001 0.001" />
         </geometry>
       </collision>
@@ -140,12 +140,12 @@
         <origin xyz="0.0 0.0 0.0" rpy="${M_PI/2.0} 0.0 ${M_PI/2.0}" />
         <geometry>
-          <mesh filename="package://sobit_edu_description/meshes/hand/hand_outer_r.stl" scale="0.001 0.001 0.001" />
-        </geometry>
-        <material name="black" />
-      </visual>
-      <collision>
-        <origin xyz="0.0 0.0 0.0" rpy="${M_PI/2.0} 0.0 ${M_PI/2.0}" />
-        <geometry>
-          <mesh filename="package://sobit_edu_description/meshes/hand/hand_outer_r.stl" scale="0.001 0.001 0.001" />
+          <mesh filename="file://$(find sobit_edu_description)/meshes/hand/hand_outer_r.stl" scale="0.001 0.001 0.001" />
+        </geometry>
+        <material name="black" />
+      </visual>
+      <collision>
+        <origin xyz="0.0 0.0 0.0" rpy="${M_PI/2.0} 0.0 ${M_PI/2.0}" />
+        <geometry>
+          <mesh filename="file://$(find sobit_edu_description)/meshes/hand/hand_outer_r.stl" scale="0.001 0.001 0.001" />
         </geometry>
       </collision>
@@ -170,12 +170,12 @@
         <origin xyz="0.0 0.0 0.0" rpy="${M_PI/2.0} 0.0 ${M_PI/2.0}" />
         <geometry>
-          <mesh filename="package://sobit_edu_description/meshes/hand/hand_finger_l.stl" scale="0.001 0.001 0.001" />
-        </geometry>
-        <material name="black" />
-      </visual>
-      <collision>
-        <origin xyz="0.0 0.0 0.0" rpy="${M_PI/2.0} 0.0 ${M_PI/2.0}" />
-        <geometry>
-          <mesh filename="package://sobit_edu_description/meshes/hand/hand_finger_l.stl" scale="0.001 0.001 0.001" />
+          <mesh filename="file://$(find sobit_edu_description)/meshes/hand/hand_finger_l.stl" scale="0.001 0.001 0.001" />
+        </geometry>
+        <material name="black" />
+      </visual>
+      <collision>
+        <origin xyz="0.0 0.0 0.0" rpy="${M_PI/2.0} 0.0 ${M_PI/2.0}" />
+        <geometry>
+          <mesh filename="file://$(find sobit_edu_description)/meshes/hand/hand_finger_l.stl" scale="0.001 0.001 0.001" />
         </geometry>
       </collision>
@@ -200,12 +200,12 @@
         <origin xyz="0.0 0.0 0.0" rpy="${M_PI/2.0} 0.0 ${M_PI/2.0}" />
         <geometry>
-          <mesh filename="package://sobit_edu_description/meshes/hand/hand_finger_r.stl" scale="0.001 0.001 0.001" />
-        </geometry>
-        <material name="black" />
-      </visual>
-      <collision>
-        <origin xyz="0.0 0.0 0.0" rpy="${M_PI/2.0} 0.0 ${M_PI/2.0}" />
-        <geometry>
-          <mesh filename="package://sobit_edu_description/meshes/hand/hand_finger_r.stl" scale="0.001 0.001 0.001" />
+          <mesh filename="file://$(find sobit_edu_description)/meshes/hand/hand_finger_r.stl" scale="0.001 0.001 0.001" />
+        </geometry>
+        <material name="black" />
+      </visual>
+      <collision>
+        <origin xyz="0.0 0.0 0.0" rpy="${M_PI/2.0} 0.0 ${M_PI/2.0}" />
+        <geometry>
+          <mesh filename="file://$(find sobit_edu_description)/meshes/hand/hand_finger_r.stl" scale="0.001 0.001 0.001" />
         </geometry>
       </collision>

File: sobit_edu_description/urdf/head/head.urdf.xacro (robot description, xacro)
@@ -12,5 +12,5 @@
         <origin xyz="0.0 0.0 0.0" rpy="${M_PI/2.0} 0.0 ${M_PI/2.0}" />
         <geometry>
-          <mesh filename="package://sobit_edu_description/meshes/head/head_camera_base.stl" scale="0.001 0.001 0.001" />
+          <mesh filename="file://$(find sobit_edu_description)/meshes/head/head_camera_base.stl" scale="0.001 0.001 0.001" />
         </geometry>
         <material name="black" />
@@ -19,5 +19,5 @@
         <origin xyz="0.0 0.0 0.0" rpy="${M_PI/2.0} 0.0 ${M_PI/2.0}" />
         <geometry>
-          <mesh filename="package://sobit_edu_description/meshes/head/head_camera_base.stl" scale="0.001 0.001 0.001" />
+          <mesh filename="file://$(find sobit_edu_description)/meshes/head/head_camera_base.stl" scale="0.001 0.001 0.001" />
         </geometry>
       </collision>
@@ -41,5 +41,5 @@
         <origin xyz="0.0 0.0 0.0" rpy="0.0 0.0 ${-M_PI/2.0}" />
         <geometry>
-          <mesh filename="package://sobit_edu_description/meshes/head/head_camera_pan.stl" scale="0.001 0.001 0.001" />
+          <mesh filename="file://$(find sobit_edu_description)/meshes/head/head_camera_pan.stl" scale="0.001 0.001 0.001" />
         </geometry>
         <material name="black" />
@@ -48,5 +48,5 @@
         <origin xyz="0.0 0.0 0.0" rpy="0.0 0.0 ${-M_PI/2.0}" />
         <geometry>
-          <mesh filename="package://sobit_edu_description/meshes/head/head_camera_pan.stl" scale="0.001 0.001 0.001" />
+          <mesh filename="file://$(find sobit_edu_description)/meshes/head/head_camera_pan.stl" scale="0.001 0.001 0.001" />
         </geometry>
       </collision>
@@ -70,5 +70,5 @@
         <origin xyz="0.0 0.0 0.0" rpy="0.0 0.0 ${M_PI/2.0}" />
         <geometry>
-          <mesh filename="package://sobit_edu_description/meshes/head/head_camera_tilt.stl" scale="0.001 0.001 0.001" />
+          <mesh filename="file://$(find sobit_edu_description)/meshes/head/head_camera_tilt.stl" scale="0.001 0.001 0.001" />
         </geometry>
         <material name="black" />
@@ -77,5 +77,5 @@
         <origin xyz="0.0 0.0 0.0" rpy="0.0 0.0 ${M_PI/2.0}" />
         <geometry>
-          <mesh filename="package://sobit_edu_description/meshes/head/head_camera_tilt.stl" scale="0.001 0.001 0.001" />
+          <mesh filename="file://$(find sobit_edu_description)/meshes/head/head_camera_tilt.stl" scale="0.001 0.001 0.001" />
         </geometry>
       </collision>

File: sobit_edu_description/urdf/sensor/head_camera.urdf.xacro (robot description, xacro)
@@ -9,7 +9,7 @@
     </joint>
     <link name="${prefix}_link"/>
-    <xacro:azure_kinect parent="${prefix}_link" tf_prefix="${prefix}_" add_cover="false">
+    <!-- <xacro:azure_kinect parent="${prefix}_link" tf_prefix="${prefix}_" add_cover="false">
       <origin xyz="0.0 0 0.0" rpy="0 0 0"/>
-    </xacro:azure_kinect>
+    </xacro:azure_kinect> -->
   </xacro:macro>
 </robot>

File: sobit_edu_description/urdf/sensor/lidar.urdf.xacro (robot description, xacro)
@@ -11,5 +11,5 @@
         <origin rpy="0.0 0.0 ${M_PI}" xyz="0.0 0.0 0.0" />
         <geometry>
-          <mesh filename="package://sobit_edu_description/meshes/sensor/lidar_base.stl" scale="0.001 0.001 0.001" />
+          <mesh filename="file://$(find sobit_edu_description)/meshes/sensor/lidar_base.stl" scale="0.001 0.001 0.001" />
         </geometry>
         <material name="black" />
@@ -18,5 +18,5 @@
         <origin rpy="0.0 0.0 ${M_PI}" xyz="0.0 0.0 0.0" />
         <geometry>
-          <mesh filename="package://sobit_edu_description/meshes/sensor/lidar_base.stl" scale="0.001 0.001 0.001" />
+          <mesh filename="file://$(find sobit_edu_description)/meshes/sensor/lidar_base.stl" scale="0.001 0.001 0.001" />
         </geometry>
       </collision>
