Commit message: [UPD]required dependencies

File: sobit_edu_description/urdf/sensor/matrix.urdf.xacro (robot description, xacro)
@@ -13,5 +13,5 @@
         <origin xyz="0.0 0.0 0.0" rpy="0.0 0.0 0.0" />
         <geometry>
-          <mesh filename="package://sobit_edu_description/meshes/sensor/matrix_base.stl" scale="0.001 0.001 0.001" />
+          <mesh filename="file://$(find sobit_edu_description)/meshes/sensor/matrix_base.stl" scale="0.001 0.001 0.001" />
         </geometry>
         <material name="black" />
@@ -20,5 +20,5 @@
         <origin xyz="0.0 0.0 0.0" rpy="0.0 0.0 0.0" />
         <geometry>
-          <mesh filename="package://sobit_edu_description/meshes/sensor/matrix_base.stl" scale="0.001 0.001 0.001" />
+          <mesh filename="file://$(find sobit_edu_description)/meshes/sensor/matrix_base.stl" scale="0.001 0.001 0.001" />
         </geometry>
       </collision>
@@ -41,5 +41,5 @@
         <origin xyz="0.0 0.0 0.0" rpy="0.0 0.0 ${M_PI}" />
         <geometry>
-          <mesh filename="package://sobit_edu_description/meshes/sensor/matrix.stl" scale="0.001 0.001 0.001" />
+          <mesh filename="file://$(find sobit_edu_description)/meshes/sensor/matrix.stl" scale="0.001 0.001 0.001" />
         </geometry>
         <material name="blue" />
@@ -48,5 +48,5 @@
         <origin xyz="0.0 0.0 0.0" rpy="0.0 0.0 0.0" />
         <geometry>
-          <mesh filename="package://sobit_edu_description/meshes/sensor/matrix.stl" scale="0.001 0.001 0.001" />
+          <mesh filename="file://$(find sobit_edu_description)/meshes/sensor/matrix.stl" scale="0.001 0.001 0.001" />
         </geometry>
       </collision>

File: sobit_edu_description/urdf/sensor/mic.urdf.xacro (robot description, xacro)
@@ -11,5 +11,5 @@
         <origin xyz="0.0 0.0 0.0" rpy="${M_PI/2} 0 ${M_PI/2}" />
         <geometry>
-          <mesh filename="package://sobit_edu_description/meshes/sensor/mic_base.stl" scale="0.001 0.001 0.001" />
+          <mesh filename="file://$(find sobit_edu_description)/meshes/sensor/mic_base.stl" scale="0.001 0.001 0.001" />
         </geometry>
         <material name="black" />
@@ -18,5 +18,5 @@
         <origin xyz="0.0 0.0 0.0" rpy="${M_PI/2} 0 ${M_PI/2}" />
         <geometry>
-          <mesh filename="package://sobit_edu_description/meshes/sensor/mic_base.stl" scale="0.001 0.001 0.001" />
+          <mesh filename="file://$(find sobit_edu_description)/meshes/sensor/mic_base.stl" scale="0.001 0.001 0.001" />
         </geometry>
         <material name="black" />
@@ -39,5 +39,5 @@
         <origin xyz="0.0 0.0 0.0" rpy="${M_PI} 0.0 ${M_PI/2}" />
         <geometry>
-          <mesh filename="package://sobit_edu_description/meshes/sensor/mic.stl" scale="0.001 0.001 0.001" />
+          <mesh filename="file://$(find sobit_edu_description)/meshes/sensor/mic.stl" scale="0.001 0.001 0.001" />
         </geometry>
         <material name="black" />
@@ -46,5 +46,5 @@
         <origin xyz="0.0 0.0 0.0" rpy="${M_PI} 0.0 ${M_PI/2}" />
         <geometry>
-          <mesh filename="package://sobit_edu_description/meshes/sensor/mic.stl" scale="0.001 0.001 0.001" />
+          <mesh filename="file://$(find sobit_edu_description)/meshes/sensor/mic.stl" scale="0.001 0.001 0.001" />
         </geometry>
         <material name="black" />

Commit message: [UPD]ros2_for_sobit_edu

File: sobit_edu_description/robots/sobit_edu.urdf.xacro (robot description, xacro)
@@ -21,16 +21,11 @@
   <xacro:include filename="$(find urg_node)/urdf/hokuyo_ust.urdf.xacro" />
   <!-- <xacro:include filename="$(find azure_kinect_ros_driver)/urdf/azure_kinect.urdf.xacro" /> -->
+  <!-- Add URDF: gazebo -->
+  <xacro:include filename="$(find sobit_edu_description)/urdf/gazebo.urdf.xacro" />
   <!-- Add variables -->
-  <xacro:arg name="enable_gz"                 default="True" />
+  <xacro:arg name="enable_gz"                 default="False" />
+  <xacro:arg name="enable_gz_lidar"           default="True" />
   <xacro:arg name="robot_name"                default="sobit_edu" />
   <xacro:controllers name="joints_control" enable_gz="$(arg enable_gz)" robot_name="$(arg robot_name)" />
-  <!-- Add URDF: gazebo -->
-  <!-- <xacro:include filename="$(find sobit_edu_description)/urdf/gazebo.urdf.xacro" /> -->
-  <gazebo>
-    <!-- <plugin filename="ignition-gazebo-joint-state-publisher-system" name="ignition::gazebo::systems::JointStatePublisher"> -->
-    <plugin filename="gz-sim-joint-state-publisher-system" name="gz::sim::systems::JointStatePublisher">
-      <topic>sobit_edu/joint_states</topic>
-    </plugin>
-  </gazebo>
   <!-- Connect the previous Links and Joints -->
   <xacro:base/>
@@ -45,3 +40,10 @@
   <xacro:matrix prefix="matrix" parent="back_base_link" />
   <xacro:lidar  prefix="lidar"  parent="plate_bottom_link" />
+  <!-- Add Gazebo: plugins -->
+  <xacro:if value="${$(arg enable_gz)}">
+    <xacro:gazebo_sensors robot_name="$(arg robot_name)"
+      enable_gz_lidar="$(arg enable_gz_lidar)"
+      enable_gz_imu="$(arg enable_gz_imu)"
+    />
+  </xacro:if>
 </robot>

File: sobit_edu_description/urdf/arm/arm.transmission.xacro (robot description, xacro)
@@ -5,7 +5,7 @@
     <xacro:position_joint_transmission joint="${prefix}_shoulder_pan_joint"    reduction="1" />
     <xacro:position_joint_transmission joint="${prefix}_shoulder_1_tilt_joint" reduction="1" />
-    <!-- <xacro:position_joint_transmission joint="${prefix}_shoulder_2_tilt_joint" reduction="1" /> -->
+    <xacro:position_joint_transmission joint="${prefix}_shoulder_2_tilt_joint" reduction="1" />
     <xacro:position_joint_transmission joint="${prefix}_elbow_1_tilt_joint"    reduction="1" />
-    <!-- <xacro:position_joint_transmission joint="${prefix}_elbow_2_tilt_joint"    reduction="1" /> -->
+    <xacro:position_joint_transmission joint="${prefix}_elbow_2_tilt_joint"    reduction="1" />
     <xacro:position_joint_transmission joint="${prefix}_wrist_tilt_joint"      reduction="1" />
   </xacro:macro>

File: sobit_edu_description/urdf/arm/arm.urdf.xacro (robot description, xacro)
@@ -95,5 +95,5 @@
       </inertial>
     </link>
-    <!-- <joint name="${prefix}_shoulder_2_tilt_joint" type="revolute">
+    <joint name="${prefix}_shoulder_2_tilt_joint" type="revolute">
       <parent link="${prefix}_shoulder_pan_link" />
       <child link="${prefix}_shoulder_2_tilt_link" />
@@ -103,5 +103,5 @@
       <limit effort="30" lower="${-M_PI/2.0}" upper="${M_PI/2.0}" velocity="${M_PI/2.0}" />
     </joint>
-    <link name="${prefix}_shoulder_2_tilt_link" /> -->
+    <link name="${prefix}_shoulder_2_tilt_link" />
     <joint name="${prefix}_elbow_1_tilt_joint" type="revolute">
       <parent link="${prefix}_shoulder_1_tilt_link" />
@@ -134,5 +134,5 @@
       </inertial>
     </link>
-    <!-- <joint name="${prefix}_elbow_2_tilt_joint" type="revolute">
+    <joint name="${prefix}_elbow_2_tilt_joint" type="revolute">
       <parent link="${prefix}_shoulder_1_tilt_link" />
       <child link="${prefix}_elbow_2_tilt_link" />
@@ -142,5 +142,5 @@
       <limit effort="30" lower="${-M_PI/2.0}" upper="${M_PI/2.0}" velocity="${M_PI/2.0}" />
     </joint>
-    <link name="${prefix}_elbow_2_tilt_link" /> -->
+    <link name="${prefix}_elbow_2_tilt_link" />
     <joint name="${prefix}_wrist_tilt_joint" type="revolute">
       <parent link="${prefix}_elbow_1_tilt_link" />
@@ -152,5 +152,5 @@
     <link name="${prefix}_wrist_tilt_link" />
     <xacro:arm_transmission prefix="${prefix}" />
-    <xacro:arm_gazebo prefix="${prefix}"/>
+    <!-- <xacro:arm_gazebo prefix="${prefix}"/> -->
   </xacro:macro>
 </robot>

File: sobit_edu_description/urdf/base/base.urdf.xacro (robot description, xacro)
@@ -54,5 +54,5 @@
       </inertial>
     </link>
-    <joint name="wheel_l_joint" type="continuous">
+    <joint name="wheel_l_joint" type="fixed">
       <parent link="base_link" />
       <child link="wheel_l_link" />
@@ -81,5 +81,5 @@
       </inertial>
     </link>
-    <joint name="wheel_r_joint" type="continuous">
+    <joint name="wheel_r_joint" type="fixed">
       <parent link="base_link" />
       <child link="wheel_r_link" />

File: sobit_edu_description/urdf/controllers.urdf.xacro (robot description, xacro)
@@ -19,7 +19,5 @@
       <!-- Position Drive: Arm -->
       <joint name="arm_shoulder_pan_joint">
-        <xacro:unless value="${$(arg enable_gz)}">
-          <param name="id">1</param>
-        </xacro:unless>
+        <param name="id">10</param>
         <command_interface name="position">
           <param name="min">-3.141592654</param>
@@ -34,7 +32,5 @@
       </joint>
       <joint name="arm_shoulder_1_tilt_joint">
-        <xacro:unless value="${$(arg enable_gz)}">
-          <param name="id">2</param>
-        </xacro:unless>
+        <param name="id">11</param>
         <!-- <param name="mimic">arm_shoulder_pitch_joint</param>
         <param name="multiplier">-1</param> -->
@@ -52,8 +48,6 @@
         <state_interface name="effort"/>
       </joint>
-      <!-- <joint name="arm_shoulder_2_tilt_joint">
-        <xacro:unless value="${$(arg enable_gz)}">
-          <param name="id">3</param>
-        </xacro:unless>
+      <joint name="arm_shoulder_2_tilt_joint">
+        <param name="id">12</param>
         <command_interface name="position">
           <param name="min">-1.570796327</param>
@@ -66,9 +60,7 @@
         <state_interface name="velocity"/>
         <state_interface name="effort"/>
-      </joint> -->
+      </joint>
       <joint name="arm_elbow_1_tilt_joint">
-        <xacro:unless value="${$(arg enable_gz)}">
-          <param name="id">3</param>
-        </xacro:unless>
+        <param name="id">13</param>
         <command_interface name="position">
           <param name="min">-1.570796327</param>
@@ -77,13 +69,11 @@
         <command_interface name="velocity"/>
         <state_interface name="position">
-          <param name="initial_value">0.0</param>
+          <param name="initial_value">-1.40</param>
         </state_interface>
         <state_interface name="velocity"/>
         <state_interface name="effort"/>
       </joint>
-      <!-- <joint name="arm_elbow_2_tilt_joint">
-        <xacro:unless value="${$(arg enable_gz)}">
-          <param name="id">5</param>
-        </xacro:unless>
+      <joint name="arm_elbow_2_tilt_joint">
+          <param name="id">14</param>
         <command_interface name="position">
           <param name="min">-3.141592654</param>
@@ -92,13 +82,11 @@
         <command_interface name="velocity"/>
         <state_interface name="position">
-          <param name="initial_value">0.0</param>
+          <param name="initial_value">1.4</param>
         </state_interface>
         <state_interface name="velocity"/>
         <state_interface name="effort"/>
-      </joint> -->
+      </joint>
       <joint name="arm_wrist_tilt_joint">
-        <xacro:unless value="${$(arg enable_gz)}">
-          <param name="id">4</param>
-        </xacro:unless>
+        <param name="id">15</param>
         <command_interface name="position">
           <param name="min">-1.570796327</param>
@@ -107,119 +95,12 @@
         <command_interface name="velocity"/>
         <state_interface name="position">
-          <param name="initial_value">0.0</param>
+          <param name="initial_value">-0.17</param>
         </state_interface>
         <state_interface name="velocity"/>
         <state_interface name="effort"/>
       </joint>
-      <joint name="hand_inner_l_joint">
-        <xacro:unless value="${$(arg enable_gz)}">
-          <param name="id">5</param>
-        </xacro:unless>
-        <command_interface name="position">
-          <param name="min">-1.570796327</param>
-          <param name="max">1.570796327</param>
-        </command_interface>
-        <command_interface name="velocity"/>
-        <state_interface name="position">
-          <param name="initial_value">0.0</param>
-        </state_interface>
-        <state_interface name="velocity"/>
-        <state_interface name="effort"/>
-      </joint>
-      <joint name="hand_inner_r_joint">
-        <xacro:unless value="${$(arg enable_gz)}">
-          <param name="id">6</param>
-        </xacro:unless>
-        <command_interface name="position">
-          <param name="min">-1.570796327</param>
-          <param name="max">1.570796327</param>
-        </command_interface>
-        <command_interface name="velocity"/>
-        <state_interface name="position">
-          <param name="initial_value">0.0</param>
-        </state_interface>
-        <state_interface name="velocity"/>
-        <state_interface name="effort"/>
-      </joint>
-      <joint name="hand_outer_l_joint">
-        <xacro:unless value="${$(arg enable_gz)}">
-          <param name="id">7</param>
-        </xacro:unless>
-        <command_interface name="position">
-          <param name="min">-1.570796327</param>
-          <param name="max">1.570796327</param>
-        </command_interface>
-        <command_interface name="velocity"/>
-        <state_interface name="position">
-          <param name="initial_value">0.0</param>
-        </state_interface>
-        <state_interface name="velocity"/>
-        <state_interface name="effort"/>
-      </joint>
-      <joint name="hand_outer_r_joint">
-        <xacro:unless value="${$(arg enable_gz)}">
-          <param name="id">8</param>
-        </xacro:unless>
-        <command_interface name="position">
-          <param name="min">-1.570796327</param>
-          <param name="max">1.570796327</param>
-        </command_interface>
-        <command_interface name="velocity"/>
-        <state_interface name="position">
-          <param name="initial_value">0.0</param>
-        </state_interface>
-        <state_interface name="velocity"/>
-        <state_interface name="effort"/>
-      </joint>
-      <joint name="hand_finger_l_joint">
-        <xacro:unless value="${$(arg enable_gz)}">
-          <param name="id">9</param>
-        </xacro:unless>
-        <command_interface name="position">
-          <param name="min">-1.570796327</param>
-          <param name="max">1.570796327</param>
-        </command_interface>
-        <command_interface name="velocity"/>
-        <state_interface name="position">
-          <param name="initial_value">0.0</param>
-        </state_interface>
-        <state_interface name="velocity"/>
-        <state_interface name="effort"/>
-      </joint>
-      <joint name="hand_finger_r_joint">
-        <xacro:unless value="${$(arg enable_gz)}">
-          <param name="id">10</param>
-        </xacro:unless>
-        <command_interface name="position">
-          <param name="min">-1.570796327</param>
-          <param name="max">1.570796327</param>
-        </command_interface>
-        <command_interface name="velocity"/>
-        <state_interface name="position">
-          <param name="initial_value">0.0</param>
-        </state_interface>
-        <state_interface name="velocity"/>
-        <state_interface name="effort"/>
-      </joint>
-      <!-- <joint name="hand_joint">
-        <xacro:unless value="${$(arg enable_gz)}">
-          <param name="id">7</param>
-        </xacro:unless>
-        <command_interface name="position">
-          <param name="min">-3.141592654</param>
-          <param name="max">3.141592654</param>
-        </command_interface>
-        <command_interface name="velocity"/>
-        <state_interface name="position">
-          <param name="initial_value">0.0</param>
-        </state_interface>
-        <state_interface name="velocity"/>
-        <state_interface name="effort"/>
-      </joint> -->
       <!-- Position Drive: Hand -->
       <joint name="hand_joint">
-        <xacro:unless value="${$(arg enable_gz)}">
-          <param name="id">8</param>
-        </xacro:unless>
+        <param name="id">16</param>
         <command_interface name="position"/>
         <command_interface name="velocity"/>
@@ -230,20 +111,7 @@
         <state_interface name="effort"/>
       </joint>
-      <!-- <xacro:if value="${$(arg enable_gz)}">
-        <joint name="hand_sub_joint">
-          <param name="mimic">hand_joint</param>
-          <param name="multiplier">-1</param>
-          <command_interface name="position"/>
-          <command_interface name="velocity"/>
-          <state_interface name="position"/>
-          <state_interface name="velocity"/>
-          <state_interface name="effort"/>
-        </joint>
-      </xacro:if> -->
       <!-- Position Drive: Head -->
       <joint name="head_camera_pan_joint">
-        <xacro:unless value="${$(arg enable_gz)}">
-          <param name="id">11</param>
-        </xacro:unless>
+        <param name="id">21</param>
         <command_interface name="position">
           <param name="min">-3.141592654</param>
@@ -258,7 +126,5 @@
       </joint>
       <joint name="head_camera_tilt_joint">
-        <xacro:unless value="${$(arg enable_gz)}">
-          <param name="id">12</param>
-        </xacro:unless>
+        <param name="id">22</param>
         <command_interface name="position">
           <param name="min">-1.570796327</param>

File: sobit_edu_description/urdf/hand/hand.urdf.xacro (robot description, xacro)
@@ -205,5 +205,4 @@
     </link>
     <xacro:hand_transmission prefix_hand="${prefix_hand}" prefix_finger="${prefix_finger}" />
-    <xacro:hand_gazebo prefix="${prefix_hand}" />
   </xacro:macro>
 </robot>

File: sobit_edu_description/urdf/head/head.urdf.xacro (robot description, xacro)
@@ -96,5 +96,5 @@
     </link>
     <xacro:head_transmission prefix="${prefix}" />
-    <xacro:head_gazebo prefix="${prefix}" />
+    <!-- <xacro:head_gazebo prefix="${prefix}" /> -->
   </xacro:macro>
 </robot>

File: sobit_edu_description/urdf/sensor/lidar.urdf.xacro (robot description, xacro)
@@ -31,4 +31,18 @@
       </inertial>
     </link>
+    <joint name="${prefix}_sim_joint" type="fixed">
+      <parent link="${prefix}_base_link" />
+      <child link="sim_laser_frame" />
+      <origin xyz="0.3 0 0.0" rpy="0 0 0" />
+    </joint>
+    <link name="sim_laser_frame">
+      <inertial>
+        <origin xyz="0.3 0 0" rpy="0 0 0" />
+        <mass value="0.2" />
+        <inertia ixx="0.001" ixy="0" ixz="0"
+                 iyy="0.001" iyz="0"
+                 izz="0.001" />
+      </inertial>
+    </link>
     <xacro:hokuyo_ust_mount prefix="${prefix}" parent="${prefix}_base_link" topic="scan" >
       <origin xyz="0.1105 0.0 0.0" rpy="0.0 0.0 0.0" />

Commit message: change the camera to gemini from azure kinect

File: sobit_edu_description/robots/sobit_edu.urdf.xacro (robot description, xacro)
@@ -20,5 +20,5 @@
   <xacro:include filename="$(find sobit_edu_description)/urdf/sensor/head_camera.urdf.xacro" />
   <xacro:include filename="$(find urg_node)/urdf/hokuyo_ust.urdf.xacro" />
-  <xacro:include filename="$(find azure_kinect_ros_driver)/urdf/azure_kinect.urdf.xacro" />
+  <xacro:include filename="$(find orbbec_description)/urdf/gemini_336.urdf.xacro" />
   <!-- Add URDF: gazebo -->
   <xacro:include filename="$(find sobit_edu_description)/urdf/gazebo.urdf.xacro" />

File: sobit_edu_description/urdf/sensor/head_camera.urdf.xacro (robot description, xacro)
@@ -9,7 +9,10 @@
     </joint>
     <link name="${prefix}_link"/>
-    <xacro:azure_kinect parent="${prefix}_link" tf_prefix="${prefix}_" add_cover="false">
+    <!-- <xacro:azure_kinect parent="${prefix}_link" tf_prefix="${prefix}_" add_cover="false">
       <origin xyz="0.0 0 0.0" rpy="0 0 0"/>
-    </xacro:azure_kinect>
+    </xacro:azure_kinect> -->
+    <xacro:gemini_336 parent="${prefix}_link" tf_prefix="${prefix}_">
+      <origin xyz="0.0 0 0.0" rpy="0 0 0"/>
+    </xacro:gemini_336>
   </xacro:macro>
 </robot>

Commit message: Update SOBIT EDU of jazzy

File: sobit_edu_description/robots/sobit_edu.urdf.xacro (robot description, xacro)
@@ -29,4 +29,6 @@
   <xacro:arg name="enable_gz_head_cam_color"  default="True" />
   <xacro:arg name="enable_gz_head_cam_depth"  default="True" />
+  <!-- DXL Ports -->
+  <xacro:arg name="dxl_se_port"  default="/dev/ttyUSB1" />
   <!-- Connect the previous Links and Joints -->
   <xacro:base/>

File: sobit_edu_description/urdf/controllers.urdf.xacro (robot description, xacro)
@@ -11,6 +11,7 @@
         </xacro:if>
         <xacro:unless value="${$(arg enable_gz)}">
+          <xacro:property name="dxl_se_port" value="$(arg dxl_se_port)"/>
           <plugin>dynamixel_hardware/DynamixelHardware</plugin>
-          <param name="port_name">/dev/ttyUSB1</param>
+          <param name="port_name">${dxl_se_port}</param>
           <param name="baud_rate">1000000</param>
           <!-- <param name="use_dummy">true</param> -->
