Commit message: UPD controller is now split into robot parts

File: sobit_edu_description/robots/sobit_edu.urdf.xacro (robot description, xacro)
@@ -25,37 +25,48 @@
   <xacro:arg name="enable_gz"                 default="False" />
   <xacro:arg name="enable_gz_lidar"           default="True" />
+  <xacro:arg name="enable_gz_imu"             default="True" />
   <xacro:arg name="robot_name"                default="sobit_edu" />
   <xacro:arg name="head_camera_name"          default="gemini_336" />
   <xacro:arg name="enable_gz_head_cam_color"  default="True" />
   <xacro:arg name="enable_gz_head_cam_depth"  default="True" />
+  <!-- Activate Components -->
+  <xacro:arg name="enable_mobile_base"  default="True" />
+  <xacro:arg name="enable_head"         default="True" />
+  <xacro:arg name="enable_arm"          default="True" />
+  <xacro:arg name="enable_hand"         default="True" />
   <!-- Connect the previous Links and Joints -->
   <xacro:base/>
   <xacro:stack_hexagons parent="base_link" />
   <xacro:cover  prefix="cover"  parent="plate_top_link" />
-  <xacro:lidar  prefix="lidar"  parent="plate_bottom_link" />
-  <xacro:arm    prefix="arm"    parent="plate_top_link" />
-  <xacro:hand   prefix_hand="hand" prefix_finger="finger" parent="arm_hand_link" />
   <xacro:back   prefix="back"   parent="plate_top_link" />
-  <xacro:head   prefix="head"   parent="back_base_link" />
-  <!-- <xacro:head_camera prefix="head_camera" parent="head_camera_tilt_link" /> -->
+  <xacro:if value="${$(arg enable_arm)}">
+    <xacro:arm    prefix="arm"    parent="plate_top_link" />
+  </xacro:if>
+  <xacro:if value="${$(arg enable_hand)}">
+    <xacro:hand   prefix_hand="hand" prefix_finger="finger" parent="arm_hand_link" />
+  </xacro:if>
+  <xacro:if value="${$(arg enable_head)}">
+    <xacro:head   prefix="head"   parent="back_base_link" />
+    <!-- Xtion -->
+    <xacro:if value="$(eval head_camera_name == 'xtion')">
+    <xacro:include filename="$(find sobit_edu_description)/urdf/sensor/xtion.urdf.xacro" />
+    <xacro:include filename="$(find sobit_edu_description)/urdf/sensor/xtion_fixed.urdf.xacro" />
+      <xacro:xtion_fixed prefix="head_camera" parent="head_camera_tilt_link"/>
+    </xacro:if>
+    <!-- AzureKinect -->
+    <xacro:if value="$(eval head_camera_name == 'azure_kinect')">
+      <xacro:include filename="$(find azure_kinect_ros_driver)/urdf/azure_kinect.urdf.xacro" />
+      <xacro:include filename="$(find sobit_edu_description)/urdf/sensor/azure_camera.urdf.xacro" />
+      <xacro:azure_camera prefix="head_camera" parent="head_camera_tilt_link" />
+    </xacro:if>
+    <!-- Gemini336L -->
+    <xacro:if value="$(eval head_camera_name == 'gemini_336')">
+      <xacro:include filename="$(find orbbec_description)/urdf/gemini_336.urdf.xacro" />
+      <xacro:head_camera prefix="head_camera" parent="head_camera_tilt_link" />
+    </xacro:if>
+  </xacro:if>
   <xacro:mic    prefix="mic"    parent="back_base_link" />
   <xacro:matrix prefix="matrix" parent="back_base_link" />
-  <!-- Xtion -->
-  <xacro:if value="$(eval head_camera_name == 'xtion')">
-  <xacro:include filename="$(find sobit_edu_description)/urdf/sensor/xtion.urdf.xacro" />
-  <xacro:include filename="$(find sobit_edu_description)/urdf/sensor/xtion_fixed.urdf.xacro" />
-    <xacro:xtion_fixed prefix="head_camera" parent="head_camera_tilt_link"/>
-  </xacro:if>
-  <!-- AzureKinect -->
-  <xacro:if value="$(eval head_camera_name == 'azure_kinect')">
-    <xacro:include filename="$(find azure_kinect_ros_driver)/urdf/azure_kinect.urdf.xacro" />
-    <xacro:include filename="$(find sobit_edu_description)/urdf/sensor/azure_camera.urdf.xacro" />
-    <xacro:azure_camera prefix="head_camera" parent="head_camera_tilt_link" />
-  </xacro:if>
-  <!-- Gemini336L -->
-  <xacro:if value="$(eval head_camera_name == 'gemini_336')">
-    <xacro:include filename="$(find orbbec_description)/urdf/gemini_336.urdf.xacro" />
-    <xacro:head_camera prefix="head_camera" parent="head_camera_tilt_link" />
-  </xacro:if>
+  <xacro:lidar  prefix="lidar"  parent="plate_bottom_link" />
   <!-- Add Dynamixel plugins -->
   <xacro:controllers name="joints_control" enable_gz="$(arg enable_gz)" robot_name="$(arg robot_name)" />

File: sobit_edu_description/urdf/controllers.urdf.xacro (robot description, xacro)
@@ -3,5 +3,5 @@
 <robot name="sobit_edu_controllers" xmlns:xacro="http://www.ros.org/wiki/xacro">
   <xacro:macro name="controllers" params="name enable_gz:=False robot_name:=sobit_edu">
-    <ros2_control name="${name}_arm" type="system">
+    <ros2_control name="dynamixel_controllers" type="system">
     <!-- <ros2_control name="joints_control" type="system"> -->
       <hardware>
@@ -17,191 +17,13 @@
         </xacro:unless>
       </hardware>
-      <!-- Position Drive: Arm -->
-      <joint name="arm_shoulder_roll_joint">
-        <xacro:unless value="${$(arg enable_gz)}">
-          <param name="id">10</param>
-          <param name="control_mode">0</param>
-          <param name="interface">rs</param>
-        </xacro:unless>
-        <command_interface name="position">
-          <param name="min">-3.141592654</param>
-          <param name="max">3.141592654</param>
-        </command_interface>
-        <!-- <command_interface name="velocity"/> -->
-        <state_interface name="position">
-          <param name="initial_value">0.0</param>
-        </state_interface>
-        <state_interface name="velocity"/>
-        <state_interface name="effort"/>
-      </joint>
-      <joint name="arm_shoulder_pitch_sub_joint">
-        <xacro:unless value="${$(arg enable_gz)}">
-          <param name="id">12</param>
-          <param name="control_mode">0</param>
-          <param name="interface">rs</param>
-        </xacro:unless>
-        <!-- <param name="mimic">arm_shoulder_pitch_joint</param>
-        <param name="multiplier">-1</param> -->
-        <!-- <command_interface name="position"/> -->
-        <command_interface name="position">
-          <param name="min">-2.356194490192345</param>
-          <param name="max">1.570796327</param>
-        </command_interface>
-        <!-- <command_interface name="velocity"/> -->
-        <state_interface name="position">
-          <param name="initial_value">0.0</param>
-        </state_interface>
-        <!-- <state_interface name="position"/> -->
-        <state_interface name="velocity"/>
-        <state_interface name="effort"/>
-      </joint>
-      <joint name="arm_shoulder_pitch_joint">
-        <xacro:unless value="${$(arg enable_gz)}">
-          <param name="id">11</param>
-          <param name="control_mode">0</param>
-          <param name="interface">rs</param>
-        </xacro:unless>
-        <command_interface name="position">
-          <param name="min">-1.570796327</param>
-          <param name="max">2.356194490192345</param>
-        </command_interface>
-        <!-- <command_interface name="velocity"/> -->
-        <state_interface name="position">
-          <param name="initial_value">0.0</param>
-        </state_interface>
-        <state_interface name="velocity"/>
-        <state_interface name="effort"/>
-      </joint>
-      <joint name="arm_elbow_pitch_joint">
-        <xacro:unless value="${$(arg enable_gz)}">
-          <param name="id">13</param>
-          <param name="control_mode">0</param>
-          <param name="interface">rs</param>
-        </xacro:unless>
-        <command_interface name="position">
-          <param name="min">-1.570796327</param>
-          <param name="max">1.570796327</param>
-        </command_interface>
-        <!-- <command_interface name="velocity"/> -->
-        <state_interface name="position">
-          <param name="initial_value">0.0</param>
-        </state_interface>
-        <state_interface name="velocity"/>
-        <state_interface name="effort"/>
-      </joint>
-      <joint name="arm_forearm_roll_joint">
-        <xacro:unless value="${$(arg enable_gz)}">
-          <param name="id">14</param>
-          <param name="control_mode">0</param>
-          <param name="interface">rs</param>
-        </xacro:unless>
-        <command_interface name="position">
-          <param name="min">-3.141592654</param>
-          <param name="max">3.141592654</param>
-        </command_interface>
-        <!-- <command_interface name="velocity"/> -->
-        <state_interface name="position">
-          <param name="initial_value">0.0</param>
-        </state_interface>
-        <state_interface name="velocity"/>
-        <state_interface name="effort"/>
-      </joint>
-      <joint name="arm_wrist_pitch_joint">
-        <xacro:unless value="${$(arg enable_gz)}">
-          <param name="id">15</param>
-          <param name="control_mode">0</param>
-          <param name="interface">rs</param>
-        </xacro:unless>
-        <command_interface name="position">
-          <param name="min">-1.570796327</param>
-          <param name="max">1.570796327</param>
-        </command_interface>
-        <!-- <command_interface name="velocity"/> -->
-        <state_interface name="position">
-          <param name="initial_value">0.0</param>
-        </state_interface>
-        <state_interface name="velocity"/>
-        <state_interface name="effort"/>
-      </joint>
-      <joint name="arm_wrist_roll_joint">
-        <xacro:unless value="${$(arg enable_gz)}">
-          <param name="id">16</param>
-          <param name="control_mode">0</param>
-          <param name="interface">rs</param>
-        </xacro:unless>
-        <command_interface name="position">
-          <param name="min">-3.141592654</param>
-          <param name="max">3.141592654</param>
-        </command_interface>
-        <!-- <command_interface name="velocity"/> -->
-        <state_interface name="position">
-          <param name="initial_value">0.0</param>
-        </state_interface>
-        <state_interface name="velocity"/>
-        <state_interface name="effort"/>
-      </joint>
-      <!-- Position Drive: Hand -->
-      <joint name="hand_joint">
-        <xacro:unless value="${$(arg enable_gz)}">
-          <param name="id">17</param>
-          <param name="control_mode">6</param>
-          <param name="Goal_Current">50</param>
-          <param name="interface">rs</param>
-          <param name="gear_ratio">-59.504383354</param>
-        </xacro:unless>
-        <command_interface name="position"/>
-        <!-- <command_interface name="velocity"/> -->
-        <state_interface name="position">
-          <param name="initial_value">0.0</param>
-        </state_interface>
-        <state_interface name="velocity"/>
-        <state_interface name="effort"/>
-      </joint>
-      <xacro:if value="${$(arg enable_gz)}">
-        <joint name="hand_sub_joint">
-          <param name="mimic">hand_joint</param>
-          <param name="multiplier">-1</param>
-          <command_interface name="position"/>
-          <!-- <command_interface name="velocity"/> -->
-          <state_interface name="position"/>
-          <state_interface name="velocity"/>
-          <state_interface name="effort"/>
-        </joint>
+      <xacro:if value="${$(arg enable_head)}">
+        <xacro:dxl_head_controllers prefix="head"  enable_gz="${$(arg enable_gz)}"/>
       </xacro:if>
-      <!-- Position Drive: Head -->
-      <joint name="head_camera_pan_joint">
-        <xacro:unless value="${$(arg enable_gz)}">
-          <param name="id">21</param>
-          <param name="control_mode">0</param>
-          <param name="interface">rs</param>
-        </xacro:unless>
-        <command_interface name="position">
-          <param name="min">-3.141592654</param>
-          <param name="max">3.141592654</param>
-        </command_interface>
-        <!-- <command_interface name="velocity"/> -->
-        <state_interface name="position">
-          <param name="initial_value">0.0</param>
-        </state_interface>
-        <state_interface name="velocity"/>
-        <state_interface name="effort"/>
-      </joint>
-      <joint name="head_camera_tilt_joint">
-        <xacro:unless value="${$(arg enable_gz)}">
-          <param name="id">22</param>
-          <param name="control_mode">0</param>
-          <param name="interface">rs</param>
-        </xacro:unless>
-        <command_interface name="position">
-          <param name="min">-1.570796327</param>
-          <param name="max">1.570796327</param>
-        </command_interface>
-        <!-- <command_interface name="velocity"/> -->
-        <state_interface name="position">
-          <param name="initial_value">0.0</param>
-        </state_interface>
-        <state_interface name="velocity"/>
-        <state_interface name="effort"/>
-      </joint>
+      <xacro:if value="${$(arg enable_arm)}">
+        <xacro:dxl_arm_controllers  prefix="arm"   enable_gz="${$(arg enable_gz)}"/>
+      </xacro:if>
+      <xacro:if value="${$(arg enable_hand)}">
+        <xacro:dxl_hand_controllers prefix="hand"  enable_gz="${$(arg enable_gz)}"/>
+      </xacro:if>
     </ros2_control>
     <!-- Differential Drive -->
@@ -247,3 +69,196 @@
     </xacro:if>
   </xacro:macro>
+  <xacro:macro name="dxl_head_controllers"  params="prefix enable_gz:=False">
+    <!-- Position Drive: Head -->
+    <joint name="head_camera_pan_joint">
+      <xacro:unless value="${$(arg enable_gz)}">
+        <param name="id">21</param>
+        <param name="control_mode">0</param>
+        <param name="interface">rs</param>
+      </xacro:unless>
+      <command_interface name="position">
+        <param name="min">-3.141592654</param>
+        <param name="max">3.141592654</param>
+      </command_interface>
+      <!-- <command_interface name="velocity"/> -->
+      <state_interface name="position">
+        <param name="initial_value">0.0</param>
+      </state_interface>
+      <state_interface name="velocity"/>
+      <state_interface name="effort"/>
+    </joint>
+    <joint name="head_camera_tilt_joint">
+      <xacro:unless value="${$(arg enable_gz)}">
+        <param name="id">22</param>
+        <param name="control_mode">0</param>
+        <param name="interface">rs</param>
+      </xacro:unless>
+      <command_interface name="position">
+        <param name="min">-1.570796327</param>
+        <param name="max">1.570796327</param>
+      </command_interface>
+      <!-- <command_interface name="velocity"/> -->
+      <state_interface name="position">
+        <param name="initial_value">0.0</param>
+      </state_interface>
+      <state_interface name="velocity"/>
+      <state_interface name="effort"/>
+    </joint>
+  </xacro:macro>
+  <xacro:macro name="dxl_arm_controllers"  params="prefix enable_gz:=False">
+    <!-- Position Drive: Arm -->
+    <joint name="arm_shoulder_roll_joint">
+      <xacro:unless value="${$(arg enable_gz)}">
+        <param name="id">10</param>
+        <param name="control_mode">0</param>
+        <param name="interface">rs</param>
+      </xacro:unless>
+      <command_interface name="position">
+        <param name="min">-3.141592654</param>
+        <param name="max">3.141592654</param>
+      </command_interface>
+      <!-- <command_interface name="velocity"/> -->
+      <state_interface name="position">
+        <param name="initial_value">0.0</param>
+      </state_interface>
+      <state_interface name="velocity"/>
+      <state_interface name="effort"/>
+    </joint>
+    <joint name="arm_shoulder_pitch_sub_joint">
+      <xacro:unless value="${$(arg enable_gz)}">
+        <param name="id">12</param>
+        <param name="control_mode">0</param>
+        <param name="interface">rs</param>
+      </xacro:unless>
+      <!-- <param name="mimic">arm_shoulder_pitch_joint</param>
+      <param name="multiplier">-1</param> -->
+      <!-- <command_interface name="position"/> -->
+      <command_interface name="position">
+        <param name="min">-2.356194490192345</param>
+        <param name="max">1.570796327</param>
+      </command_interface>
+      <!-- <command_interface name="velocity"/> -->
+      <state_interface name="position">
+        <param name="initial_value">0.0</param>
+      </state_interface>
+      <!-- <state_interface name="position"/> -->
+      <state_interface name="velocity"/>
+      <state_interface name="effort"/>
+    </joint>
+    <joint name="arm_shoulder_pitch_joint">
+      <xacro:unless value="${$(arg enable_gz)}">
+        <param name="id">11</param>
+        <param name="control_mode">0</param>
+        <param name="interface">rs</param>
+      </xacro:unless>
+      <command_interface name="position">
+        <param name="min">-1.570796327</param>
+        <param name="max">2.356194490192345</param>
+      </command_interface>
+      <!-- <command_interface name="velocity"/> -->
+      <state_interface name="position">
+        <param name="initial_value">0.0</param>
+      </state_interface>
+      <state_interface name="velocity"/>
+      <state_interface name="effort"/>
+    </joint>
+    <joint name="arm_elbow_pitch_joint">
+      <xacro:unless value="${$(arg enable_gz)}">
+        <param name="id">13</param>
+        <param name="control_mode">0</param>
+        <param name="interface">rs</param>
+      </xacro:unless>
+      <command_interface name="position">
+        <param name="min">-1.570796327</param>
+        <param name="max">1.570796327</param>
+      </command_interface>
+      <!-- <command_interface name="velocity"/> -->
+      <state_interface name="position">
+        <param name="initial_value">0.0</param>
+      </state_interface>
+      <state_interface name="velocity"/>
+      <state_interface name="effort"/>
+    </joint>
+    <joint name="arm_forearm_roll_joint">
+      <xacro:unless value="${$(arg enable_gz)}">
+        <param name="id">14</param>
+        <param name="control_mode">0</param>
+        <param name="interface">rs</param>
+      </xacro:unless>
+      <command_interface name="position">
+        <param name="min">-3.141592654</param>
+        <param name="max">3.141592654</param>
+      </command_interface>
+      <!-- <command_interface name="velocity"/> -->
+      <state_interface name="position">
+        <param name="initial_value">0.0</param>
+      </state_interface>
+      <state_interface name="velocity"/>
+      <state_interface name="effort"/>
+    </joint>
+    <joint name="arm_wrist_pitch_joint">
+      <xacro:unless value="${$(arg enable_gz)}">
+        <param name="id">15</param>
+        <param name="control_mode">0</param>
+        <param name="interface">rs</param>
+      </xacro:unless>
+      <command_interface name="position">
+        <param name="min">-1.570796327</param>
+        <param name="max">1.570796327</param>
+      </command_interface>
+      <!-- <command_interface name="velocity"/> -->
+      <state_interface name="position">
+        <param name="initial_value">0.0</param>
+      </state_interface>
+      <state_interface name="velocity"/>
+      <state_interface name="effort"/>
+    </joint>
+    <joint name="arm_wrist_roll_joint">
+      <xacro:unless value="${$(arg enable_gz)}">
+        <param name="id">16</param>
+        <param name="control_mode">0</param>
+        <param name="interface">rs</param>
+      </xacro:unless>
+      <command_interface name="position">
+        <param name="min">-3.141592654</param>
+        <param name="max">3.141592654</param>
+      </command_interface>
+      <!-- <command_interface name="velocity"/> -->
+      <state_interface name="position">
+        <param name="initial_value">0.0</param>
+      </state_interface>
+      <state_interface name="velocity"/>
+      <state_interface name="effort"/>
+    </joint>
+  </xacro:macro>
+  <xacro:macro name="dxl_hand_controllers"  params="prefix enable_gz:=False">
+    <!-- Position Drive: Hand -->
+    <joint name="hand_joint">
+      <xacro:unless value="${$(arg enable_gz)}">
+        <param name="id">17</param>
+        <param name="control_mode">6</param>
+        <param name="Goal_Current">50</param>
+        <param name="interface">rs</param>
+        <param name="gear_ratio">-59.504383354</param>
+      </xacro:unless>
+      <command_interface name="position"/>
+      <!-- <command_interface name="velocity"/> -->
+      <state_interface name="position">
+        <param name="initial_value">0.0</param>
+      </state_interface>
+      <state_interface name="velocity"/>
+      <state_interface name="effort"/>
+    </joint>
+    <xacro:if value="${$(arg enable_gz)}">
+      <joint name="hand_sub_joint">
+        <param name="mimic">hand_joint</param>
+        <param name="multiplier">-1</param>
+        <command_interface name="position"/>
+        <!-- <command_interface name="velocity"/> -->
+        <state_interface name="position"/>
+        <state_interface name="velocity"/>
+        <state_interface name="effort"/>
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
File: sobit_edu_description/urdf/gazebo.urdf.xacro (robot description, xacro)
@@ -4,5 +4,5 @@
   <xacro:macro name="gazebo_sensors" params="robot_name enable_gz_front_cam_color:=True enable_gz_back_cam_color:=True enable_gz_head_cam_color:=True enable_gz_head_cam_depth:=True enable_gz_hand_cam_color:=True enable_gz_hand_cam_depth:=True enable_gz_lidar:=True enable_gz_imu:=True">
     <!-- Sensor: LiDAR -->
-    <xacro:if value="${enable_gz_lidar}">
+    <xacro:if value="${$(arg enable_gz_lidar) and $(arg enable_mobile_base)}">
       <gazebo reference="lidar_laser">
         <sensor name="lidar" type="gpu_lidar">
@@ -39,5 +39,5 @@
     </xacro:if>
     <!-- Sensor - Head Camera (Color) -->
-    <xacro:if value="${enable_gz_head_cam_color}">
+    <xacro:if value="${$(arg enable_gz_head_cam_color) and $(arg enable_head)}">
       <!-- Xtion -->
       <xacro:if value="$(eval head_camera_name == 'xtion')">
@@ -138,5 +138,5 @@
     </xacro:if>
     <!-- Sensor - Head Camera (Depth) -->
-    <xacro:if value="${enable_gz_head_cam_depth}">
+    <xacro:if value="${$(arg enable_gz_head_cam_depth) and $(arg enable_head)}">
       <!-- Xtion -->
       <xacro:if value="$(eval head_camera_name == 'xtion')">
